File: Hardware/Ring-Light/SEG_1-8.kicad_sch (KiCad schematic)
At the start: 78 parts, among them IC1 TPS92624QPWPRQ1, IC2 74HC125PW,112, IC3 74HC125PW,112, IC4 TPS92624QPWPRQ1

Commit message: .
Parts:
- removed D11, D12, D17, D18, D19, D2, D20, D21, D22, D23, D24, D3, D5, D6, D8, D9: LED, Library:STW9Q14CT0U0HA, symbol Library:LED
- D1, D10, D13, D14, D15, D16, D4, D7: footprint Library:STW9Q14CT0U0HA -> Library:GWJTLRS1EMLVL5XX531
Connections:
- net GND: now also D1.1 (K), D1.2 (K), D10.1 (K), D10.2 (K), D13.1 (K), D13.2 (K), D14.1 (K), D14.2 (K), D15.1 (K), D15.2 (K), D16.1 (K), D16.2 (K), D4.1 (K), D4.2 (K), D7.1 (K), D7.2 (K)
- net at IC1.15 (OUT3), R11.2, R7.2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: now also D7.3 (A), D7.4 (A); no longer D7.2 (A), D7.5 (A)
- net at IC4.19 (OUT1), R25.2, R29.2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: now also D13.3 (A), D13.4 (A); no longer D13.2 (A), D13.5 (A)
- net at IC4.13 (OUT4), R28.2, R32.2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: now also D16.3 (A), D16.4 (A); no longer D16.2 (A), D16.5 (A)
- net at IC4.15 (OUT3), R27.2, R31.2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: now also D15.3 (A), D15.4 (A); no longer D15.2 (A), D15.5 (A)
- net at IC4.17 (OUT2), R26.2, R30.2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: now also D14.3 (A), D14.4 (A); no longer D14.2 (A), D14.5 (A)
- net at IC1.19 (OUT1), R1.2, R2.2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: now also D1.3 (A), D1.4 (A); no longer D1.2 (A), D1.5 (A)
- net at IC1.13 (OUT4), R10.2, R12.2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: now also D10.3 (A), D10.4 (A); no longer D10.2 (A), D10.5 (A)
- net at IC1.17 (OUT2), R4.2, R5.2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: now also D4.3 (A), D4.4 (A); no longer D4.2 (A), D4.5 (A)

Commit message: m
Parts:
- removed C16, C17: 1uF, symbol Device:C_Small
- removed C18: 0.1uF, symbol Device:C_Small
- removed C19, C21: 10nF, symbol Device:C_Small
- removed D13, D14, D15, D16: LED, Library:GWJTLRS1EMLVL5XX531, symbol Library:LED
- removed IC2: 74HC125PW,112, Library:SOP65P640X110-14N, symbol Library:74HC125PW,112
- removed IC4: TPS92624QPWPRQ1, Library:SOP65P640X120-21N, symbol Library:TPS92624QPWPRQ1
- removed R21, R22, R23, R24, R29, R3, R30, R31, R32, R33, R34, R35, R36, R6: 162, symbol Device:R_Small
- added C5, C6, C7, C8: 10nF, symbol Device:C_Small
- added C9: 1uF, symbol Device:C_Small
- added D5, D6, D7, D8: LED, Library:GWJTLRS1EMLVL5XX531, symbol Library:LED
- added R10, R13, R14, R15, R16, R9: 162, symbol Device:R_Small
- added U18: 74HC125PW,112, Library:SOP65P640X110-14N, symbol Library:74HC125PW,112
- added U2: TPS92624QPWPRQ1, Library:SOP65P640X120-21N, symbol Library:TPS92624QPWPRQ1
- C20: value 10nF -> 1uF
- C22: value 10nF -> 0.1uF
- renumbered C7 to C18, C6 to C19, C5 to C21, D4 to D2, D7 to D3, D10 to D4, R13 to R21, R14 to R22, R15 to R23, R16 to R24, R4 to R3, R5 to R4, R7 to R5, R9 to R6, R8 to R7, R10 to R8, IC1 to U1, IC3 to U17
Connections:
- net VLED is gone; now on net +12V: C19.2, C21.2, R17.2, R19.2, R21.1, R22.1, R23.1, R24.1, U1.1 (SUPPLY)
- net +3.3V: now also C9.2, U18.14 (VCC)
- net EN1: now also U18.1 (~{1OE})
- net EN2: now also U18.4 (~{2OE})
- net EN3: now also U18.10 (~{3OE})
- net EN4: now also U18.13 (~{4OE})
- net GND: now also C20.1, C22.1, C5.2, C6.2, C7.2, C8.2, C9.1, D5.1 (K), D5.2 (K), D6.1 (K), D6.2 (K), D7.1 (K), D7.2 (K), D8.1 (K), D8.2 (K), U18.7 (GND), U2.21 (EP); no longer C20.2, C22.2
- net PWM: now also U18.12 (4A), U18.2 (1A), U18.5 (2A), U18.9 (3A)
- net at C3.1, R5.1, R6.1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: no longer R11.1
- net at D3.3 (A), D3.4 (A), R5.2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: no longer R11.2
- net +12V: now reaches R25.1
- net +12V: now also C20.2, C22.2, R26.1, R27.1, R28.1, U2.1 (SUPPLY); no longer C20.1
- net at R25.2: now also U2.2 (IN1)
- net at R19.1, R20.2: now also U2.6 (DIAGEN)
- net at R28.2: now also U2.5 (IN4)
- net at R27.2: now also U2.4 (IN3)
- net at R26.2: now also U2.3 (IN2)
- net at C4.1, R7.1, R8.1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: no longer R12.1
- net at D4.3 (A), D4.4 (A), R7.2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: no longer R12.2
- new net: C8.1, R15.1, R16.1, U2.14 (RES4)
- new net: D8.3 (A), D8.4 (A), R15.2, R16.2, U2.13 (OUT4)
- new net: C6.1, R11.1, R12.1, U2.18 (RES2)
- new net: D6.3 (A), D6.4 (A), R11.2, R12.2, U2.17 (OUT2)
- new net: C5.1, R10.1, R9.1, U2.20 (RES1)
- new net: C7.1, R13.1, R14.1, U2.16 (RES3)
- new net: D7.3 (A), D7.4 (A), R13.2, R14.2, U2.15 (OUT3)
- new net: D5.3 (A), D5.4 (A), R10.2, R9.2, U2.19 (OUT1)
- new net: U18.11 (4Y), U2.10 (PWM4)
- new net: U18.3 (1Y), U2.7 (PWM1)
- new net: U18.6 (2Y), U2.8 (PWM2)
- new net: U18.8 (3Y), U2.9 (PWM3)
