File: Hardware/Ring-Light/SEG_17-24.kicad_sch (KiCad schematic)
At the start: 62 parts, among them IC10 74HC125PW,112, IC11 TPS92624QPWPRQ1, IC12 TPS92624QPWPRQ1, IC9 74HC125PW,112

Commit message: m
Parts:
- renumbered C33 to C37, C34 to C38, C35 to C39, C36 to C40, C37 to C41, C38 to C42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
