File: Hardware/Ring-Light/SEG_25-32.kicad_sch (KiCad schematic)
At the start: 62 parts, among them IC13 74HC125PW,112, IC14 74HC125PW,112, IC15 TPS92624QPWPRQ1, IC16 TPS92624QPWPRQ1

Commit message: m
Parts:
- renumbered C47 to C51, C48 to C52, C49 to C53, C50 to C54, C51 to C55, C52 to C56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
