File: Hardware/Ring-Light/SEG_9-16.kicad_sch (KiCad schematic)
At the start: 62 parts, among them IC5 74HC125PW,112, IC6 74HC125PW,112, IC7 TPS92624QPWPRQ1, IC8 TPS92624QPWPRQ1

Commit message: m
Parts:
- renumbered C10 to C23, C11 to C24, C12 to C25, C13 to C26, C23 to C27, C24 to C28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
