File: Hardware/Ring-Light/Ring-Light.kicad_pcb (KiCad board)
At the start: 2 copper layers, 122 x 122 mm, 32 parts

Commit message: m
Parts:
- removed LED** (x2), LED**1, LED**10, LED**11, LED**12, LED**13, LED**14, LED**15, LED**16, LED**17, LED**18, LED**19, LED**2, LED**20, LED**21, LED**22, LED**23, LED**24, LED**25, LED**26, LED**27, LED**28, LED**29, LED**3, LED**30, LED**4, LED**5, LED**6, LED**7, LED**8, LED**9: GWJTLRS1EMLVL5XX531, Library:GWJTLRS1EMLVL5XX531
- added C1: 0.1uF, Capacitor_SMD:C_0603_1608Metric, F.Cu at (10.4, 97.0)
- added C1: 0.1uF, Capacitor_SMD:C_0603_1608Metric, F.Cu at (46.8, 98.4)
- added C10: 0.1uF, Capacitor_SMD:C_0603_1608Metric, F.Cu at (78.2, 148.5)
- added C11: 1uF, Capacitor_SMD:C_0805_2012Metric, F.Cu at (77.3, 150.2)
- added C12: 10nF, Capacitor_SMD:C_0603_1608Metric, F.Cu at (78.3, 143.8)
- added C13: 0.1uF, Capacitor_SMD:C_0603_1608Metric, F.Cu at (98.4, 153.2)
- added C14: 1uF, Capacitor_SMD:C_0805_2012Metric, F.Cu at (98.2, 155.1)
- added C15: 10nF, Capacitor_SMD:C_0603_1608Metric, F.Cu at (96.7, 148.8)
- added C16: 0.1uF, Capacitor_SMD:C_0603_1608Metric, F.Cu at (118.9, 149.8)
- added C17: 1uF, Capacitor_SMD:C_0805_2012Metric, F.Cu at (119.4, 151.6)
- added C18: 10nF, Capacitor_SMD:C_0603_1608Metric, F.Cu at (115.6, 146.3)
- added C19: 0.1uF, Capacitor_SMD:C_0603_1608Metric, F.Cu at (136.5, 138.8)
- added C2: 1uF, Capacitor_SMD:C_0805_2012Metric, F.Cu at (8.52, 96.8)
- added C2: 1uF, Capacitor_SMD:C_0805_2012Metric, F.Cu at (44.9, 98.2)
- added C20: 1uF, Capacitor_SMD:C_0805_2012Metric, F.Cu at (137.7, 140.2)
- added C21: 10nF, Capacitor_SMD:C_0603_1608Metric, F.Cu at (132.2, 136.8)
- added C22: 0.1uF, Capacitor_SMD:C_0603_1608Metric, F.Cu at (148.5, 121.8)
- added C23: 1uF, Capacitor_SMD:C_0805_2012Metric, F.Cu at (150.2, 122.7)
- added C24: 10nF, Capacitor_SMD:C_0603_1608Metric, F.Cu at (143.8, 121.7)
- added C25: 0.1uF, Capacitor_SMD:C_0603_1608Metric, F.Cu at (153.2, 101.6)
- added C26: 1uF, Capacitor_SMD:C_0805_2012Metric, F.Cu at (155.1, 101.8)
- added C27: 10nF, Capacitor_SMD:C_0603_1608Metric, F.Cu at (148.8, 103.3)
- added C28: 0.1uF, Capacitor_SMD:C_0603_1608Metric, F.Cu at (149.8, 81.1)
- added C29: 1uF, Capacitor_SMD:C_0805_2012Metric, F.Cu at (151.6, 80.6)
- added C3: 10nF, Capacitor_SMD:C_0603_1608Metric, F.Cu at (16.3, 94.9)
- added C3: 10nF, Capacitor_SMD:C_0603_1608Metric, F.Cu at (51.2, 96.7)
- added C30: 10nF, Capacitor_SMD:C_0603_1608Metric, F.Cu at (146.3, 84.4)
- added C31: 0.1uF, Capacitor_SMD:C_0603_1608Metric, F.Cu at (138.8, 63.5)
- added C32: 1uF, Capacitor_SMD:C_0805_2012Metric, F.Cu at (140.2, 62.3)
- added C33: 10nF, Capacitor_SMD:C_0603_1608Metric, F.Cu at (136.8, 67.8)
- added C34: 0.1uF, Capacitor_SMD:C_0603_1608Metric, F.Cu at (121.8, 51.5)
- added C35: 1uF, Capacitor_SMD:C_0805_2012Metric, F.Cu at (122.7, 49.8)
- added C36: 10nF, Capacitor_SMD:C_0603_1608Metric, F.Cu at (121.7, 56.2)
- added C37: 0.1uF, Capacitor_SMD:C_0603_1608Metric, F.Cu at (101.6, 46.8)
- added C38: 1uF, Capacitor_SMD:C_0805_2012Metric, F.Cu at (101.8, 44.9)
- added C39: 10nF, Capacitor_SMD:C_0603_1608Metric, F.Cu at (103.3, 51.2)
- added C4: 0.1uF, Capacitor_SMD:C_0603_1608Metric, F.Cu at (50.2, 118.9)
- added C40: 0.1uF, Capacitor_SMD:C_0603_1608Metric, F.Cu at (81.1, 50.2)
- added C41: 1uF, Capacitor_SMD:C_0805_2012Metric, F.Cu at (80.6, 48.4)
- added C42: 10nF, Capacitor_SMD:C_0603_1608Metric, F.Cu at (84.4, 53.7)
- added C43: 0.1uF, Capacitor_SMD:C_0603_1608Metric, F.Cu at (63.5, 61.2)
- added C44: 1uF, Capacitor_SMD:C_0805_2012Metric, F.Cu at (62.3, 59.8)
- added C45: 10nF, Capacitor_SMD:C_0603_1608Metric, F.Cu at (67.8, 63.2)
- added C46: 0.1uF, Capacitor_SMD:C_0603_1608Metric, F.Cu at (51.5, 78.2)
- added C47: 1uF, Capacitor_SMD:C_0805_2012Metric, F.Cu at (49.8, 77.3)
- added C48: 10nF, Capacitor_SMD:C_0603_1608Metric, F.Cu at (56.2, 78.3)
- added C5: 1uF, Capacitor_SMD:C_0805_2012Metric, F.Cu at (48.4, 119.4)
- added C6: 10nF, Capacitor_SMD:C_0603_1608Metric, F.Cu at (53.7, 115.6)
- added C7: 0.1uF, Capacitor_SMD:C_0603_1608Metric, F.Cu at (61.2, 136.5)
- added C8: 1uF, Capacitor_SMD:C_0805_2012Metric, F.Cu at (59.8, 137.7)
- added C9: 10nF, Capacitor_SMD:C_0603_1608Metric, F.Cu at (63.2, 132.2)
- added D1: LED, Library:GWJTLRS1EMLVL5XX531, F.Cu at (55.1, 100.0)
- added D1: LED, Library:GWJTLRS1EMLVL5XX531, F.Cu at (24.8, 96.5)
- added D10: LED, Library:GWJTLRS1EMLVL5XX531, F.Cu at (141.4, 82.8)
- added D11: LED, Library:GWJTLRS1EMLVL5XX531, F.Cu at (131.7, 68.2)
- added D12: LED, Library:GWJTLRS1EMLVL5XX531, F.Cu at (117.1, 58.5)
- added D13: LED, Library:GWJTLRS1EMLVL5XX531, F.Cu at (100.0, 55.1)
- added D14: LED, Library:GWJTLRS1EMLVL5XX531, F.Cu at (82.8, 58.6)
- added D15: LED, Library:GWJTLRS1EMLVL5XX531, F.Cu at (68.2, 68.3)
- added D16: LED, Library:GWJTLRS1EMLVL5XX531, F.Cu at (58.5, 82.9)
- added D2: LED, Library:GWJTLRS1EMLVL5XX531, F.Cu at (58.6, 117.2)
- added D3: LED, Library:GWJTLRS1EMLVL5XX531, F.Cu at (68.3, 131.8)
- added D4: LED, Library:GWJTLRS1EMLVL5XX531, F.Cu at (82.9, 141.5)
- added D5: LED, Library:GWJTLRS1EMLVL5XX531, F.Cu at (100.0, 144.9)
- added D6: LED, Library:GWJTLRS1EMLVL5XX531, F.Cu at (117.2, 141.4)
- added D7: LED, Library:GWJTLRS1EMLVL5XX531, F.Cu at (131.8, 131.7)
- added D8: LED, Library:GWJTLRS1EMLVL5XX531, F.Cu at (141.5, 117.1)
- added D9: LED, Library:GWJTLRS1EMLVL5XX531, F.Cu at (144.9, 100.0)
- added Q1: MMBT3904, Library:SOT95P240X120-3N, F.Cu at (19.5, 98.8)
- added Q1: MMBT3904, Library:SOT95P240X120-3N, F.Cu at (60.4, 100.7)
- added Q10: MMBT3904, Library:SOT95P240X120-3N, F.Cu at (136.4, 84.2)
- added Q11: MMBT3904, Library:SOT95P240X120-3N, F.Cu at (127.6, 71.5)
- added Q12: MMBT3904, Library:SOT95P240X120-3N, F.Cu at (114.6, 63.1)
- added Q13: MMBT3904, Library:SOT95P240X120-3N, F.Cu at (99.3, 60.4)
- added Q14: MMBT3904, Library:SOT95P240X120-3N, F.Cu at (84.2, 63.6)
- added Q15: MMBT3904, Library:SOT95P240X120-3N, F.Cu at (71.5, 72.4)
- added Q16: MMBT3904, Library:SOT95P240X120-3N, F.Cu at (63.1, 85.4)
- added Q2: MMBT3904, Library:SOT95P240X120-3N, F.Cu at (63.6, 115.8)
- added Q3: MMBT3904, Library:SOT95P240X120-3N, F.Cu at (72.4, 128.5)
- added Q4: MMBT3904, Library:SOT95P240X120-3N, F.Cu at (85.4, 136.9)
- added Q5: MMBT3904, Library:SOT95P240X120-3N, F.Cu at (100.7, 139.6)
- added Q6: MMBT3904, Library:SOT95P240X120-3N, F.Cu at (115.8, 136.4)
- added Q7: MMBT3904, Library:SOT95P240X120-3N, F.Cu at (128.5, 127.6)
- added Q8: MMBT3904, Library:SOT95P240X120-3N, F.Cu at (136.9, 114.6)
- added Q9: MMBT3904, Library:SOT95P240X120-3N, F.Cu at (139.6, 99.3)
- added R1: 102, Resistor_SMD:R_1210_3225Metric, F.Cu at (54.5, 95.8)
- added R1: 102, Resistor_SMD:R_1210_3225Metric, F.Cu at (19.5, 95.2)
- added R10: 102, Resistor_SMD:R_1210_3225Metric, F.Cu at (78.7, 140.4)
- added R11: 0.1, Resistor_SMD:R_0805_2012Metric, F.Cu at (80.2, 150.6)
- added R12: 270, Resistor_SMD:R_0603_1608Metric, F.Cu at (88.1, 137.5)
- added R13: 102, Resistor_SMD:R_1210_3225Metric, F.Cu at (95.8, 145.5)
- added R14: 0.1, Resistor_SMD:R_0805_2012Metric, F.Cu at (101.0, 154.4)
- added R15: 270, Resistor_SMD:R_0603_1608Metric, F.Cu at (103.4, 139.2)
- added R16: 102, Resistor_SMD:R_1210_3225Metric, F.Cu at (113.5, 143.6)
- added R17: 0.1, Resistor_SMD:R_0805_2012Metric, F.Cu at (121.8, 149.8)
- added R18: 270, Resistor_SMD:R_0603_1608Metric, F.Cu at (118.1, 134.9)
- added R19: 102, Resistor_SMD:R_1210_3225Metric, F.Cu at (129.2, 135.1)
- added R2: 0.1, Resistor_SMD:R_0805_2012Metric, F.Cu at (9.22, 99.7)
- added R2: 0.1, Resistor_SMD:R_0805_2012Metric, F.Cu at (45.6, 101.0)
- added R20: 0.1, Resistor_SMD:R_0805_2012Metric, F.Cu at (139.2, 137.7)
- added R21: 270, Resistor_SMD:R_0603_1608Metric, F.Cu at (130.1, 125.3)
- added R22: 102, Resistor_SMD:R_1210_3225Metric, F.Cu at (140.4, 121.3)
- added R23: 0.1, Resistor_SMD:R_0805_2012Metric, F.Cu at (150.6, 119.8)
- added R24: 270, Resistor_SMD:R_0603_1608Metric, F.Cu at (137.5, 111.9)
- added R25: 102, Resistor_SMD:R_1210_3225Metric, F.Cu at (145.5, 104.2)
- added R26: 0.1, Resistor_SMD:R_0805_2012Metric, F.Cu at (154.4, 99.0)
- added R27: 270, Resistor_SMD:R_0603_1608Metric, F.Cu at (139.2, 96.6)
- added R28: 102, Resistor_SMD:R_1210_3225Metric, F.Cu at (143.6, 86.5)
- added R29: 0.1, Resistor_SMD:R_0805_2012Metric, F.Cu at (149.8, 78.2)
- added R3: 270, Resistor_SMD:R_0603_1608Metric, F.Cu at (16.3, 98.5)
- added R3: 270, Resistor_SMD:R_0603_1608Metric, F.Cu at (60.8, 103.4)
- added R30: 270, Resistor_SMD:R_0603_1608Metric, F.Cu at (134.9, 81.9)
- added R31: 102, Resistor_SMD:R_1210_3225Metric, F.Cu at (135.1, 70.8)
- added R32: 0.1, Resistor_SMD:R_0805_2012Metric, F.Cu at (137.7, 60.8)
- added R33: 270, Resistor_SMD:R_0603_1608Metric, F.Cu at (125.3, 69.9)
- added R34: 102, Resistor_SMD:R_1210_3225Metric, F.Cu at (121.3, 59.6)
- added R35: 0.1, Resistor_SMD:R_0805_2012Metric, F.Cu at (119.8, 49.4)
- added R36: 270, Resistor_SMD:R_0603_1608Metric, F.Cu at (111.9, 62.5)
- added R37: 102, Resistor_SMD:R_1210_3225Metric, F.Cu at (104.2, 54.5)
- added R38: 0.1, Resistor_SMD:R_0805_2012Metric, F.Cu at (99.0, 45.6)
- added R39: 270, Resistor_SMD:R_0603_1608Metric, F.Cu at (96.6, 60.8)
- added R4: 102, Resistor_SMD:R_1210_3225Metric, F.Cu at (56.4, 113.5)
- added R40: 102, Resistor_SMD:R_1210_3225Metric, F.Cu at (86.5, 56.4)
- added R41: 0.1, Resistor_SMD:R_0805_2012Metric, F.Cu at (78.2, 50.2)
- added R42: 270, Resistor_SMD:R_0603_1608Metric, F.Cu at (81.9, 65.1)
- added R43: 102, Resistor_SMD:R_1210_3225Metric, F.Cu at (70.8, 64.9)
- added R44: 0.1, Resistor_SMD:R_0805_2012Metric, F.Cu at (60.8, 62.3)
- added R45: 270, Resistor_SMD:R_0603_1608Metric, F.Cu at (69.9, 74.7)
- added R46: 102, Resistor_SMD:R_1210_3225Metric, F.Cu at (59.6, 78.7)
- added R47: 0.1, Resistor_SMD:R_0805_2012Metric, F.Cu at (49.4, 80.2)
- added R48: 270, Resistor_SMD:R_0603_1608Metric, F.Cu at (62.5, 88.1)
- added R5: 0.1, Resistor_SMD:R_0805_2012Metric, F.Cu at (50.2, 121.8)
- added R6: 270, Resistor_SMD:R_0603_1608Metric, F.Cu at (65.1, 118.1)
- added R7: 102, Resistor_SMD:R_1210_3225Metric, F.Cu at (64.9, 129.2)
- added R8: 0.1, Resistor_SMD:R_0805_2012Metric, F.Cu at (62.3, 139.2)
- added R9: 270, Resistor_SMD:R_0603_1608Metric, F.Cu at (74.7, 130.1)
- added REF**: QFN-16-1EP_4x4mm_P0.5mm_EP2.45x2.45mm, Package_DFN_QFN:QFN-16-1EP_4x4mm_P0.5mm_EP2.45x2.45mm, F.Cu at (37.4, 100.0)
- added U1: TPS92612QDBVRQ1, Library:SOT95P280X145-5N, F.Cu at (13.4, 96.8)
- added U1: TPS92612QDBVRQ1, Library:SOT95P280X145-5N, F.Cu at (49.9, 100.1)
- added U10: TPS92612QDBVRQ1, Library:SOT95P280X145-5N, F.Cu at (146.3, 80.7)
- added U11: TPS92612QDBVRQ1, Library:SOT95P280X145-5N, F.Cu at (135.4, 64.5)
- added U12: TPS92612QDBVRQ1, Library:SOT95P280X145-5N, F.Cu at (119.1, 53.6)
- added U13: TPS92612QDBVRQ1, Library:SOT95P280X145-5N, F.Cu at (99.9, 49.9)
- added U14: TPS92612QDBVRQ1, Library:SOT95P280X145-5N, F.Cu at (80.7, 53.7)
- added U15: TPS92612QDBVRQ1, Library:SOT95P280X145-5N, F.Cu at (64.5, 64.6)
- added U16: TPS92612QDBVRQ1, Library:SOT95P280X145-5N, F.Cu at (53.6, 80.9)
- added U2: TPS92612QDBVRQ1, Library:SOT95P280X145-5N, F.Cu at (53.7, 119.3)
- added U3: TPS92612QDBVRQ1, Library:SOT95P280X145-5N, F.Cu at (64.6, 135.5)
- added U4: TPS92612QDBVRQ1, Library:SOT95P280X145-5N, F.Cu at (80.9, 146.4)
- added U5: TPS92612QDBVRQ1, Library:SOT95P280X145-5N, F.Cu at (100.1, 150.1)
- added U6: TPS92612QDBVRQ1, Library:SOT95P280X145-5N, F.Cu at (119.3, 146.3)
- added U7: TPS92612QDBVRQ1, Library:SOT95P280X145-5N, F.Cu at (135.5, 135.4)
- added U8: TPS92612QDBVRQ1, Library:SOT95P280X145-5N, F.Cu at (146.4, 119.1)
- added U9: TPS92612QDBVRQ1, Library:SOT95P280X145-5N, F.Cu at (150.1, 99.9)
Other:
- board size 122 x 122 mm -> 132 x 132 mm

Commit message: m
Parts:
- removed the C1 at (10.4, 97.0)
- removed the C1 at (46.8, 98.4)
- removed C10, C13, C16, C19, C22, C25, C28, C31, C34, C37, C4, C40, C43, C46, C7: 0.1uF, Capacitor_SMD:C_0603_1608Metric
- removed C11, C14, C17, C20, C23, C26, C29, C32, C35, C38, C41, C44, C47, C5, C8: 1uF, Capacitor_SMD:C_0805_2012Metric
- removed C12, C15, C18, C21, C24, C27, C30, C33, C36, C39, C42, C45, C48, C6, C9: 10nF, Capacitor_SMD:C_0603_1608Metric
- removed the C2 at (8.52, 96.8)
- removed the C2 at (44.9, 98.2)
- removed the C3 at (16.3, 94.9)
- removed the C3 at (51.2, 96.7)
- removed the D1 at (55.1, 100.0)
- removed the D1 at (24.8, 96.5)
- removed D10, D11, D12, D13, D14, D15, D16, D3, D4, D5, D6, D7, D8, D9: LED, Library:GWJTLRS1EMLVL5XX531
- removed the Q1 at (19.5, 98.8)
- removed the Q1 at (60.4, 100.7)
- removed Q10, Q11, Q12, Q13, Q14, Q15, Q16, Q2, Q3, Q4, Q5, Q6, Q7, Q8, Q9: MMBT3904, Library:SOT95P240X120-3N
- removed the R1 at (54.5, 95.8)
- removed the R1 at (19.5, 95.2)
- removed R10, R13, R16, R19, R22, R25, R28, R31, R34, R37, R40, R43, R46, R7: 102, Resistor_SMD:R_1210_3225Metric
- removed R11, R14, R17, R20, R23, R26, R29, R32, R35, R38, R41, R44, R47, R8: 0.1, Resistor_SMD:R_0805_2012Metric
- removed R12, R15, R18, R21, R24, R27, R30, R33, R36, R39, R42, R45, R48, R6, R9: 270, Resistor_SMD:R_0603_1608Metric
- removed the R2 at (9.22, 99.7)
- removed the R2 at (45.6, 101.0)
- removed the R3 at (16.3, 98.5)
- removed the R3 at (60.8, 103.4)
- removed REF**: QFN-16-1EP_4x4mm_P0.5mm_EP2.45x2.45mm, Package_DFN_QFN:QFN-16-1EP_4x4mm_P0.5mm_EP2.45x2.45mm
- removed the U1 at (13.4, 96.8)
- removed the U1 at (49.9, 100.1)
- removed U10, U11, U12, U13, U14, U15, U16, U2, U3, U4, U5, U6, U7, U8, U9: TPS92612QDBVRQ1, Library:SOT95P280X145-5N
- added C1: 1uF, Capacitor_SMD:C_0805_2012Metric, F.Cu at (40.8, 103.1)
- added C2: 0.1uF, Capacitor_SMD:C_0603_1608Metric, F.Cu at (41.0, 105.0)
- added C3: 10nF, Capacitor_SMD:C_0402_1005Metric, F.Cu at (46.2, 98.8)
- added D1: LED, Library:GWJTLRS1EMLVL5XX531, F.Cu at (49.8, 100.0)
- added Q1: MMBT3904, Package_TO_SOT_SMD:SOT-416, F.Cu at (39.9, 99.4)
- added R1: 1, Resistor_SMD:R_0402_1005Metric, F.Cu at (46.2, 101.9)
- added R2: 80.6, Resistor_SMD:R_1210_3225Metric, F.Cu at (49.2, 105.7)
- added R3: 1k, Resistor_SMD:R_0402_1005Metric, F.Cu at (39.4, 101.3)
- added U1: TPS92612QDBVRQ1, Library:SOT95P280X145-5N, F.Cu at (43.4, 100.2)
- R4: value 102 -> 10k; footprint Resistor_SMD:R_1210_3225Metric -> Resistor_SMD:R_0402_1005Metric
- R5: value 0.1 -> 10k; footprint Resistor_SMD:R_0805_2012Metric -> Resistor_SMD:R_0402_1005Metric
- moved R5 25.5 mm to (42.2, 97.6), turned to 0 degrees
- moved R4 22.9 mm to (39.9, 97.6), turned to 0 degrees
- moved D2 17.3 mm to (57.0, 100.0), turned to 180 degrees
Connections:
- D2 pad 1: Net-(Q1-C) -> GND
- D2 pad 2: Net-(Q1-C) -> GND
- D2 pad 3: Net-(U1-OUT) -> /LED1
- D2 pad 4: Net-(U1-OUT) -> /LED1
- R4 pad 1: Net-(U1-IN) -> EN1
- R4 pad 2: Net-(U1-OUT) -> /B1
- R5 pad 1: +12V -> /B1
- R5 pad 2: Net-(U1-IN) -> GND
Routing:
- net /IN1: track 0.00 -> 3.89 mm
- net /PWM1: track 0.00 -> 3.56 mm
- net +12V: track 0.00 -> 3.15 mm, vias 0 -> 5
- net /OUT1: track 0.00 -> 2.54 mm
- net /B1: track 0.00 -> 2.43 mm
- added copper zone on F.Cu, net +12V
- added copper zone on F.Cu, net /IN1
- added copper zone on F.Cu, net /LED1
- added copper zone on F.Cu, net /OUT1
- added copper zone on B.Cu, net GND
- added copper zone on F.Cu, net GND
- added copper zone on In1.Cu, net GND
- added copper zone on In2.Cu, net GND
Other:
- copper layers 2 -> 4

Commit message: d
Routing:
- net +12V: track 3.15 -> 3.29 mm, vias 5 -> 0
- added copper zone on B.Cu, net /IN1
- added copper zone on In2.Cu, net /IN1
- added copper zone on B.Cu, net /LED1
- added copper zone on In2.Cu, net /LED1
- added copper zone on B.Cu, net /OUT1
- added copper zone on In2.Cu, net /OUT1
- removed copper zone on B.Cu, net GND
- removed copper zone on In1.Cu, net GND
- removed copper zone on In2.Cu, net GND
