File: Hardware/Ring-Light/Ring-Light.kicad_sch (KiCad schematic)
At the start: 2 parts, among them IC2 74HC125PW,112, U1 74HC595

Commit message: .
Parts:
- removed IC2: 74HC125PW,112, Library:SOP65P640X110-14N, symbol Library:74HC125PW,112
- added C14, C61, C63, C8: 0.1uF, symbol Device:C_Small
- added C15, C62, C64, C9: 1uF, symbol Device:C_Small
- added U2, U5, U6: 74HC595, symbol 74xx:74HC595
Connections:
- net SEG_9-16/EN10: now reaches U1.1 (QB)
- net ~{CLR}: now reaches U1.10 (~{SRCLR})
- net ~{CLR}: now also U2.10 (~{SRCLR}), U5.10 (~{SRCLR}), U6.10 (~{SRCLR})
- net SCLK: now reaches U1.11 (SRCLK)
- net SCLK: now also U2.11 (SRCLK), U5.11 (SRCLK), U6.11 (SRCLK)
- net RCLK: now reaches U1.12 (RCLK)
- net RCLK: now also U2.12 (RCLK), U5.12 (RCLK), U6.12 (RCLK)
- net ~{OE}: now reaches U1.13 (~{OE})
- net ~{OE}: now also U2.13 (~{OE}), U5.13 (~{OE}), U6.13 (~{OE})
- net at U1.14 (SER): now also U2.9 (QH')
- net SEG_9-16/EN9: now reaches U1.15 (QA)
- net +3.3V: now reaches U1.16 (VCC)
- net +3.3V: now also C14.1, C15.1, C61.1, C62.1, C63.1, C64.1, C8.1, C9.1, U2.16 (VCC), U5.16 (VCC), U6.16 (VCC)
- net SEG_9-16/EN11: now reaches U1.2 (QC)
- net SEG_9-16/EN12: now reaches U1.3 (QD)
- net SEG_9-16/EN13: now reaches U1.4 (QE)
- net SEG_9-16/EN14: now reaches U1.5 (QF)
- net SEG_9-16/EN15: now reaches U1.6 (QG)
- net SEG_9-16/EN16: now reaches U1.7 (QH)
- net GND: now reaches U1.8 (GND)
- net GND: now also C14.2, C15.2, C61.2, C62.2, C63.2, C64.2, C8.2, C9.2, U2.8 (GND), U5.8 (GND), U6.8 (GND)
- net at U1.9 (QH'): now also U5.14 (SER)
- new net: U5.9 (QH'), U6.14 (SER)
- new net DATA: U2.14 (SER)
- new net SEG_1-8/EN1: U2.15 (QA)
- new net SEG_1-8/EN2: U2.1 (QB)
- new net SEG_1-8/EN3: U2.2 (QC)
- new net SEG_1-8/EN4: U2.3 (QD)
- new net SEG_1-8/EN5: U2.4 (QE)
- new net SEG_1-8/EN6: U2.5 (QF)
- new net SEG_1-8/EN7: U2.6 (QG)
- new net SEG_1-8/EN8: U2.7 (QH)
- new net SEG_17-24/EN17: U5.15 (QA)
- new net SEG_17-24/EN18: U5.1 (QB)
- new net SEG_17-24/EN19: U5.2 (QC)
- new net SEG_17-24/EN20: U5.3 (QD)
- new net SEG_17-24/EN21: U5.4 (QE)
- new net SEG_17-24/EN22: U5.5 (QF)
- new net SEG_17-24/EN23: U5.6 (QG)
- new net SEG_17-24/EN24: U5.7 (QH)
- new net SEG_25-32/EN25: U6.15 (QA)
- new net SEG_25-32/EN26: U6.1 (QB)
- new net SEG_25-32/EN27: U6.2 (QC)
- new net SEG_25-32/EN28: U6.3 (QD)
- new net SEG_25-32/EN29: U6.4 (QE)
- new net SEG_25-32/EN30: U6.5 (QF)
- new net SEG_25-32/EN31: U6.6 (QG)
- new net SEG_25-32/EN32: U6.7 (QH)
Other:
- sheet SEG_1-4 renamed SEG_1-8
- removed sheet SEG5-8
- added sheet SEG_17-24 (SEG_17-24.kicad_sch)
- added sheet SEG_25-32 (SEG_25-32.kicad_sch)
- added sheet SEG_9-16 (SEG_9-16.kicad_sch)
- sheet SEG_1-8: file SEG_1-4.kicad_sch -> SEG_1-8.kicad_sch
- sheet SEG_1-8 ports: added EN1, EN2, EN3, EN4, EN5, EN6, EN7, EN8, PWM; removed PWM1, PWM2, PWM3, PWM4
- moved on the sheet: U1

Commit message: m
Parts:
- removed C14, C61, C63, C8: 0.1uF, symbol Device:C_Small
- removed C15, C62, C64, C9: 1uF, symbol Device:C_Small
- removed U1, U5, U6: 74HC595, symbol 74xx:74HC595
- added C1: 0.1uF, Capacitor_SMD:C_0603_1608Metric, symbol Device:C_Small
- added C2: 1uF, Capacitor_SMD:C_0805_2012Metric, symbol Device:C_Small
- added C3: 10nF, Capacitor_SMD:C_0603_1608Metric, symbol Device:C_Small
- added D1: LED, Library:GWJTLRS1EMLVL5XX531, symbol Library:LED
- added Q1: MMBT3904, Library:SOT95P240X120-3N, symbol Library:MMBT3904
- added R1: 102, Resistor_SMD:R_1210_3225Metric, symbol Device:R_Small
- added R2: 0.1, Resistor_SMD:R_0805_2012Metric, symbol Device:R_Small
- added R3: 270, Resistor_SMD:R_0603_1608Metric, symbol Device:R_Small
- added U1: TPS92612QDBVRQ1, Library:SOT95P280X145-5N, symbol Library:TPS92612QDBVRQ1
Connections:
- net GND: now also C1.2, C2.2, C3.2, Q1.2 (E), U1.1 (GND); no longer U2.8 (GND)
- net PWM: now also R3.1, U1.2 (PWM)
- net +3.3V: no longer names the net of U2.16 (VCC)
- net DATA: no longer names the net of U2.14 (SER)
- net RCLK: no longer names the net of U2.12 (RCLK)
- net SCLK: no longer names the net of U2.11 (SRCLK)
- net SEG_1-8/EN1: no longer names the net of U2.15 (QA)
- net SEG_1-8/EN2: no longer names the net of U2.1 (QB)
- net SEG_1-8/EN3: no longer names the net of U2.2 (QC)
- net SEG_1-8/EN4: no longer names the net of U2.3 (QD)
- net SEG_1-8/EN5: no longer names the net of U2.4 (QE)
- net SEG_1-8/EN6: no longer names the net of U2.5 (QF)
- net SEG_1-8/EN7: no longer names the net of U2.6 (QG)
- net SEG_1-8/EN8: no longer names the net of U2.7 (QH)
- net ~{CLR}: no longer names the net of U2.10 (~{SRCLR})
- net ~{OE}: no longer names the net of U2.13 (~{OE})
- new net: Q1.1 (B), R3.2
- new net: C3.1, D1.3 (A), D1.4 (A), R1.2, U1.5 (OUT)
- new net: R1.1, R2.2, U1.4 (IN)
- new net: D1.1 (K), D1.2 (K), Q1.3 (C)
- new net +12V: C1.1, C2.1, R2.1, U1.3 (SUPPLY)
Other:
- removed sheet SEG_1-8
- removed sheet SEG_17-24
- removed sheet SEG_25-32
- removed sheet SEG_9-16

Commit message: m
Parts:
- removed Q1: MMBT3904, Library:SOT95P240X120-3N, symbol Library:MMBT3904
- removed U2: 74HC595, symbol 74xx:74HC595
- added C4: 1uF, Capacitor_SMD:C_0805_2012Metric, symbol Device:C_Small
- added C5: 0.1uF, Capacitor_SMD:C_0603_1608Metric, symbol Device:C_Small
- added C6: 10nF, Capacitor_SMD:C_0402_1005Metric, symbol Device:C_Small
- added D2, D3, D4: LED, Library:GWJTLRS1EMLVL5XX531, symbol Library:LED
- added Q1, Q2: MMBT3904, Package_TO_SOT_SMD:SOT-416, symbol Library:MMBT39042-2
- added R10, R5, R9: 10k, Resistor_SMD:R_0402_1005Metric, symbol Device:R_Small
- added R3, R8: 1k, Resistor_SMD:R_0402_1005Metric, symbol Device:R_Small
- added R6: 1, Resistor_SMD:R_0402_1005Metric, symbol Device:R_Small
- added R7: 80.6, Resistor_SMD:R_1210_3225Metric, symbol Device:R_Small
- added U2: TPS92612QDBVRQ1, Library:SOT95P280X145-5N, symbol Library:TPS92612QDBVRQ1
- C3: footprint Capacitor_SMD:C_0603_1608Metric -> Capacitor_SMD:C_0402_1005Metric
- R1: renamed from R2; value 0.1 -> 1; footprint Resistor_SMD:R_0805_2012Metric -> Resistor_SMD:R_0402_1005Metric
- R2: renamed from R1; value 102 -> 80.6
- R4: renamed from R3; value 270 -> 10k; footprint Resistor_SMD:R_0603_1608Metric -> Resistor_SMD:R_0402_1005Metric
- renumbered C2 to C1, C1 to C2
Connections:
- net +12V: now also C4.1, C5.1, R6.1, U2.3 (SUPPLY)
- net GND: now also C4.2, C5.2, C6.2, D2.1 (K), D2.2 (K), D4.1 (K), D4.2 (K), Q1.2 (E), Q2.2 (E), R10.2, R5.2, U2.1 (GND)
- net PWM: now also R3.1, R8.1; no longer R4.1, U1.2 (PWM)
- net B1: now reaches R4.2
- net B1: now also Q1.1 (B), R5.1
- net OUT1: now reaches C3.1, D1.3 (A), D1.4 (A), R2.2, U1.5 (OUT)
- net IN1: now reaches R1.2, R2.1, U1.4 (IN)
- net LED1: now reaches D1.1 (K), D1.2 (K)
- net LED1: now also D2.3 (A), D2.4 (A)
- new net B2: Q2.1 (B), R10.1, R9.2
- new net EN1: R4.1, R9.1
- new net IN2: R6.2, R7.1, U2.4 (IN)
- new net LED2: D3.1 (K), D3.2 (K), D4.3 (A), D4.4 (A)
- new net OUT2: C6.1, D3.3 (A), D3.4 (A), R7.2, U2.5 (OUT)
- new net PWM1: Q1.3 (C), R3.2, U1.2 (PWM)
- new net PWM2: Q2.3 (C), R8.2, U2.2 (PWM)
Other:
- moved on the sheet: C1, C2, C3, D1, R1, R2, R4, U1

Commit message: d
Parts:
- added C10, C13, C16, C19, C22, C25, C28, C31, C34, C37, C40, C43, C46, C49, C52, C55, C58, C61, C64, C67, C7, C70: 1uF, Capacitor_SMD:C_0805_2012Metric, symbol Device:C_Small
- added C11, C14, C17, C20, C23, C26, C29, C32, C35, C38, C41, C44, C47, C50, C53, C56, C59, C62, C65, C68, C71, C8: 0.1uF, Capacitor_SMD:C_0603_1608Metric, symbol Device:C_Small
- added C12, C15, C18, C21, C24, C27, C30, C33, C36, C39, C42, C45, C48, C51, C54, C57, C60, C63, C66, C69, C72, C9: 10nF, Capacitor_SMD:C_0402_1005Metric, symbol Device:C_Small
- added D10, D11, D12, D13, D14, D15, D16, D17, D18, D19, D20, D21, D22, D23, D24, D25, D26, D27, D28, D29, D30, D31, D32, D33, D34, D35, D36, D37, D38, D39, D40, D41, D42, D43, D44, D45, D46, D47, D48, D5, D6, D7, D8, D9: LED, Library:GWJTLRS1EMLVL5XX531, symbol Library:LED
- added Q10, Q11, Q12, Q13, Q14, Q15, Q16, Q17, Q18, Q19, Q20, Q21, Q22, Q23, Q24, Q3, Q4, Q5, Q6, Q7, Q8, Q9: MMBT3904, Package_TO_SOT_SMD:SOT-416, symbol Library:MMBT39042-2
- added R100, R104, R105, R109, R110, R114, R115, R119, R120, R14, R15, R19, R20, R24, R25, R29, R30, R34, R35, R39, R40, R44, R45, R49, R50, R54, R55, R59, R60, R64, R65, R69, R70, R74, R75, R79, R80, R84, R85, R89, R90, R94, R95, R99: 10k, Resistor_SMD:R_0402_1005Metric, symbol Device:R_Small
- added R101, R106, R11, R111, R116, R16, R21, R26, R31, R36, R41, R46, R51, R56, R61, R66, R71, R76, R81, R86, R91, R96: 1, Resistor_SMD:R_0402_1005Metric, symbol Device:R_Small
- added R102, R107, R112, R117, R12, R17, R22, R27, R32, R37, R42, R47, R52, R57, R62, R67, R72, R77, R82, R87, R92, R97: 80.6, Resistor_SMD:R_1210_3225Metric, symbol Device:R_Small
- added R103, R108, R113, R118, R13, R18, R23, R28, R33, R38, R43, R48, R53, R58, R63, R68, R73, R78, R83, R88, R93, R98: 1k, Resistor_SMD:R_0402_1005Metric, symbol Device:R_Small
- added U10, U11, U12, U13, U14, U15, U16, U17, U18, U19, U20, U21, U22, U23, U24, U3, U4, U5, U6, U7, U8, U9: TPS92612QDBVRQ1, Library:SOT95P280X145-5N, symbol Library:TPS92612QDBVRQ1
Connections:
- net +12V: now also C10.1, C11.1, C13.1, C14.1, C16.1, C17.1, C19.1, C20.1, C22.1, C23.1, C25.1, C26.1, C28.1, C29.1, C31.1, C32.1, C34.1, C35.1, C37.1, C38.1, C40.1, C41.1, C43.1, C44.1, C46.1, C47.1, C49.1, C50.1, C52.1, C53.1, C55.1, C56.1, C58.1, C59.1, C61.1, C62.1, C64.1, C65.1, C67.1, C68.1, C7.1, C70.1, C71.1, C8.1, R101.1, R106.1, R11.1, R111.1, R116.1, R16.1, R21.1, R26.1, R31.1, R36.1, R41.1, R46.1, R51.1, R56.1, R61.1, R66.1, R71.1, R76.1, R81.1, R86.1, R91.1, R96.1, U10.3 (SUPPLY), U11.3 (SUPPLY), U12.3 (SUPPLY), U13.3 (SUPPLY), U14.3 (SUPPLY), U15.3 (SUPPLY), U16.3 (SUPPLY), U17.3 (SUPPLY), U18.3 (SUPPLY), U19.3 (SUPPLY), U20.3 (SUPPLY), U21.3 (SUPPLY), U22.3 (SUPPLY), U23.3 (SUPPLY), U24.3 (SUPPLY), U3.3 (SUPPLY), U4.3 (SUPPLY), U5.3 (SUPPLY), U6.3 (SUPPLY), U7.3 (SUPPLY), U8.3 (SUPPLY), U9.3 (SUPPLY)
- net EN1: now also R104.1, R109.1, R114.1, R119.1, R14.1, R19.1, R24.1, R29.1, R34.1, R39.1, R44.1, R49.1, R54.1, R59.1, R64.1, R69.1, R74.1, R79.1, R84.1, R89.1, R94.1, R99.1
- net GND: now also C10.2, C11.2, C12.2, C13.2, C14.2, C15.2, C16.2, C17.2, C18.2, C19.2, C20.2, C21.2, C22.2, C23.2, C24.2, C25.2, C26.2, C27.2, C28.2, C29.2, C30.2, C31.2, C32.2, C33.2, C34.2, C35.2, C36.2, C37.2, C38.2, C39.2, C40.2, C41.2, C42.2, C43.2, C44.2, C45.2, C46.2, C47.2, C48.2, C49.2, C50.2, C51.2, C52.2, C53.2, C54.2, C55.2, C56.2, C57.2, C58.2, C59.2, C60.2, C61.2, C62.2, C63.2, C64.2, C65.2, C66.2, C67.2, C68.2, C69.2, C7.2, C70.2, C71.2, C72.2, C8.2, C9.2, D10.1 (K), D10.2 (K), D12.1 (K), D12.2 (K), D14.1 (K), D14.2 (K), D16.1 (K), D16.2 (K), D18.1 (K), D18.2 (K), D20.1 (K), D20.2 (K), D22.1 (K), D22.2 (K), D24.1 (K), D24.2 (K), D26.1 (K), D26.2 (K), D28.1 (K), D28.2 (K), D30.1 (K), D30.2 (K), D32.1 (K), D32.2 (K), D34.1 (K), D34.2 (K), D36.1 (K), D36.2 (K), D38.1 (K), D38.2 (K), D40.1 (K), D40.2 (K), D42.1 (K), D42.2 (K), D44.1 (K), D44.2 (K), D46.1 (K), D46.2 (K), D48.1 (K), D48.2 (K), D6.1 (K), D6.2 (K), D8.1 (K), D8.2 (K), Q10.2 (E), Q11.2 (E), Q12.2 (E), Q13.2 (E), Q14.2 (E), Q15.2 (E), Q16.2 (E), Q17.2 (E), Q18.2 (E), Q19.2 (E), Q20.2 (E), Q21.2 (E), Q22.2 (E), Q23.2 (E), Q24.2 (E), Q3.2 (E), Q4.2 (E), Q5.2 (E), Q6.2 (E), Q7.2 (E), Q8.2 (E), Q9.2 (E), R100.2, R105.2, R110.2, R115.2, R120.2, R15.2, R20.2, R25.2, R30.2, R35.2, R40.2, R45.2, R50.2, R55.2, R60.2, R65.2, R70.2, R75.2, R80.2, R85.2, R90.2, R95.2, U10.1 (GND), U11.1 (GND), U12.1 (GND), U13.1 (GND), U14.1 (GND), U15.1 (GND), U16.1 (GND), U17.1 (GND), U18.1 (GND), U19.1 (GND), U20.1 (GND), U21.1 (GND), U22.1 (GND), U23.1 (GND), U24.1 (GND), U3.1 (GND), U4.1 (GND), U5.1 (GND), U6.1 (GND), U7.1 (GND), U8.1 (GND), U9.1 (GND)
- net LED1: now also D29.1 (K), D29.2 (K), D30.3 (A), D30.4 (A)
- net PWM: now also R103.1, R108.1, R113.1, R118.1, R13.1, R18.1, R23.1, R28.1, R33.1, R38.1, R43.1, R48.1, R53.1, R58.1, R63.1, R68.1, R73.1, R78.1, R83.1, R88.1, R93.1, R98.1
- new net B10: Q10.1 (B), R49.2, R50.1
- new net B11: Q11.1 (B), R54.2, R55.1
- new net B12: Q12.1 (B), R59.2, R60.1
- new net B13: Q13.1 (B), R64.2, R65.1
- new net B14: Q14.1 (B), R69.2, R70.1
- new net B15: Q15.1 (B), R74.2, R75.1
- new net B16: Q16.1 (B), R79.2, R80.1
- new net B17: Q17.1 (B), R84.2, R85.1
- new net B18: Q18.1 (B), R89.2, R90.1
- new net B19: Q19.1 (B), R94.2, R95.1
- new net B20: Q20.1 (B), R100.1, R99.2
- new net B21: Q21.1 (B), R104.2, R105.1
- new net B22: Q22.1 (B), R109.2, R110.1
- new net B23: Q23.1 (B), R114.2, R115.1
- new net B24: Q24.1 (B), R119.2, R120.1
- new net B3: Q3.1 (B), R14.2, R15.1
- new net B4: Q4.1 (B), R19.2, R20.1
- new net B5: Q5.1 (B), R24.2, R25.1
- new net B6: Q6.1 (B), R29.2, R30.1
- new net B7: Q7.1 (B), R34.2, R35.1
- new net B8: Q8.1 (B), R39.2, R40.1
- new net B9: Q9.1 (B), R44.2, R45.1
- new net IN10: R46.2, R47.1, U10.4 (IN)
- new net IN11: R51.2, R52.1, U11.4 (IN)
- new net IN12: R56.2, R57.1, U12.4 (IN)
- new net IN13: R61.2, R62.1, U13.4 (IN)
- new net IN14: R66.2, R67.1, U14.4 (IN)
- new net IN15: R71.2, R72.1, U15.4 (IN)
- new net IN16: R76.2, R77.1, U16.4 (IN)
- new net IN17: R81.2, R82.1, U17.4 (IN)
- new net IN18: R86.2, R87.1, U18.4 (IN)
- new net IN19: R91.2, R92.1, U19.4 (IN)
- new net IN20: R96.2, R97.1, U20.4 (IN)
- new net IN21: R101.2, R102.1, U21.4 (IN)
- new net IN22: R106.2, R107.1, U22.4 (IN)
- new net IN23: R111.2, R112.1, U23.4 (IN)
- new net IN24: R116.2, R117.1, U24.4 (IN)
- new net IN3: R11.2, R12.1, U3.4 (IN)
- new net IN4: R16.2, R17.1, U4.4 (IN)
- new net IN5: R21.2, R22.1, U5.4 (IN)
- new net IN6: R26.2, R27.1, U6.4 (IN)
- new net IN7: R31.2, R32.1, U7.4 (IN)
- new net IN8: R36.2, R37.1, U8.4 (IN)
- new net IN9: R41.2, R42.1, U9.4 (IN)
- new net LED10: D19.1 (K), D19.2 (K), D20.3 (A), D20.4 (A)
- new net LED11: D21.1 (K), D21.2 (K), D22.3 (A), D22.4 (A)
- new net LED12: D23.1 (K), D23.2 (K), D24.3 (A), D24.4 (A)
- new net LED13: D25.1 (K), D25.2 (K), D26.3 (A), D26.4 (A)
- new net LED14: D27.1 (K), D27.2 (K), D28.3 (A), D28.4 (A)
- new net LED16: D31.1 (K), D31.2 (K), D32.3 (A), D32.4 (A)
- new net LED17: D33.1 (K), D33.2 (K), D34.3 (A), D34.4 (A)
- new net LED18: D35.1 (K), D35.2 (K), D36.3 (A), D36.4 (A)
- new net LED19: D37.1 (K), D37.2 (K), D38.3 (A), D38.4 (A)
- new net LED20: D39.1 (K), D39.2 (K), D40.3 (A), D40.4 (A)
- new net LED21: D41.1 (K), D41.2 (K), D42.3 (A), D42.4 (A)
- new net LED22: D43.1 (K), D43.2 (K), D44.3 (A), D44.4 (A)
- new net LED23: D45.1 (K), D45.2 (K), D46.3 (A), D46.4 (A)
- new net LED24: D47.1 (K), D47.2 (K), D48.3 (A), D48.4 (A)
- new net LED3: D5.1 (K), D5.2 (K), D6.3 (A), D6.4 (A)
- new net LED4: D7.1 (K), D7.2 (K), D8.3 (A), D8.4 (A)
- new net LED5: D10.3 (A), D10.4 (A), D9.1 (K), D9.2 (K)
- new net LED6: D11.1 (K), D11.2 (K), D12.3 (A), D12.4 (A)
- new net LED7: D13.1 (K), D13.2 (K), D14.3 (A), D14.4 (A)
- new net LED8: D15.1 (K), D15.2 (K), D16.3 (A), D16.4 (A)
- new net LED9: D17.1 (K), D17.2 (K), D18.3 (A), D18.4 (A)
- new net OUT10: C30.1, D19.3 (A), D19.4 (A), R47.2, U10.5 (OUT)
- new net OUT11: C33.1, D21.3 (A), D21.4 (A), R52.2, U11.5 (OUT)
- new net OUT12: C36.1, D23.3 (A), D23.4 (A), R57.2, U12.5 (OUT)
- new net OUT13: C39.1, D25.3 (A), D25.4 (A), R62.2, U13.5 (OUT)
- new net OUT14: C42.1, D27.3 (A), D27.4 (A), R67.2, U14.5 (OUT)
- new net OUT15: C45.1, D29.3 (A), D29.4 (A), R72.2, U15.5 (OUT)
- new net OUT16: C48.1, D31.3 (A), D31.4 (A), R77.2, U16.5 (OUT)
- new net OUT17: C51.1, D33.3 (A), D33.4 (A), R82.2, U17.5 (OUT)
- new net OUT18: C54.1, D35.3 (A), D35.4 (A), R87.2, U18.5 (OUT)
- new net OUT19: C57.1, D37.3 (A), D37.4 (A), R92.2, U19.5 (OUT)
- new net OUT20: C60.1, D39.3 (A), D39.4 (A), R97.2, U20.5 (OUT)
- new net OUT21: C63.1, D41.3 (A), D41.4 (A), R102.2, U21.5 (OUT)
- new net OUT22: C66.1, D43.3 (A), D43.4 (A), R107.2, U22.5 (OUT)
- new net OUT23: C69.1, D45.3 (A), D45.4 (A), R112.2, U23.5 (OUT)
- new net OUT24: C72.1, D47.3 (A), D47.4 (A), R117.2, U24.5 (OUT)
- new net OUT3: C9.1, D5.3 (A), D5.4 (A), R12.2, U3.5 (OUT)
- new net OUT4: C12.1, D7.3 (A), D7.4 (A), R17.2, U4.5 (OUT)
- new net OUT5: C15.1, D9.3 (A), D9.4 (A), R22.2, U5.5 (OUT)
- new net OUT6: C18.1, D11.3 (A), D11.4 (A), R27.2, U6.5 (OUT)
- new net OUT7: C21.1, D13.3 (A), D13.4 (A), R32.2, U7.5 (OUT)
- new net OUT8: C24.1, D15.3 (A), D15.4 (A), R37.2, U8.5 (OUT)
- new net OUT9: C27.1, D17.3 (A), D17.4 (A), R42.2, U9.5 (OUT)
- new net PWM10: Q10.3 (C), R48.2, U10.2 (PWM)
- new net PWM11: Q11.3 (C), R53.2, U11.2 (PWM)
- new net PWM12: Q12.3 (C), R58.2, U12.2 (PWM)
- new net PWM13: Q13.3 (C), R63.2, U13.2 (PWM)
- new net PWM14: Q14.3 (C), R68.2, U14.2 (PWM)
- new net PWM15: Q15.3 (C), R73.2, U15.2 (PWM)
- new net PWM16: Q16.3 (C), R78.2, U16.2 (PWM)
- new net PWM17: Q17.3 (C), R83.2, U17.2 (PWM)
- new net PWM18: Q18.3 (C), R88.2, U18.2 (PWM)
- new net PWM19: Q19.3 (C), R93.2, U19.2 (PWM)
- new net PWM20: Q20.3 (C), R98.2, U20.2 (PWM)
- new net PWM21: Q21.3 (C), R103.2, U21.2 (PWM)
- new net PWM22: Q22.3 (C), R108.2, U22.2 (PWM)
- new net PWM23: Q23.3 (C), R113.2, U23.2 (PWM)
- new net PWM24: Q24.3 (C), R118.2, U24.2 (PWM)
- new net PWM3: Q3.3 (C), R13.2, U3.2 (PWM)
- new net PWM4: Q4.3 (C), R18.2, U4.2 (PWM)
- new net PWM5: Q5.3 (C), R23.2, U5.2 (PWM)
- new net PWM6: Q6.3 (C), R28.2, U6.2 (PWM)
- new net PWM7: Q7.3 (C), R33.2, U7.2 (PWM)
- new net PWM8: Q8.3 (C), R38.2, U8.2 (PWM)
- new net PWM9: Q9.3 (C), R43.2, U9.2 (PWM)
