File: Hardware/Ring-Light v4/Ring-Light.kicad_pcb (KiCad board)
At the start: 4 copper layers, 124 x 135 mm, 134 parts, among them U1 NCR321PASX, U10 NCR321PASX, U11 NCR321PASX, U12 NCR321PASX, U13 NCR321PASX, U14 NCR321PASX, U15 NCR321PASX, U16 NCR321PASX, U17 NCR321PASX, U18 NCR321PASX, U19 NCR321PASX, U2 NCR321PASX, U20 NCR321PASX, U21 NCR321PASX, U22 NCR321PASX, U23 NCR321PASX, U24 NCR321PASX, U25 NCR321PASX, U26 NCR321PASX, U27 NCR321PASX, U28 NCR321PASX, U29 PCA9685BS,118, U3 NCR321PASX, U30 NCR321PASX, U31 NCR321PASX, U32 NCR321PASX, U33 NCR321PASX, U4 NCR321PASX, U5 NCR321PASX, U6 NCR321PASX, U7 NCR321PASX, U8 NCR321PASX, U9 NCR321PASX

Commit message: m
Parts:
- removed C1: 1uF, Capacitor_SMD:C_0805_2012Metric
- removed C2, C73: 0.1uF, Capacitor_SMD:C_0603_1608Metric
- removed D33, D34, D35, D36, D37, D38, D39, D40, D41, D42, D43, D44, D45, D46, D47, D48, D49, D50, D51, D52, D53, D54, D55, D56, D57, D58, D59, D60, D61, D62, D63, D64, D65, D66, D67, D68, D69, D70, D71, D72, D73, D74, D75, D76, D77, D78, D79, D80, D81, D82, D83, D84, D85, D86, D87, D88, D89, D90, D91, D92, D93, D94, D95, D96: LED, Library:GWJTLRS1EMLVL5XX531
- added C33: 0.1uF, Capacitor_SMD:C_0603_1608Metric, F.Cu at (34.0, 46.4)
- added C34: 0.1uF, Capacitor_SMD:C_0603_1608Metric, F.Cu at (34.0, 48.9)
- added R1: 100k, Resistor_SMD:R_0402_1005Metric, F.Cu at (123.2, 47.8)
- added R10: 9.09, Resistor_SMD:R_0402_1005Metric, F.Cu at (80.9, 65.3)
- added R11: 100k, Resistor_SMD:R_0402_1005Metric, F.Cu at (78.4, 68.3)
- added R12: 9.09, Resistor_SMD:R_0402_1005Metric, F.Cu at (74.9, 73.6)
- added R13: 100k, Resistor_SMD:R_0402_1005Metric, F.Cu at (73.0, 77.1)
- added R14: 9.09, Resistor_SMD:R_0402_1005Metric, F.Cu at (70.6, 82.9)
- added R15: 100k, Resistor_SMD:R_0402_1005Metric, F.Cu at (69.4, 86.7)
- added R16: 9.09, Resistor_SMD:R_0402_1005Metric, F.Cu at (68.2, 92.9)
- added R17: 100k, Resistor_SMD:R_0402_1005Metric, F.Cu at (67.8, 96.8)
- added R18: 9.09, Resistor_SMD:R_0402_1005Metric, F.Cu at (67.8, 103.1)
- added R19: 100k, Resistor_SMD:R_0402_1005Metric, F.Cu at (68.2, 107.0)
- added R20: 9.09, Resistor_SMD:R_0402_1005Metric, F.Cu at (69.4, 113.2)
- added R21: 100k, Resistor_SMD:R_0402_1005Metric, F.Cu at (70.5, 117.0)
- added R22: 9.09, Resistor_SMD:R_0402_1005Metric, F.Cu at (72.9, 122.9)
- added R23: 100k, Resistor_SMD:R_0402_1005Metric, F.Cu at (74.8, 126.3)
- added R24: 9.09, Resistor_SMD:R_0402_1005Metric, F.Cu at (78.3, 131.6)
- added R25: 100k, Resistor_SMD:R_0402_1005Metric, F.Cu at (80.8, 134.7)
- added R26: 9.09, Resistor_SMD:R_0402_1005Metric, F.Cu at (85.3, 139.1)
- added R27: 100k, Resistor_SMD:R_0402_1005Metric, F.Cu at (88.3, 141.6)
- added R28: 9.09, Resistor_SMD:R_0402_1005Metric, F.Cu at (93.6, 145.1)
- added R29: 100k, Resistor_SMD:R_0402_1005Metric, F.Cu at (97.1, 147.0)
- added R3: 100k, Resistor_SMD:R_0402_1005Metric, F.Cu at (113.0, 48.2)
- added R30: 9.09, Resistor_SMD:R_0402_1005Metric, F.Cu at (102.9, 149.4)
- added R31: 100k, Resistor_SMD:R_0402_1005Metric, F.Cu at (106.7, 150.6)
- added R32: 9.09, Resistor_SMD:R_0402_1005Metric, F.Cu at (112.9, 151.8)
- added R33: 100k, Resistor_SMD:R_0402_1005Metric, F.Cu at (116.8, 152.2)
- added R34: 9.09, Resistor_SMD:R_0402_1005Metric, F.Cu at (123.1, 152.2)
- added R35: 100k, Resistor_SMD:R_0402_1005Metric, F.Cu at (127.0, 151.8)
- added R36: 9.09, Resistor_SMD:R_0402_1005Metric, F.Cu at (133.2, 150.6)
- added R37: 100k, Resistor_SMD:R_0402_1005Metric, F.Cu at (137.0, 149.5)
- added R38: 9.09, Resistor_SMD:R_0402_1005Metric, F.Cu at (142.9, 147.1)
- added R39: 100k, Resistor_SMD:R_0402_1005Metric, F.Cu at (146.3, 145.2)
- added R40: 9.09, Resistor_SMD:R_0402_1005Metric, F.Cu at (151.6, 141.7)
- added R41: 100k, Resistor_SMD:R_0402_1005Metric, F.Cu at (154.7, 139.2)
- added R42: 9.09, Resistor_SMD:R_0402_1005Metric, F.Cu at (159.1, 134.7)
- added R43: 100k, Resistor_SMD:R_0402_1005Metric, F.Cu at (161.6, 131.7)
- added R44: 9.09, Resistor_SMD:R_0402_1005Metric, F.Cu at (165.1, 126.4)
- added R45: 100k, Resistor_SMD:R_0402_1005Metric, F.Cu at (167.0, 122.9)
- added R46: 9.09, Resistor_SMD:R_0402_1005Metric, F.Cu at (169.4, 117.1)
- added R47: 100k, Resistor_SMD:R_0402_1005Metric, F.Cu at (170.6, 113.3)
- added R48: 9.09, Resistor_SMD:R_0402_1005Metric, F.Cu at (171.8, 107.1)
- added R49: 100k, Resistor_SMD:R_0402_1005Metric, F.Cu at (172.2, 103.2)
- added R5: 100k, Resistor_SMD:R_0402_1005Metric, F.Cu at (103.0, 50.5)
- added R50: 9.09, Resistor_SMD:R_0402_1005Metric, F.Cu at (172.2, 96.9)
- added R51: 100k, Resistor_SMD:R_0402_1005Metric, F.Cu at (171.8, 93.0)
- added R52: 9.09, Resistor_SMD:R_0402_1005Metric, F.Cu at (170.6, 86.8)
- added R53: 100k, Resistor_SMD:R_0402_1005Metric, F.Cu at (169.5, 83.0)
- added R54: 9.09, Resistor_SMD:R_0402_1005Metric, F.Cu at (167.1, 77.1)
- added R55: 100k, Resistor_SMD:R_0402_1005Metric, F.Cu at (165.2, 73.7)
- added R56: 9.09, Resistor_SMD:R_0402_1005Metric, F.Cu at (161.7, 68.4)
- added R57: 100k, Resistor_SMD:R_0402_1005Metric, F.Cu at (159.2, 65.3)
- added R58: 9.09, Resistor_SMD:R_0402_1005Metric, F.Cu at (154.7, 60.9)
- added R59: 100k, Resistor_SMD:R_0402_1005Metric, F.Cu at (151.7, 58.4)
- added R6: 9.09, Resistor_SMD:R_0402_1005Metric, F.Cu at (97.1, 52.9)
- added R60: 9.09, Resistor_SMD:R_0402_1005Metric, F.Cu at (146.4, 54.9)
- added R61: 100k, Resistor_SMD:R_0402_1005Metric, F.Cu at (142.9, 53.0)
- added R62: 9.09, Resistor_SMD:R_0402_1005Metric, F.Cu at (137.1, 50.6)
- added R63: 100k, Resistor_SMD:R_0402_1005Metric, F.Cu at (133.3, 49.4)
- added R64: 9.09, Resistor_SMD:R_0402_1005Metric, F.Cu at (127.1, 48.2)
- added R65: 10k, Resistor_SMD:R_0402_1005Metric, F.Cu at (37.4, 46.1)
- added R66: 10k, Resistor_SMD:R_0402_1005Metric, F.Cu at (37.4, 48.1)
- added R7: 100k, Resistor_SMD:R_0402_1005Metric, F.Cu at (93.7, 54.8)
- added R8: 9.09, Resistor_SMD:R_0402_1005Metric, F.Cu at (88.4, 58.3)
- added R9: 100k, Resistor_SMD:R_0402_1005Metric, F.Cu at (85.3, 60.8)
- added REF**: R_0201_0603Metric, Resistor_SMD:R_0201_0603Metric, F.Cu at (118.6, 27.7)
- added REF**: R_0201_0603Metric, Resistor_SMD:R_0201_0603Metric, F.Cu at (110.3, 30.9)
- added REF**: R_0201_0603Metric, Resistor_SMD:R_0201_0603Metric, F.Cu at (106.0, 25.1)
- added REF**: R_0201_0603Metric, Resistor_SMD:R_0201_0603Metric, F.Cu at (116.8, 27.1)
- added REF**: R_0201_0603Metric, Resistor_SMD:R_0201_0603Metric, F.Cu at (116.8, 25.8)
- added REF**: R_0201_0603Metric, Resistor_SMD:R_0201_0603Metric, F.Cu at (116.8, 28.4)
- added REF**: R_0201_0603Metric, Resistor_SMD:R_0201_0603Metric, F.Cu at (111.0, 32.7)
- added REF**: R_0201_0603Metric, Resistor_SMD:R_0201_0603Metric, F.Cu at (118.6, 26.4)
- added REF**: R_0201_0603Metric, Resistor_SMD:R_0201_0603Metric, F.Cu at (113.6, 32.7)
- added REF**: R_0201_0603Metric, Resistor_SMD:R_0201_0603Metric, F.Cu at (111.6, 30.9)
- added REF**: R_0201_0603Metric, Resistor_SMD:R_0201_0603Metric, F.Cu at (107.8, 28.4)
- added REF**: R_0201_0603Metric, Resistor_SMD:R_0201_0603Metric, F.Cu at (106.0, 27.7)
- added REF**: R_0201_0603Metric, Resistor_SMD:R_0201_0603Metric, F.Cu at (107.8, 24.5)
- added REF**: R_0201_0603Metric, Resistor_SMD:R_0201_0603Metric, F.Cu at (112.9, 30.9)
- added REF**: R_0201_0603Metric, Resistor_SMD:R_0201_0603Metric, F.Cu at (107.8, 27.1)
- added REF**: R_0201_0603Metric, Resistor_SMD:R_0201_0603Metric, F.Cu at (107.8, 25.8)
- added REF**: R_0201_0603Metric, Resistor_SMD:R_0201_0603Metric, F.Cu at (114.2, 30.9)
- added U34: PCA9685BS,118, Library:QFN65P600X600X100-29N-D, F.Cu at (133.3, 29.1)
- added U35: STM32WB50CGUx, Package_DFN_QFN:QFN-48-1EP_7x7mm_P0.5mm_EP5.6x5.6mm, F.Cu at (37.0, 40.5)
- R2: value 80.6 -> 9.09; footprint Resistor_SMD:R_1210_3225Metric -> Resistor_SMD:R_0402_1005Metric
- R4: value 10k -> 9.09
- U29: value PCA9685BS,118 -> NCR321PASX; footprint Library:QFN65P600X600X100-29N-D -> Library:NCR321PASX
- U33: value NCR321PASX -> PCA9685BS,118; footprint Library:NCR321PASX -> Library:QFN65P600X600X100-29N-D
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Connections:
- D1 pad 1: Net-(D1-K-Pad1) -> /OUT1
- D1 pad 2: Net-(D1-K-Pad1) -> /OUT1
- D1 pad 3: Net-(D1-A-Pad3) -> +12V
- D1 pad 4: Net-(D1-A-Pad3) -> +12V
- D10 pad 1: Net-(D1-K-Pad1) -> /OUT10
- D10 pad 2: Net-(D1-K-Pad1) -> /OUT10
- D10 pad 3: Net-(D1-A-Pad3) -> +12V
- D10 pad 4: Net-(D1-A-Pad3) -> +12V
- D11 pad 1: Net-(D1-A-Pad3) -> /OUT11
- D11 pad 2: Net-(D1-A-Pad3) -> /OUT11
- D11 pad 3: Net-(D2-A-Pad3) -> +12V
- D11 pad 4: Net-(D2-A-Pad3) -> +12V
- D12 pad 1: Net-(D2-A-Pad3) -> /OUT12
- D12 pad 2: Net-(D2-A-Pad3) -> /OUT12
- D13 pad 1: Net-(D1-K-Pad1) -> /OUT13
- D13 pad 2: Net-(D1-K-Pad1) -> /OUT13
- D13 pad 3: Net-(D1-A-Pad3) -> +12V
- D13 pad 4: Net-(D1-A-Pad3) -> +12V
- D14 pad 1: Net-(D1-A-Pad3) -> /OUT14
- D14 pad 2: Net-(D1-A-Pad3) -> /OUT14
- D14 pad 3: Net-(D2-A-Pad3) -> +12V
- D14 pad 4: Net-(D2-A-Pad3) -> +12V
- D15 pad 1: Net-(D2-A-Pad3) -> /OUT15
- D15 pad 2: Net-(D2-A-Pad3) -> /OUT15
- D16 pad 1: Net-(D1-K-Pad1) -> /OUT16
- D16 pad 2: Net-(D1-K-Pad1) -> /OUT16
- D16 pad 3: Net-(D1-A-Pad3) -> +12V
- D16 pad 4: Net-(D1-A-Pad3) -> +12V
- D17 pad 1: Net-(D1-A-Pad3) -> /OUT17
- D17 pad 2: Net-(D1-A-Pad3) -> /OUT17
- D17 pad 3: Net-(D2-A-Pad3) -> +12V
- D17 pad 4: Net-(D2-A-Pad3) -> +12V
- D18 pad 1: Net-(D2-A-Pad3) -> /OUT18
- D18 pad 2: Net-(D2-A-Pad3) -> /OUT18
- D19 pad 1: Net-(D1-K-Pad1) -> /OUT19
- D19 pad 2: Net-(D1-K-Pad1) -> /OUT19
- D19 pad 3: Net-(D1-A-Pad3) -> +12V
- D19 pad 4: Net-(D1-A-Pad3) -> +12V
- D2 pad 1: Net-(D1-A-Pad3) -> /OUT2
- D2 pad 2: Net-(D1-A-Pad3) -> /OUT2
- D2 pad 3: Net-(D2-A-Pad3) -> +12V
- D2 pad 4: Net-(D2-A-Pad3) -> +12V
- D20 pad 1: Net-(D1-A-Pad3) -> /OUT20
- D20 pad 2: Net-(D1-A-Pad3) -> /OUT20
- D20 pad 3: Net-(D2-A-Pad3) -> +12V
- D20 pad 4: Net-(D2-A-Pad3) -> +12V
- D21 pad 1: Net-(D2-A-Pad3) -> /OUT21
- D21 pad 2: Net-(D2-A-Pad3) -> /OUT21
- D22 pad 1: Net-(D1-K-Pad1) -> /OUT22
- D22 pad 2: Net-(D1-K-Pad1) -> /OUT22
- D22 pad 3: Net-(D1-A-Pad3) -> +12V
- D22 pad 4: Net-(D1-A-Pad3) -> +12V
- D23 pad 1: Net-(D1-A-Pad3) -> /OUT23
- D23 pad 2: Net-(D1-A-Pad3) -> /OUT23
- D23 pad 3: Net-(D2-A-Pad3) -> +12V
- D23 pad 4: Net-(D2-A-Pad3) -> +12V
- D24 pad 1: Net-(D2-A-Pad3) -> /OUT24
- D24 pad 2: Net-(D2-A-Pad3) -> /OUT24
- D25 pad 1: Net-(D1-K-Pad1) -> /OUT25
- D25 pad 2: Net-(D1-K-Pad1) -> /OUT25
- D25 pad 3: Net-(D1-A-Pad3) -> +12V
- D25 pad 4: Net-(D1-A-Pad3) -> +12V
- D26 pad 1: Net-(D1-A-Pad3) -> /OUT26
- D26 pad 2: Net-(D1-A-Pad3) -> /OUT26
- D26 pad 3: Net-(D2-A-Pad3) -> +12V
- D26 pad 4: Net-(D2-A-Pad3) -> +12V
- D27 pad 1: Net-(D2-A-Pad3) -> /OUT27
- D27 pad 2: Net-(D2-A-Pad3) -> /OUT27
- D28 pad 1: Net-(D1-K-Pad1) -> /OUT28
- D28 pad 2: Net-(D1-K-Pad1) -> /OUT28
- D28 pad 3: Net-(D1-A-Pad3) -> +12V
- D28 pad 4: Net-(D1-A-Pad3) -> +12V
- D29 pad 1: Net-(D1-A-Pad3) -> /OUT29
- D29 pad 2: Net-(D1-A-Pad3) -> /OUT29
- D29 pad 3: Net-(D2-A-Pad3) -> +12V
- D29 pad 4: Net-(D2-A-Pad3) -> +12V
- D3 pad 1: Net-(D2-A-Pad3) -> /OUT3
- D3 pad 2: Net-(D2-A-Pad3) -> /OUT3
- D30 pad 1: Net-(D2-A-Pad3) -> /OUT30
- D30 pad 2: Net-(D2-A-Pad3) -> /OUT30
- D31 pad 1: Net-(D1-K-Pad1) -> /OUT31
- D31 pad 2: Net-(D1-K-Pad1) -> /OUT31
- D31 pad 3: Net-(D1-A-Pad3) -> +12V
- D31 pad 4: Net-(D1-A-Pad3) -> +12V
- D32 pad 1: Net-(D1-A-Pad3) -> /OUT32
- D32 pad 2: Net-(D1-A-Pad3) -> /OUT32
- D32 pad 3: Net-(D2-A-Pad3) -> +12V
- D32 pad 4: Net-(D2-A-Pad3) -> +12V
- D4 pad 1: Net-(D1-K-Pad1) -> /OUT4
- D4 pad 2: Net-(D1-K-Pad1) -> /OUT4
- D4 pad 3: Net-(D1-A-Pad3) -> +12V
- D4 pad 4: Net-(D1-A-Pad3) -> +12V
- D5 pad 1: Net-(D1-A-Pad3) -> /OUT5
- D5 pad 2: Net-(D1-A-Pad3) -> /OUT5
- D5 pad 3: Net-(D2-A-Pad3) -> +12V
- D5 pad 4: Net-(D2-A-Pad3) -> +12V
- D6 pad 1: Net-(D2-A-Pad3) -> /OUT6
- D6 pad 2: Net-(D2-A-Pad3) -> /OUT6
- D7 pad 1: Net-(D1-K-Pad1) -> /OUT7
- D7 pad 2: Net-(D1-K-Pad1) -> /OUT7
- D7 pad 3: Net-(D1-A-Pad3) -> +12V
- D7 pad 4: Net-(D1-A-Pad3) -> +12V
- D8 pad 1: Net-(D1-A-Pad3) -> /OUT8
- D8 pad 2: Net-(D1-A-Pad3) -> /OUT8
- D8 pad 3: Net-(D2-A-Pad3) -> +12V
- D8 pad 4: Net-(D2-A-Pad3) -> +12V
- D9 pad 1: Net-(D2-A-Pad3) -> /OUT9
- D9 pad 2: Net-(D2-A-Pad3) -> /OUT9
- R2 pad 1: Net-(U1-REXT) -> /REXT1
- R4 pad 1: SDA -> /REXT2
- R4 pad 2: +3.3V -> GND
- U1 pad 1: +12V -> PWM1
- U1 pad 2: Net-(U1-REXT) -> /REXT1
- U1 pad 6: Net-(D1-K-Pad1) -> /OUT1
- U1 pad 7: Net-(D1-K-Pad1) -> /OUT1
- U10 pad 1: +12V -> PWM10
- U10 pad 2: Net-(U1-REXT) -> /REXT10
- U10 pad 3: unconnected-(U1-N/C_1-Pad3) -> unconnected-(U10-N/C_1-Pad3)
- U10 pad 4: unconnected-(U1-N/C_2-Pad4) -> unconnected-(U10-N/C_2-Pad4)
- U10 pad 6: Net-(D1-K-Pad1) -> /OUT10
- U10 pad 7: Net-(D1-K-Pad1) -> /OUT10
- U10 pad 8: unconnected-(U1-N/C_3-Pad8) -> unconnected-(U10-N/C_3-Pad8)
- U11 pad 1: +12V -> PWM11
- U11 pad 2: Net-(U1-REXT) -> /REXT11
- U11 pad 3: unconnected-(U1-N/C_1-Pad3) -> unconnected-(U11-N/C_1-Pad3)
- U11 pad 4: unconnected-(U1-N/C_2-Pad4) -> unconnected-(U11-N/C_2-Pad4)
- U11 pad 6: Net-(D1-K-Pad1) -> /OUT11
- U11 pad 7: Net-(D1-K-Pad1) -> /OUT11
- U11 pad 8: unconnected-(U1-N/C_3-Pad8) -> unconnected-(U11-N/C_3-Pad8)
- U12 pad 1: +12V -> PWM12
- U12 pad 2: Net-(U1-REXT) -> /REXT12
- U12 pad 3: unconnected-(U1-N/C_1-Pad3) -> unconnected-(U12-N/C_1-Pad3)
- U12 pad 4: unconnected-(U1-N/C_2-Pad4) -> unconnected-(U12-N/C_2-Pad4)
- U12 pad 6: Net-(D1-K-Pad1) -> /OUT12
- U12 pad 7: Net-(D1-K-Pad1) -> /OUT12
- U12 pad 8: unconnected-(U1-N/C_3-Pad8) -> unconnected-(U12-N/C_3-Pad8)
- U13 pad 1: +12V -> PWM13
- U13 pad 2: Net-(U1-REXT) -> /REXT13
- U13 pad 3: unconnected-(U1-N/C_1-Pad3) -> unconnected-(U13-N/C_1-Pad3)
- U13 pad 4: unconnected-(U1-N/C_2-Pad4) -> unconnected-(U13-N/C_2-Pad4)
- U13 pad 6: Net-(D1-K-Pad1) -> /OUT13
- U13 pad 7: Net-(D1-K-Pad1) -> /OUT13
- U13 pad 8: unconnected-(U1-N/C_3-Pad8) -> unconnected-(U13-N/C_3-Pad8)
- U14 pad 1: +12V -> PWM14
- U14 pad 2: Net-(U1-REXT) -> /REXT14
- U14 pad 3: unconnected-(U1-N/C_1-Pad3) -> unconnected-(U14-N/C_1-Pad3)
- U14 pad 4: unconnected-(U1-N/C_2-Pad4) -> unconnected-(U14-N/C_2-Pad4)
- U14 pad 6: Net-(D1-K-Pad1) -> /OUT14
- U14 pad 7: Net-(D1-K-Pad1) -> /OUT14
- U14 pad 8: unconnected-(U1-N/C_3-Pad8) -> unconnected-(U14-N/C_3-Pad8)
- U15 pad 1: +12V -> PWM15
- U15 pad 2: Net-(U1-REXT) -> /REXT15
- U15 pad 3: unconnected-(U1-N/C_1-Pad3) -> unconnected-(U15-N/C_1-Pad3)
- U15 pad 4: unconnected-(U1-N/C_2-Pad4) -> unconnected-(U15-N/C_2-Pad4)
- U15 pad 6: Net-(D1-K-Pad1) -> /OUT15
- U15 pad 7: Net-(D1-K-Pad1) -> /OUT15
- U15 pad 8: unconnected-(U1-N/C_3-Pad8) -> unconnected-(U15-N/C_3-Pad8)
- U16 pad 1: +12V -> PWM16
- U16 pad 2: Net-(U1-REXT) -> /REXT16
- U16 pad 3: unconnected-(U1-N/C_1-Pad3) -> unconnected-(U16-N/C_1-Pad3)
- U16 pad 4: unconnected-(U1-N/C_2-Pad4) -> unconnected-(U16-N/C_2-Pad4)
- U16 pad 6: Net-(D1-K-Pad1) -> /OUT16
- U16 pad 7: Net-(D1-K-Pad1) -> /OUT16
- U16 pad 8: unconnected-(U1-N/C_3-Pad8) -> unconnected-(U16-N/C_3-Pad8)
- U17 pad 1: +12V -> PWM17
- U17 pad 2: Net-(U1-REXT) -> /REXT17
- U17 pad 3: unconnected-(U1-N/C_1-Pad3) -> unconnected-(U17-N/C_1-Pad3)
- U17 pad 4: unconnected-(U1-N/C_2-Pad4) -> unconnected-(U17-N/C_2-Pad4)
- U17 pad 6: Net-(D1-K-Pad1) -> /OUT17
- U17 pad 7: Net-(D1-K-Pad1) -> /OUT17
- U17 pad 8: unconnected-(U1-N/C_3-Pad8) -> unconnected-(U17-N/C_3-Pad8)
- U18 pad 1: +12V -> PWM18
- U18 pad 2: Net-(U1-REXT) -> /REXT18
- U18 pad 3: unconnected-(U1-N/C_1-Pad3) -> unconnected-(U18-N/C_1-Pad3)
- U18 pad 4: unconnected-(U1-N/C_2-Pad4) -> unconnected-(U18-N/C_2-Pad4)
- U18 pad 6: Net-(D1-K-Pad1) -> /OUT18
- U18 pad 7: Net-(D1-K-Pad1) -> /OUT18
- U18 pad 8: unconnected-(U1-N/C_3-Pad8) -> unconnected-(U18-N/C_3-Pad8)
- U19 pad 1: +12V -> PWM19
- U19 pad 2: Net-(U1-REXT) -> /REXT19
- U19 pad 3: unconnected-(U1-N/C_1-Pad3) -> unconnected-(U19-N/C_1-Pad3)
- U19 pad 4: unconnected-(U1-N/C_2-Pad4) -> unconnected-(U19-N/C_2-Pad4)
- U19 pad 6: Net-(D1-K-Pad1) -> /OUT19
- U19 pad 7: Net-(D1-K-Pad1) -> /OUT19
- U19 pad 8: unconnected-(U1-N/C_3-Pad8) -> unconnected-(U19-N/C_3-Pad8)
- U2 pad 1: +12V -> PWM2
- U2 pad 2: Net-(U1-REXT) -> /REXT2
- U2 pad 3: unconnected-(U1-N/C_1-Pad3) -> unconnected-(U2-N/C_1-Pad3)
- U2 pad 4: unconnected-(U1-N/C_2-Pad4) -> unconnected-(U2-N/C_2-Pad4)
- U2 pad 6: Net-(D1-K-Pad1) -> /OUT2
- U2 pad 7: Net-(D1-K-Pad1) -> /OUT2
- U2 pad 8: unconnected-(U1-N/C_3-Pad8) -> unconnected-(U2-N/C_3-Pad8)
- U20 pad 1: +12V -> PWM20
- U20 pad 2: Net-(U1-REXT) -> /REXT20
- U20 pad 3: unconnected-(U1-N/C_1-Pad3) -> unconnected-(U20-N/C_1-Pad3)
- U20 pad 4: unconnected-(U1-N/C_2-Pad4) -> unconnected-(U20-N/C_2-Pad4)
- U20 pad 6: Net-(D1-K-Pad1) -> /OUT20
- U20 pad 7: Net-(D1-K-Pad1) -> /OUT20
- U20 pad 8: unconnected-(U1-N/C_3-Pad8) -> unconnected-(U20-N/C_3-Pad8)
- U21 pad 1: +12V -> PWM21
- U21 pad 2: Net-(U1-REXT) -> /REXT21
- U21 pad 3: unconnected-(U1-N/C_1-Pad3) -> unconnected-(U21-N/C_1-Pad3)
- U21 pad 4: unconnected-(U1-N/C_2-Pad4) -> unconnected-(U21-N/C_2-Pad4)
- U21 pad 6: Net-(D1-K-Pad1) -> /OUT21
- U21 pad 7: Net-(D1-K-Pad1) -> /OUT21
- U21 pad 8: unconnected-(U1-N/C_3-Pad8) -> unconnected-(U21-N/C_3-Pad8)
- U22 pad 1: +12V -> PWM22
- U22 pad 2: Net-(U1-REXT) -> /REXT22
- U22 pad 3: unconnected-(U1-N/C_1-Pad3) -> unconnected-(U22-N/C_1-Pad3)
- U22 pad 4: unconnected-(U1-N/C_2-Pad4) -> unconnected-(U22-N/C_2-Pad4)
- U22 pad 6: Net-(D1-K-Pad1) -> /OUT22
- U22 pad 7: Net-(D1-K-Pad1) -> /OUT22
- U22 pad 8: unconnected-(U1-N/C_3-Pad8) -> unconnected-(U22-N/C_3-Pad8)
- U23 pad 1: +12V -> PWM23
- U23 pad 2: Net-(U1-REXT) -> /REXT23
- U23 pad 3: unconnected-(U1-N/C_1-Pad3) -> unconnected-(U23-N/C_1-Pad3)
- U23 pad 4: unconnected-(U1-N/C_2-Pad4) -> unconnected-(U23-N/C_2-Pad4)
- U23 pad 6: Net-(D1-K-Pad1) -> /OUT23
- U23 pad 7: Net-(D1-K-Pad1) -> /OUT23
- U23 pad 8: unconnected-(U1-N/C_3-Pad8) -> unconnected-(U23-N/C_3-Pad8)
- U24 pad 1: +12V -> PWM24
- U24 pad 2: Net-(U1-REXT) -> /REXT24
- U24 pad 3: unconnected-(U1-N/C_1-Pad3) -> unconnected-(U24-N/C_1-Pad3)
- U24 pad 4: unconnected-(U1-N/C_2-Pad4) -> unconnected-(U24-N/C_2-Pad4)
- U24 pad 6: Net-(D1-K-Pad1) -> /OUT24
- U24 pad 7: Net-(D1-K-Pad1) -> /OUT24
- U24 pad 8: unconnected-(U1-N/C_3-Pad8) -> unconnected-(U24-N/C_3-Pad8)
- U25 pad 1: +12V -> PWM25
- U25 pad 2: Net-(U1-REXT) -> /REXT25
- U25 pad 3: unconnected-(U1-N/C_1-Pad3) -> unconnected-(U25-N/C_1-Pad3)
- U25 pad 4: unconnected-(U1-N/C_2-Pad4) -> unconnected-(U25-N/C_2-Pad4)
- U25 pad 6: Net-(D1-K-Pad1) -> /OUT25
- U25 pad 7: Net-(D1-K-Pad1) -> /OUT25
- U25 pad 8: unconnected-(U1-N/C_3-Pad8) -> unconnected-(U25-N/C_3-Pad8)
- U26 pad 1: +12V -> PWM26
- U26 pad 2: Net-(U1-REXT) -> /REXT26
- U26 pad 3: unconnected-(U1-N/C_1-Pad3) -> unconnected-(U26-N/C_1-Pad3)
- U26 pad 4: unconnected-(U1-N/C_2-Pad4) -> unconnected-(U26-N/C_2-Pad4)
- U26 pad 6: Net-(D1-K-Pad1) -> /OUT26
- U26 pad 7: Net-(D1-K-Pad1) -> /OUT26
- U26 pad 8: unconnected-(U1-N/C_3-Pad8) -> unconnected-(U26-N/C_3-Pad8)
- U27 pad 1: +12V -> PWM27
- U27 pad 2: Net-(U1-REXT) -> /REXT27
- U27 pad 3: unconnected-(U1-N/C_1-Pad3) -> unconnected-(U27-N/C_1-Pad3)
- U27 pad 4: unconnected-(U1-N/C_2-Pad4) -> unconnected-(U27-N/C_2-Pad4)
- U27 pad 6: Net-(D1-K-Pad1) -> /OUT27
- U27 pad 7: Net-(D1-K-Pad1) -> /OUT27
- U27 pad 8: unconnected-(U1-N/C_3-Pad8) -> unconnected-(U27-N/C_3-Pad8)
- U28 pad 1: +12V -> PWM28
- U28 pad 2: Net-(U1-REXT) -> /REXT28
- U28 pad 3: unconnected-(U1-N/C_1-Pad3) -> unconnected-(U28-N/C_1-Pad3)
- U28 pad 4: unconnected-(U1-N/C_2-Pad4) -> unconnected-(U28-N/C_2-Pad4)
- U28 pad 6: Net-(D1-K-Pad1) -> /OUT28
- U28 pad 7: Net-(D1-K-Pad1) -> /OUT28
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Routing:
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- added copper zone on B.Cu, net +12V
- added copper zone on In1.Cu, net +12V
- added copper zone on In2.Cu, net +12V
- added copper zone on B.Cu, net /OUT1
- added copper zone on F.Cu, net /OUT1
- added copper zone on In1.Cu, net /OUT1
- added copper zone on In2.Cu, net /OUT1
- added copper zone on B.Cu, net /OUT10
- added copper zone on F.Cu, net /OUT10
- added copper zone on In1.Cu, net /OUT10
- added copper zone on In2.Cu, net /OUT10
- added copper zone on B.Cu, net /OUT11
- added copper zone on F.Cu, net /OUT11
- added copper zone on In1.Cu, net /OUT11
- added copper zone on In2.Cu, net /OUT11
- added copper zone on B.Cu, net /OUT12
- added copper zone on F.Cu, net /OUT12
- added copper zone on In1.Cu, net /OUT12
- added copper zone on In2.Cu, net /OUT12
- added copper zone on B.Cu, net /OUT13
- added copper zone on F.Cu, net /OUT13
- added copper zone on In1.Cu, net /OUT13
- added copper zone on In2.Cu, net /OUT13
- added copper zone on B.Cu, net /OUT14
- added copper zone on F.Cu, net /OUT14
- added copper zone on In1.Cu, net /OUT14
- added copper zone on In2.Cu, net /OUT14
- added copper zone on B.Cu, net /OUT15
- added copper zone on F.Cu, net /OUT15
- added copper zone on In1.Cu, net /OUT15
- added copper zone on In2.Cu, net /OUT15
- added copper zone on B.Cu, net /OUT16
- added copper zone on F.Cu, net /OUT16
- added copper zone on In1.Cu, net /OUT16
- added copper zone on In2.Cu, net /OUT16
- added copper zone on B.Cu, net /OUT17
- added copper zone on F.Cu, net /OUT17
- added copper zone on In1.Cu, net /OUT17
- added copper zone on In2.Cu, net /OUT17
- added copper zone on B.Cu, net /OUT18
- added copper zone on F.Cu, net /OUT18
- added copper zone on In1.Cu, net /OUT18
- added copper zone on In2.Cu, net /OUT18
- added copper zone on B.Cu, net /OUT19
- added copper zone on F.Cu, net /OUT19
- added copper zone on In1.Cu, net /OUT19
- added copper zone on In2.Cu, net /OUT19
- added copper zone on B.Cu, net /OUT2
- added copper zone on F.Cu, net /OUT2
- added copper zone on In1.Cu, net /OUT2
- added copper zone on In2.Cu, net /OUT2
- added copper zone on B.Cu, net /OUT20
- added copper zone on F.Cu, net /OUT20
- added copper zone on In1.Cu, net /OUT20
- added copper zone on In2.Cu, net /OUT20
- added copper zone on B.Cu, net /OUT21
- added copper zone on F.Cu, net /OUT21
- added copper zone on In1.Cu, net /OUT21
- added copper zone on In2.Cu, net /OUT21
- added copper zone on B.Cu, net /OUT22
- added copper zone on F.Cu, net /OUT22
- added copper zone on In1.Cu, net /OUT22
- added copper zone on In2.Cu, net /OUT22
- added copper zone on B.Cu, net /OUT23
- added copper zone on F.Cu, net /OUT23
- added copper zone on In1.Cu, net /OUT23
- added copper zone on In2.Cu, net /OUT23
- added copper zone on B.Cu, net /OUT24
- added copper zone on F.Cu, net /OUT24
- added copper zone on In1.Cu, net /OUT24
- added copper zone on In2.Cu, net /OUT24
- added copper zone on B.Cu, net /OUT25
- added copper zone on F.Cu, net /OUT25
- added copper zone on In1.Cu, net /OUT25
- added copper zone on In2.Cu, net /OUT25
- added copper zone on B.Cu, net /OUT26
- added copper zone on F.Cu, net /OUT26
- added copper zone on In1.Cu, net /OUT26
- added copper zone on In2.Cu, net /OUT26
- added copper zone on B.Cu, net /OUT27
- added copper zone on F.Cu, net /OUT27
- added copper zone on In1.Cu, net /OUT27
- added copper zone on In2.Cu, net /OUT27
- added copper zone on B.Cu, net /OUT28
- added copper zone on F.Cu, net /OUT28
- added copper zone on In1.Cu, net /OUT28
- added copper zone on In2.Cu, net /OUT28
- added copper zone on B.Cu, net /OUT29
- added copper zone on F.Cu, net /OUT29
- added copper zone on In1.Cu, net /OUT29
- added copper zone on In2.Cu, net /OUT29
- added copper zone on B.Cu, net /OUT3
- added copper zone on F.Cu, net /OUT3
- added copper zone on In1.Cu, net /OUT3
- added copper zone on In2.Cu, net /OUT3
- added copper zone on B.Cu, net /OUT30
- added copper zone on F.Cu, net /OUT30
- added copper zone on In1.Cu, net /OUT30
- added copper zone on In2.Cu, net /OUT30
- added copper zone on B.Cu, net /OUT31
- added copper zone on F.Cu, net /OUT31
- added copper zone on In1.Cu, net /OUT31
- added copper zone on In2.Cu, net /OUT31
- added copper zone on B.Cu, net /OUT32
- added copper zone on F.Cu, net /OUT32
- added copper zone on In1.Cu, net /OUT32
- added copper zone on In2.Cu, net /OUT32
- added copper zone on B.Cu, net /OUT4
- added copper zone on F.Cu, net /OUT4
- added copper zone on In1.Cu, net /OUT4
- added copper zone on In2.Cu, net /OUT4
- added copper zone on B.Cu, net /OUT5
- added copper zone on F.Cu, net /OUT5
- added copper zone on In1.Cu, net /OUT5
- added copper zone on In2.Cu, net /OUT5
- added copper zone on B.Cu, net /OUT6
- added copper zone on F.Cu, net /OUT6
- added copper zone on In1.Cu, net /OUT6
- added copper zone on In2.Cu, net /OUT6
- added copper zone on B.Cu, net /OUT7
- added copper zone on F.Cu, net /OUT7
- added copper zone on In1.Cu, net /OUT7
- added copper zone on In2.Cu, net /OUT7
- added copper zone on B.Cu, net /OUT8
- added copper zone on F.Cu, net /OUT8
- added copper zone on In1.Cu, net /OUT8
- added copper zone on In2.Cu, net /OUT8
- added copper zone on B.Cu, net /OUT9
- added copper zone on F.Cu, net /OUT9
- added copper zone on In1.Cu, net /OUT9
- added copper zone on In2.Cu, net /OUT9
- added copper zone on B.Cu, net GND
- added copper zone on F.Cu, net GND
- added copper zone on In1.Cu, net GND
Other:
- board size 124 x 135 mm -> 115 x 115 mm

Commit message: d
Routing:
- net PWM1: track 8.26 -> 4.45 mm
- net PWM2: track 5.31 -> 2.31 mm
- net PWM3: track 4.98 -> 2.38 mm
- net PWM4: track 4.73 -> 2.53 mm
- net PWM5: track 4.10 -> 2.30 mm
- net PWM6: track 3.88 -> 2.38 mm
- net PWM7: track 3.70 -> 2.50 mm
- net PWM8: track 3.20 -> 2.30 mm
Changed lines of the file:
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@@
 			(fill no)
 			(layer "F.CrtYd")
-			(net 1)
 		)
 		(fp_rect
@@
 			(fill no)
 			(layer "F.Fab")
-			(net 1)
 		)
 		(fp_text user "${REFERENCE}"
@@
 			(fill no)
 			(layer "F.CrtYd")
-			(net 1)
 		)
 		(fp_rect
@@
 			(fill no)
 			(layer "F.Fab")
-			(net 1)
 		)
 		(fp_text user "${REFERENCE}"
@@
 			(fill no)
 			(layer "F.CrtYd")
-			(net 16777472)
 		)
 		(fp_rect
@@
 			(fill no)
 			(layer "F.Fab")
-			(net 16777472)
 		)
 		(fp_text user "${REFERENCE}"
@@
 			(fill no)
 			(layer "F.CrtYd")
-			(net 1)
 		)
 		(fp_rect
@@
 			(fill no)
 			(layer "F.Fab")
-			(net 1)
 		)
 		(fp_text user "${REFERENCE}"
@@
 	)
 	(segment
-		(start 121.1 42)
-		(end 121.1 44.6)
-		(width 0.15)
-		(layer "F.Cu")
-		(net 8)
-	)
-	(segment
 		(start 102.510745 50.721766)
 		(end 102.6 50.632511)
@@
 	)
 	(segment
-		(start 119.9 41.9)
-		(end 119.9 43.4)
-		(width 0.15)
-		(layer "F.Cu")
-		(net 9)
-	)
-	(segment
 		(start 77.353355 70.722674)
 		(end 78.217267 69.429739)
@@
 	)
 	(segment
-		(start 119.1 41.9)
-		(end 119.1 42.8)
-		(width 0.15)
-		(layer "F.Cu")
-		(net 10)
-	)
-	(segment
 		(start 69.39569 89.271443)
 		(end 69.699055 87.746322)
@@
 	)
 	(segment
-		(start 121.9 44.8)
-		(end 121.9 42.1)
-		(width 0.15)
-		(layer "F.Cu")
-		(net 11)
-	)
-	(segment
-		(start 122.69 45.59)
-		(end 121.9 44.8)
-		(width 0.15)
-		(layer "F.Cu")
-		(net 11)
-	)
-	(segment
 		(start 122.205 48.275)
 		(end 122.7 47.78)
@@
 	)
 	(segment
-		(start 119.5 41.9)
-		(end 119.5 43.1)
-		(width 0.15)
-		(layer "F.Cu")
-		(net 13)
-	)
-	(segment
 		(start 72.788256 77.521797)
 		(end 72.720053 77.59)
@@
 	)
 	(segment
-		(start 121.5 42.1)
-		(end 121.5 45.1)
-		(width 0.15)
-		(layer "F.Cu")
-		(net 15)
-	)
-	(segment
 		(start 112.460504 48.256649)
 		(end 112.406649 48.256649)
@@
 	)
 	(segment
-		(start 120.3 42)
-		(end 120.3 43.8)
-		(width 0.15)
-		(layer "F.Cu")
-		(net 16)
-	)
-	(segment
 		(start 90.722674 142.646645)
 		(end 89.429739 141.782733)
@@
 		(layer "F.Cu")
 		(net 22)
-	)
-	(segment
-		(start 120.7 42)
-		(end 120.7 44.2)
-		(width 0.15)
-		(layer "F.Cu")
-		(net 22)

Commit message: m
Parts:
- removed U34: PCA9685BS,118, Library:QFN65P600X600X100-29N-D
- added REF**: R_0201_0603Metric, Resistor_SMD:R_0201_0603Metric, F.Cu at (126.0, 39.5)
- added REF**: R_0201_0603Metric, Resistor_SMD:R_0201_0603Metric, F.Cu at (126.7, 37.7)
- added REF**: R_0201_0603Metric, Resistor_SMD:R_0201_0603Metric, F.Cu at (128.7, 39.5)
- added REF**: R_0201_0603Metric, Resistor_SMD:R_0201_0603Metric, F.Cu at (122.9, 33.9)
- added REF**: R_0201_0603Metric, Resistor_SMD:R_0201_0603Metric, F.Cu at (125.4, 37.7)
- added REF**: R_0201_0603Metric, Resistor_SMD:R_0201_0603Metric, F.Cu at (122.9, 36.5)
- added REF**: R_0201_0603Metric, Resistor_SMD:R_0201_0603Metric, F.Cu at (128.0, 37.7)
- added REF**: R_0201_0603Metric, Resistor_SMD:R_0201_0603Metric, F.Cu at (121.1, 33.2)
- added REF**: MountingHole_2.2mm_M2, MountingHole:MountingHole_2.2mm_M2, F.Cu at (163.5, 113.2)
- added REF**: R_0201_0603Metric, Resistor_SMD:R_0201_0603Metric, F.Cu at (146.7, 32.5)
- added REF**: R_0201_0603Metric, Resistor_SMD:R_0201_0603Metric, F.Cu at (121.1, 35.9)
- added REF**: R_0201_0603Metric, Resistor_SMD:R_0201_0603Metric, F.Cu at (122.9, 35.2)
- added REF**: R_0201_0603Metric, Resistor_SMD:R_0201_0603Metric, F.Cu at (129.3, 37.7)
- added REF**: R_0201_0603Metric, Resistor_SMD:R_0201_0603Metric, F.Cu at (148.5, 34.5)
- added REF**: R_0201_0603Metric, Resistor_SMD:R_0201_0603Metric, F.Cu at (122.9, 32.6)
- added REF**: R_0201_0603Metric, Resistor_SMD:R_0201_0603Metric, F.Cu at (146.7, 35.1)
- added REF**: R_0201_0603Metric, Resistor_SMD:R_0201_0603Metric, F.Cu at (148.5, 33.1)
- added REF**: R_0201_0603Metric, Resistor_SMD:R_0201_0603Metric, F.Cu at (146.7, 33.8)
- added REF**12: MountingHole_2.2mm_M2, MountingHole:MountingHole_2.2mm_M2, F.Cu at (98.6, 59.9)
- added REF**16: MountingHole_2.2mm_M2, MountingHole:MountingHole_2.2mm_M2, F.Cu at (76.5, 86.8)
- added REF**20: MountingHole_2.2mm_M2, MountingHole:MountingHole_2.2mm_M2, F.Cu at (79.9, 121.4)
- added REF**24: MountingHole_2.2mm_M2, MountingHole:MountingHole_2.2mm_M2, F.Cu at (106.8, 143.5)
- added REF**28: MountingHole_2.2mm_M2, MountingHole:MountingHole_2.2mm_M2, F.Cu at (141.4, 140.1)
- added REF**4: MountingHole_2.2mm_M2, MountingHole:MountingHole_2.2mm_M2, F.Cu at (160.1, 78.6)
- added REF**8: MountingHole_2.2mm_M2, MountingHole:MountingHole_2.2mm_M2, F.Cu at (133.2, 56.5)
- added U33: PCA9685BS,118, Library:QFN65P600X600X100-29N-D, F.Cu at (127.3, 33.2)
- moved REF** 6.84 mm to (116.8, 35.2)
- moved REF** 6.84 mm to (107.9, 35.2)
- moved REF** 6.84 mm to (107.9, 31.3)
- moved REF** 6.84 mm to (113.0, 37.8)
- moved REF** 6.84 mm to (107.9, 33.9)
- moved REF** 6.84 mm to (107.9, 32.6)
- moved REF** 6.84 mm to (111.7, 37.8)
- moved REF** 6.84 mm to (114.3, 37.8)
- moved REF** 6.84 mm to (110.4, 37.8)
- moved REF** 6.84 mm to (106.1, 31.9)
- moved REF** 6.84 mm to (116.8, 33.9)
- moved REF** 6.84 mm to (116.8, 32.6)
- moved REF** 6.84 mm to (118.7, 33.2)
- moved U33 6.84 mm to (112.3, 33.2)
- moved REF** 6.84 mm to (118.7, 34.5)
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Routing:
- net /OUT8: vias 61 -> 58
- net /OUT7: vias 61 -> 58
- net /OUT4: vias 61 -> 58
- net /OUT32: vias 61 -> 58
- net /OUT31: vias 61 -> 58
- net /OUT3: vias 61 -> 58
- net /OUT28: vias 61 -> 58
- net /OUT27: vias 61 -> 58
- net /OUT24: vias 61 -> 58
- net /OUT23: vias 64 -> 61
- net /OUT20: vias 61 -> 58
- net /OUT19: vias 61 -> 58
- net /OUT16: vias 60 -> 57
- net /OUT15: vias 61 -> 58
- net /OUT12: vias 61 -> 58
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
Commit message: d
Routing:
- net PWM9: track 3.53 -> 8.55 mm
- net PWM10: track 3.29 -> 7.74 mm
- net PWM11: track 3.29 -> 7.17 mm
Changed lines of the file:
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@@
 	)
 	(gr_arc
-		(start 85.080291 143.784724)
-		(mid 66.111527 84.751372)
-		(end 113.2 44.41)
+		(start 85.083084 143.781222)
+		(mid 66.667862 82.921667)
+		(end 117.01 44.08)
 		(stroke
 			(width 0.15)
@@
 	)
 	(gr_arc
-		(start 77.978893 136.235469)
-		(mid 68.326017 79.783212)
-		(end 113.71 44.85)
+		(start 77.981562 136.23317)
+		(mid 69.055768 78.016839)
+		(end 117.52 44.55)
 		(stroke
 			(width 0.15)
@@
 	)
 	(gr_arc
-		(start 93.286741 149.821496)
-		(mid 64.421367 89.808153)
-		(end 112.72 43.96)
+		(start 93.293483 149.808937)
+		(mid 64.810466 87.944976)
+		(end 116.51 43.61)
 		(stroke
 			(width 0.15)
@@
 	)
 	(gr_arc
-		(start 68.499334 117.798457)
-		(mid 74.14576 70.58327)
-		(end 114.71 45.77)
+		(start 68.488352 117.802249)
+		(mid 75.192278 68.992161)
+		(end 118.51 45.52)
 		(stroke
 			(width 0.15)
@@
 	)
 	(gr_arc
-		(start 72.367341 127.523833)
-		(mid 70.979115 75.064125)
-		(end 114.2 45.3)
+		(start 72.36872 127.523035)
+		(mid 71.873649 73.382125)
+		(end 118 45.03)
 		(stroke
 			(width 0.15)
@@
 	)
 	(gr_arc
-		(start 66.594999 97.30076)
-		(mid 81.625842 62.760182)
-		(end 115.7 46.7)
+		(start 66.585845 97.300295)
+		(mid 82.968343 61.41222)
+		(end 119.5 46.52)
 		(stroke
 			(width 0.15)
@@
 	)
 	(gr_arc
-		(start 66.557058 107.584311)
-		(mid 77.704188 66.449564)
-		(end 115.21 46.21)
+		(start 66.56223 107.583573)
+		(mid 78.916437 64.98273)
+		(end 119.01 46.01)
 		(stroke
 			(width 0.15)
@@
 	)
 	(gr_arc
-		(start 103.015924 154.415864)
-		(mid 63.190164 95.289626)
-		(end 112.21 43.53)
+		(start 103.017401 154.41113)
+		(mid 63.38482 93.389316)
+		(end 116.01 43.14)
 		(stroke
 			(width 0.15)
@@
 	)
 	(segment
+		(start 119.01 46.01)
+		(end 119.25 45.77)
+		(width 0.15)
+		(layer "In2.Cu")
+		(net 12)
+	)
+	(segment
+		(start 119.25 45.7)
+		(end 119.25 41.65)
+		(width 0.15)
+		(layer "In2.Cu")
+		(net 12)
+	)
+	(segment
+		(start 119.25 45.77)
+		(end 119.25 45.7)
+		(width 0.15)
+		(layer "In2.Cu")
+		(net 12)
+	)
+	(segment
 		(start 72.788256 77.521797)
 		(end 72.720053 77.59)
@@
 	)
 	(segment
-		(start 115.7 46.7)
-		(end 115.72 46.7)
+		(start 119.53 46.52)
+		(end 119.75 46.3)
+		(width 0.15)
+		(layer "In2.Cu")
+		(net 20)
+	)
+	(segment
+		(start 119.75 46.3)
+		(end 119.75 41.6)
+		(width 0.15)
+		(layer "In2.Cu")
+		(net 20)
+	)
+	(segment
+		(start 119.5 46.52)
+		(end 119.53 46.52)
 		(width 0.15)
 		(layer "In2.Cu")
@@
 		(net 23)
 	)
+	(segment
+		(start 118.75 45.3)
+		(end 118.75 41.75)
+		(width 0.15)
+		(layer "In2.Cu")
+		(net 23)
+	)
+	(segment
+		(start 118.53 45.52)
+		(end 118.75 45.3)
+		(width 0.15)
+		(layer "In2.Cu")
+		(net 23)
+	)
+	(segment
+		(start 118.51 45.52)
+		(end 118.53 45.52)
+		(width 0.15)
+		(layer "In2.Cu")
+		(net 23)
+	)

Commit message: d
Routing:
- net PWM24: track 3.50 -> 8.49 mm
- net PWM32: track 2.26 -> 7.25 mm
- net PWM1: track 4.45 -> 9.30 mm
- net PWM2: track 2.31 -> 6.78 mm
- net PWM31: track 2.26 -> 6.68 mm
- net PWM23: track 3.29 -> 7.69 mm
- net PWM3: track 2.38 -> 6.27 mm
- net PWM30: track 2.26 -> 6.05 mm
- net PWM22: track 3.29 -> 7.07 mm
- net /REXT30: track 3.37 -> 0.00 mm
- net /REXT4: track 3.37 -> 0.00 mm
- net /REXT6: track 3.37 -> 0.00 mm
- net /REXT28: track 3.37 -> 0.00 mm
- net /REXT20: track 3.37 -> 0.00 mm
- net /REXT14: track 3.37 -> 0.00 mm
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
Commit message: m
Parts:
- removed the REF** at (118.7, 34.5)
- removed the REF** at (126.0, 39.5)
- removed the REF** at (107.9, 31.3)
- removed the REF** at (126.7, 37.7)
- removed the REF** at (128.7, 39.5)
- removed the REF** at (113.0, 37.8)
- removed the REF** at (122.9, 33.9)
- removed the REF** at (107.9, 33.9)
- removed the REF** at (125.4, 37.7)
- removed the REF** at (122.9, 36.5)
- removed the REF** at (107.9, 32.6)
- removed the REF** at (111.7, 37.8)
- removed the REF** at (114.3, 37.8)
- removed the REF** at (128.0, 37.7)
- removed the REF** at (110.4, 37.8)
- removed the REF** at (121.1, 33.2)
- removed the REF** at (106.1, 31.9)
- removed the REF** at (146.7, 32.5)
- removed the REF** at (121.1, 35.9)
- removed the REF** at (116.8, 33.9)
- removed the REF** at (122.9, 35.2)
- removed the REF** at (129.3, 37.7)
- removed the REF** at (148.5, 34.5)
- removed the REF** at (116.8, 32.6)
- removed the REF** at (116.8, 35.2)
- removed the REF** at (111.0, 39.5)
- removed the REF** at (118.7, 33.2)
- removed the REF** at (113.7, 39.5)
- removed the REF** at (122.9, 32.6)
- removed the REF** at (146.7, 35.1)
- removed the REF** at (148.5, 33.1)
- removed the REF** at (146.7, 33.8)
- removed the REF** at (107.9, 35.2)
- removed the REF** at (106.1, 34.5)
- added IC**: QFN40P400X400X100-33N-D, Library:QFN40P400X400X100-33N-D, F.Cu at (117.6, 21.2)
- added J**: ACZ11BR4E15FA120C, Library:ACZ11BR4E15FA120C, F.Cu at (143.1, 37.0)
- added REF**: C_0402_1005Metric, Capacitor_SMD:C_0402_1005Metric, F.Cu at (109.6, 28.2)
- added REF**: 694106301002, Library:694106301002, F.Cu at (132.7, 23.3)
- added REF**: R_0402_1005Metric, Resistor_SMD:R_0402_1005Metric, F.Cu at (102.1, 30.8)
- added REF**: MountingHole_2.2mm_M2_DIN965_Pad_TopBottom, MountingHole:MountingHole_2.2mm_M2_DIN965_Pad_TopBottom, F.Cu at (146.5, 18.5)
- added REF**: MountingHole_2.2mm_M2_DIN965_Pad_TopBottom, MountingHole:MountingHole_2.2mm_M2_DIN965_Pad_TopBottom, F.Cu at (93.5, 18.5)
- added REF**: R_0402_1005Metric, Resistor_SMD:R_0402_1005Metric, F.Cu at (115.3, 30.7)
- added REF**: C_0402_1005Metric, Capacitor_SMD:C_0402_1005Metric, F.Cu at (96.4, 28.3)
- added REF**10: R_0201_0603Metric, Resistor_SMD:R_0201_0603Metric, F.Cu at (108.9, 40.0)
- added REF**10: R_0201_0603Metric, Resistor_SMD:R_0201_0603Metric, F.Cu at (95.7, 40.1)
- added REF**11: R_0201_0603Metric, Resistor_SMD:R_0201_0603Metric, F.Cu at (109.5, 38.4)
- added REF**11: R_0201_0603Metric, Resistor_SMD:R_0201_0603Metric, F.Cu at (96.4, 38.5)
- added REF**13: R_0201_0603Metric, Resistor_SMD:R_0201_0603Metric, F.Cu at (110.2, 40.0)
- added REF**13: R_0201_0603Metric, Resistor_SMD:R_0201_0603Metric, F.Cu at (97.0, 40.1)
- added REF**14: R_0201_0603Metric, Resistor_SMD:R_0201_0603Metric, F.Cu at (110.8, 38.4)
- added REF**14: R_0201_0603Metric, Resistor_SMD:R_0201_0603Metric, F.Cu at (97.7, 38.5)
- added REF**15: R_0201_0603Metric, Resistor_SMD:R_0201_0603Metric, F.Cu at (111.5, 40.0)
- added REF**15: R_0201_0603Metric, Resistor_SMD:R_0201_0603Metric, F.Cu at (98.3, 40.1)
- added REF**17: R_0201_0603Metric, Resistor_SMD:R_0201_0603Metric, F.Cu at (112.1, 38.4)
- added REF**17: R_0201_0603Metric, Resistor_SMD:R_0201_0603Metric, F.Cu at (99.0, 38.5)
- added REF**18: R_0201_0603Metric, Resistor_SMD:R_0201_0603Metric, F.Cu at (112.8, 40.0)
- added REF**18: R_0201_0603Metric, Resistor_SMD:R_0201_0603Metric, F.Cu at (99.6, 40.1)
- added REF**19: R_0201_0603Metric, Resistor_SMD:R_0201_0603Metric, F.Cu at (113.4, 38.4)
- added REF**19: R_0201_0603Metric, Resistor_SMD:R_0201_0603Metric, F.Cu at (100.3, 38.5)
- added REF**21: R_0201_0603Metric, Resistor_SMD:R_0201_0603Metric, F.Cu at (114.1, 40.0)
- added REF**21: R_0201_0603Metric, Resistor_SMD:R_0201_0603Metric, F.Cu at (100.9, 40.1)
- added REF**22: R_0201_0603Metric, Resistor_SMD:R_0201_0603Metric, F.Cu at (101.6, 38.5)
- added REF**22: R_0201_0603Metric, Resistor_SMD:R_0201_0603Metric, F.Cu at (114.7, 38.4)
- added REF**23: R_0201_0603Metric, Resistor_SMD:R_0201_0603Metric, F.Cu at (102.2, 40.1)
- added REF**23: R_0201_0603Metric, Resistor_SMD:R_0201_0603Metric, F.Cu at (115.4, 40.0)
- added REF**3: R_0201_0603Metric, Resistor_SMD:R_0201_0603Metric, F.Cu at (92.5, 38.5)
- added REF**3: R_0201_0603Metric, Resistor_SMD:R_0201_0603Metric, F.Cu at (105.6, 38.4)
- added REF**5: R_0201_0603Metric, Resistor_SMD:R_0201_0603Metric, F.Cu at (93.1, 40.1)
- added REF**5: R_0201_0603Metric, Resistor_SMD:R_0201_0603Metric, F.Cu at (106.3, 40.0)
- added REF**6: R_0201_0603Metric, Resistor_SMD:R_0201_0603Metric, F.Cu at (93.8, 38.5)
- added REF**6: R_0201_0603Metric, Resistor_SMD:R_0201_0603Metric, F.Cu at (106.9, 38.4)
- added REF**7: R_0201_0603Metric, Resistor_SMD:R_0201_0603Metric, F.Cu at (107.6, 40.0)
- added REF**7: R_0201_0603Metric, Resistor_SMD:R_0201_0603Metric, F.Cu at (94.4, 40.1)
- added REF**9: R_0201_0603Metric, Resistor_SMD:R_0201_0603Metric, F.Cu at (108.2, 38.4)
- added REF**9: R_0201_0603Metric, Resistor_SMD:R_0201_0603Metric, F.Cu at (95.1, 38.5)
- moved U33 30.0 mm to (97.3, 32.6)
- moved U33 2.01 mm to (110.5, 32.5)
Routing:
- net SDA: track 0.00 -> 19.3 mm, vias 0 -> 2
- net Net-(U33-LED15): track 0.00 -> 19.0 mm
- net Net-(U33-LED1): track 0.00 -> 17.6 mm
- net SCL: track 0.00 -> 17.1 mm, vias 0 -> 2
- net Net-(U33-LED13): track 0.00 -> 16.0 mm
- net Net-(U33-LED0): track 0.00 -> 15.9 mm
- net Net-(U33-LED3): track 0.00 -> 14.6 mm
- net Net-(U33-LED14): track 0.00 -> 14.4 mm
- net Net-(U33-LED2): track 0.00 -> 12.9 mm
- net Net-(U33-LED12): track 0.00 -> 11.3 mm
- net Net-(U33-LED11): track 0.00 -> 10.9 mm
- net Net-(U33-LED7): track 0.00 -> 8.99 mm
- net Net-(U33-LED5): track 0.00 -> 8.95 mm
- net Net-(U33-LED9): track 0.00 -> 8.91 mm
- net Net-(U33-LED4): track 0.00 -> 7.76 mm
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- added copper zone on In2.Cu, net GND
Other:
- board size 115 x 115 mm -> 115 x 142.5 mm
