File: Hardware/Ring-Light v4/Ring-Light.kicad_pcb (KiCad board)
At the start: 4 copper layers, 115 x 142.5 mm, 184 parts, among them U1 NCR321PASX, U10 NCR321PASX, U11 NCR321PASX, U12 NCR321PASX, U13 NCR321PASX, U14 NCR321PASX, U15 NCR321PASX, U16 NCR321PASX, U17 NCR321PASX, U18 NCR321PASX, U19 NCR321PASX, U2 NCR321PASX, U20 NCR321PASX, U21 NCR321PASX, U22 NCR321PASX, U23 NCR321PASX, U24 NCR321PASX, U25 NCR321PASX, U26 NCR321PASX, U27 NCR321PASX, U28 NCR321PASX, U29 NCR321PASX, U3 NCR321PASX, U30 NCR321PASX, U31 NCR321PASX, U32 NCR321PASX, U33 PCA9685BS,118, U35 STM32WB50CGUx, U4 NCR321PASX, U5 NCR321PASX, U6 NCR321PASX, U7 NCR321PASX, U8 NCR321PASX, U9 NCR321PASX

Commit message: m
Parts:
- removed C33, C34: 0.1uF, Capacitor_SMD:C_0603_1608Metric
- removed R65, R66: 10k, Resistor_SMD:R_0402_1005Metric
- removed U35: STM32WB50CGUx, Package_DFN_QFN:QFN-48-1EP_7x7mm_P0.5mm_EP5.6x5.6mm

Commit message: m
Parts:
- removed the J** at (143.1, 37.0)
- removed the REF** at (102.1, 30.8)
- removed the REF** at (96.4, 28.3)
- removed the REF**10 at (95.7, 40.1)
- removed the REF**11 at (96.4, 38.5)
- removed the REF**13 at (97.0, 40.1)
- removed the REF**14 at (97.7, 38.5)
- removed the REF**15 at (98.3, 40.1)
- removed the REF**17 at (99.0, 38.5)
- removed the REF**18 at (99.6, 40.1)
- removed the REF**19 at (100.3, 38.5)
- removed the REF**21 at (100.9, 40.1)
- removed the REF**22 at (101.6, 38.5)
- removed the REF**23 at (102.2, 40.1)
- removed the REF**3 at (92.5, 38.5)
- removed the REF**5 at (93.1, 40.1)
- removed the REF**6 at (93.8, 38.5)
- removed the REF**7 at (94.4, 40.1)
- removed the REF**9 at (95.1, 38.5)
- removed the U33 at (97.3, 32.6)
- added J**: 2171750001, Library:2171750001, F.Cu at (145.1, 34.2)
- added REF**: CP_Elec_6.3x7.7, Capacitor_SMD:CP_Elec_6.3x7.7, F.Cu at (95.3, 41.5)
- added REF**: CP_Elec_6.3x7.7, Capacitor_SMD:CP_Elec_6.3x7.7, F.Cu at (104.6, 37.7)
- moved REF** 50.6 mm to (160.2, 27.9)
- moved REF**14 50.6 mm to (161.5, 38.1)
- moved REF**15 50.6 mm to (162.1, 39.7)
- moved REF**21 50.6 mm to (164.7, 39.7)
- moved REF**22 50.6 mm to (165.4, 38.1)
- moved REF**7 50.6 mm to (158.2, 39.7)
- moved REF**9 50.6 mm to (158.9, 38.1)
- moved U33 50.6 mm to (161.1, 32.2)
- moved REF** 50.6 mm to (165.9, 30.4)
- moved REF**11 50.6 mm to (160.2, 38.1)
- moved REF**13 50.6 mm to (160.8, 39.7)
- moved REF**18 50.6 mm to (163.4, 39.7)
- moved REF**19 50.6 mm to (164.1, 38.1)
- moved REF**5 50.6 mm to (156.9, 39.7)
- moved REF**6 50.6 mm to (157.6, 38.1)
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Routing:
- net SDA: track 19.3 -> 2.56 mm, vias 2 -> 1
- net SCL: track 17.1 -> 1.05 mm, vias 2 -> 1
- net Net-(U33-LED15): track 19.0 -> 9.52 mm
- net Net-(U33-LED1): track 17.6 -> 8.79 mm
- net Net-(U33-LED13): track 16.0 -> 8.01 mm
- net Net-(U33-LED0): track 15.9 -> 7.94 mm
- net Net-(U33-LED3): track 14.6 -> 7.28 mm
- net Net-(U33-LED14): track 14.4 -> 7.19 mm
- net Net-(U33-LED2): track 12.9 -> 6.43 mm
- net Net-(U33-LED12): track 11.3 -> 5.66 mm
- net Net-(U33-LED11): track 10.9 -> 5.46 mm
- net Net-(U33-LED7): track 8.99 -> 4.49 mm
- net Net-(U33-LED5): track 8.95 -> 4.47 mm
- net Net-(U33-LED9): track 8.91 -> 4.45 mm
- net Net-(U33-LED4): track 7.76 -> 3.88 mm
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Other:
- outline, holes or cut-outs redrawn

Commit message: d
Parts:
- removed J**: 2171750001, Library:2171750001
- added REF**: R_0402_1005Metric, Resistor_SMD:R_0402_1005Metric, F.Cu at (135.3, 32.5)
- added REF**: USB_Micro-B_Molex-105017-0001, Connector_USB:USB_Micro-B_Molex-105017-0001, F.Cu at (146.3, 27.5)
- added REF**: C_0402_1005Metric, Capacitor_SMD:C_0402_1005Metric, F.Cu at (129.7, 30.0)
- added REF**10: R_0201_0603Metric, Resistor_SMD:R_0201_0603Metric, F.Cu at (128.9, 41.8)
- added REF**11: R_0201_0603Metric, Resistor_SMD:R_0201_0603Metric, F.Cu at (129.6, 40.2)
- added REF**13: R_0201_0603Metric, Resistor_SMD:R_0201_0603Metric, F.Cu at (130.2, 41.8)
- added REF**14: R_0201_0603Metric, Resistor_SMD:R_0201_0603Metric, F.Cu at (130.9, 40.2)
- added REF**15: R_0201_0603Metric, Resistor_SMD:R_0201_0603Metric, F.Cu at (131.6, 41.8)
- added REF**17: R_0201_0603Metric, Resistor_SMD:R_0201_0603Metric, F.Cu at (132.2, 40.2)
- added REF**18: R_0201_0603Metric, Resistor_SMD:R_0201_0603Metric, F.Cu at (132.8, 41.8)
- added REF**19: R_0201_0603Metric, Resistor_SMD:R_0201_0603Metric, F.Cu at (133.5, 40.2)
- added REF**21: R_0201_0603Metric, Resistor_SMD:R_0201_0603Metric, F.Cu at (134.2, 41.8)
- added REF**22: R_0201_0603Metric, Resistor_SMD:R_0201_0603Metric, F.Cu at (134.8, 40.2)
- added REF**23: R_0201_0603Metric, Resistor_SMD:R_0201_0603Metric, F.Cu at (135.4, 41.8)
- added REF**3: R_0201_0603Metric, Resistor_SMD:R_0201_0603Metric, F.Cu at (125.7, 40.2)
- added REF**5: R_0201_0603Metric, Resistor_SMD:R_0201_0603Metric, F.Cu at (126.3, 41.8)
- added REF**6: R_0201_0603Metric, Resistor_SMD:R_0201_0603Metric, F.Cu at (127.0, 40.2)
- added REF**7: R_0201_0603Metric, Resistor_SMD:R_0201_0603Metric, F.Cu at (127.7, 41.8)
- added REF**9: R_0201_0603Metric, Resistor_SMD:R_0201_0603Metric, F.Cu at (128.3, 40.2)
- added U33: PCA9685BS,118, Library:QFN65P600X600X100-29N-D, F.Cu at (130.6, 34.3)
- moved REF**10 18.7 mm to (141.4, 44.7)
- moved REF**11 18.7 mm to (142.1, 43.1)
- moved REF**13 18.7 mm to (142.8, 44.7)
- moved REF**14 18.7 mm to (143.4, 43.1)
- moved REF**15 18.7 mm to (144.1, 44.7)
- moved REF**17 18.7 mm to (144.7, 43.1)
- moved REF**18 18.7 mm to (145.3, 44.7)
- moved REF**19 18.7 mm to (146.0, 43.1)
- moved REF**21 18.7 mm to (146.7, 44.7)
- moved REF**22 18.7 mm to (147.3, 43.1)
- moved REF**23 18.7 mm to (147.9, 44.7)
- moved REF**3 18.7 mm to (138.2, 43.1)
- moved REF**5 18.7 mm to (138.8, 44.7)
- moved REF**6 18.7 mm to (139.5, 43.1)
- moved REF**7 18.7 mm to (140.2, 44.7)
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Routing:
- net Net-(U33-LED15): track 9.52 -> 19.0 mm
- net Net-(U33-LED1): track 8.79 -> 17.6 mm
- net Net-(U33-LED13): track 8.01 -> 16.0 mm
- net Net-(U33-LED0): track 7.94 -> 15.9 mm
- net Net-(U33-LED3): track 7.28 -> 14.6 mm
- net Net-(U33-LED14): track 7.19 -> 14.4 mm
- net Net-(U33-LED2): track 6.43 -> 12.9 mm
- net Net-(U33-LED12): track 5.66 -> 11.3 mm
- net Net-(U33-LED11): track 5.46 -> 10.9 mm
- net Net-(U33-LED7): track 4.49 -> 8.99 mm
- net Net-(U33-LED5): track 4.47 -> 8.95 mm
- net Net-(U33-LED9): track 4.45 -> 8.91 mm
- net Net-(U33-LED4): track 3.88 -> 7.76 mm
- net Net-(U33-LED6): track 2.87 -> 5.75 mm
- net Net-(U33-LED10): track 2.85 -> 5.71 mm
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
Commit message: m
Parts:
- removed the IC** at (120.8, 33.1)
- added IC**: CP2102NA02GQFN20, Library:CP2102NA02GQFN20, F.Cu at (137.2, 25.5)
- added REF**: PSON50P300X200X60-9N, Library:PSON50P300X200X60-9N, F.Cu at (112.6, 30.7)
- added REF**: QFN-32-1EP_7x7mm_P0.65mm_EP4.7x4.7mm, Package_DFN_QFN:QFN-32-1EP_7x7mm_P0.65mm_EP4.7x4.7mm, F.Cu at (119.5, 30.7)
- added REF**: WSON-10-1EP_2x3mm_P0.5mm_EP0.84x2.4mm_ThermalVias, Package_SON:WSON-10-1EP_2x3mm_P0.5mm_EP0.84x2.4mm_ThermalVias, F.Cu at (113.7, 37.9)
- moved REF** 1.88 mm to (103.3, 23.3)
- moved REF**11 0.64 mm to (130.2, 40.1)
- moved REF**17 0.64 mm to (132.8, 40.1)
- moved REF** 0.64 mm to (136.0, 32.5)
- moved REF**10 0.64 mm to (129.6, 41.8)
- moved REF**18 0.64 mm to (133.5, 41.8)
- moved REF**23 0.64 mm to (136.1, 41.8)
- moved REF**3 0.64 mm to (126.3, 40.1)
- moved REF**6 0.64 mm to (127.6, 40.1)
- moved REF**5 0.64 mm to (127.0, 41.8)
- moved REF**14 0.64 mm to (131.5, 40.1)
- moved REF**19 0.64 mm to (134.1, 40.1)
- moved REF**22 0.64 mm to (135.4, 40.1)
- moved REF**9 0.64 mm to (128.9, 40.1)
- moved REF** 0.64 mm to (130.3, 29.9)
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
Commit message: d
Parts:
- added J**: 2002112100010C4LF, Library:2002112100010C4LF, F.Cu at (117.0, 21.3)

Commit message: m
Parts:
- removed the REF** at (136.0, 32.5)
- removed the REF** at (147.8, 35.4)
- removed the REF** at (146.3, 27.5)
- removed the REF** at (119.5, 30.7)
- removed the REF** at (142.2, 32.9)
- removed the REF** at (130.3, 29.9)
- removed REF**10 (x2), REF**11 (x2), REF**13 (x2), REF**14 (x2), REF**15 (x2), REF**17 (x2), REF**18 (x2), REF**19 (x2), REF**21 (x2), REF**22 (x2), REF**23 (x2), REF**3 (x2), REF**5 (x2), REF**6 (x2), REF**7 (x2), REF**9 (x2): R_0201_0603Metric, Resistor_SMD:R_0201_0603Metric
- added C20: 1.0uF, Capacitor_SMD:C_0402_1005Metric, F.Cu at (114.2, 52.2)
- added C22: 12pF, Capacitor_SMD:C_0402_1005Metric, F.Cu at (110.5, 45.6)
- added C23: DNM, Capacitor_SMD:C_0402_1005Metric, F.Cu at (116.0, 38.6)
- added C24: 12pF, Capacitor_SMD:C_0402_1005Metric, F.Cu at (107.9, 39.3)
- added C25: 12pF, Capacitor_SMD:C_0402_1005Metric, F.Cu at (109.9, 39.3)
- added C27: 1.2pF, Capacitor_SMD:C_0402_1005Metric, F.Cu at (106.1, 46.0)
- added C28: DNM, Capacitor_SMD:C_0402_1005Metric, F.Cu at (103.3, 52.9)
- added C29: DNM, Capacitor_SMD:C_0402_1005Metric, F.Cu at (107.4, 49.7)
- added C31: 100nF, Capacitor_SMD:C_0402_1005Metric, F.Cu at (111.0, 50.0)
- added C7: 0.1uF, Capacitor_SMD:C_0402_1005Metric, F.Cu at (116.3, 51.7)
- added C8: 0.1uF, Capacitor_SMD:C_0402_1005Metric, F.Cu at (114.2, 51.1)
- added D33: TPD1E10B06DPYR, Library:TPD1E10B06DPYR, F.Cu at (118.6, 59.2)
- added D34: TPD1E10B06DPYR, Library:TPD1E10B06DPYR, F.Cu at (118.6, 56.1)
- added D35: TPD1E10B06DPYR, Library:TPD1E10B06DPYR, F.Cu at (118.6, 53.7)
- added D36: LTST-C170YKT, Diode_SMD:D_0402_1005Metric, F.Cu at (114.4, 59.3)
- added D37: LTST-C170YKT, Diode_SMD:D_0402_1005Metric, F.Cu at (113.2, 59.3)
- added J2: 1017457000B11LF, Library:1017457000B11LF, F.Cu at (124.5, 54.9)
- added J3: U.FL-R-SMT-1_80, Library:UFLRSMT180, F.Cu at (124.1, 42.8)
- added L3: 2nH, Inductor_SMD:L_0402_1005Metric, F.Cu at (107.6, 45.6)
- added L7: 15nH, Inductor_SMD:L_0402_1005Metric, F.Cu at (107.2, 44.3)
- added R100: 1k, Resistor_SMD:R_0402_1005Metric, F.Cu at (112.1, 52.2)
- added R102: 1k, Resistor_SMD:R_0402_1005Metric, F.Cu at (115.6, 59.3)
- added R103: 1k, Resistor_SMD:R_0402_1005Metric, F.Cu at (112.0, 59.3)
- added R105: 100k, Resistor_SMD:R_0402_1005Metric, F.Cu at (109.4, 55.5)
- added R106: 100k, Resistor_SMD:R_0402_1005Metric, F.Cu at (110.6, 55.5)
- added R107: 1k, Resistor_SMD:R_0402_1005Metric, F.Cu at (117.4, 59.1)
- added R109: 10k, Resistor_SMD:R_0402_1005Metric, F.Cu at (115.6, 47.8)
- added R110: 2.2k, Resistor_SMD:R_0402_1005Metric, F.Cu at (115.6, 48.9)
- added R111: DNM, Resistor_SMD:R_0402_1005Metric, F.Cu at (118.0, 45.6)
- added R112: 0, Resistor_SMD:R_0402_1005Metric, F.Cu at (116.5, 45.1)
- added R113: 0, Resistor_SMD:R_0402_1005Metric, F.Cu at (116.5, 40.1)
- added R114: 1k, Resistor_SMD:R_0402_1005Metric, F.Cu at (118.1, 50.7)
- added REF**: MountingHole_2.2mm_M2_DIN965_Pad_TopBottom, MountingHole:MountingHole_2.2mm_M2_DIN965_Pad_TopBottom, F.Cu at (125.1, 66.1)
- added REF**: C14, Capacitor_SMD:C_0402_1005Metric, F.Cu at (109.1, 45.1)
- added REF**: MountingHole_2.2mm_M2_DIN965_Pad_TopBottom, MountingHole:MountingHole_2.2mm_M2_DIN965_Pad_TopBottom, F.Cu at (63.1, 66.1)
- added U39: CC2640R2FRSMR, Library:QFN40P400X400X100-33N-D, F.Cu at (102.7, 44.2)
- added Y1: 32.768kHz, Library:FC135327680KAAG0, F.Cu at (108.9, 41.1)
- added Y2: 24MHz, Library:TSX-3225, F.Cu at (105.9, 51.8)
- U37: renamed from IC**; value CP2102NA02GQFN20 -> CP2102N-A02-GQFN20R
- U38: renamed from REF**; value PSON50P300X200X60-9N -> W25X40CLUXIG_TR
- moved U33 106.6 mm to (39.0, 60.3)
- moved U33 87.6 mm to (47.5, 60.3)
- moved J** 70.7 mm to (51.1, 46.7), turned to 90 degrees
- moved U37 37.7 mm to (114.2, 55.4), turned to 180 degrees
- moved REF** 37.6 mm to (68.1, 46.7), turned to 180 degrees
- moved REF** 37.1 mm to (79.9, 53.2)
- moved REF** 34.4 mm to (62.6, 33.6)
- moved R31 31.9 mm to (80.8, 169.3)
- moved R61 31.9 mm to (117.1, 71.7)
- moved D12 31.9 mm to (59.2, 142.0)
- moved D22 31.9 mm to (129.0, 142.0)
- moved D23 31.9 mm to (132.9, 134.7)
- moved D29 31.9 mm to (123.8, 89.0)
- moved D3 31.9 mm to (78.0, 79.9)
- moved R3 31.9 mm to (87.1, 66.8)
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- renumbered REF** to J1
Connections:
- net /OUT1 renamed /LEDs_1-16/OUT1
- net /OUT10 renamed /LEDs_1-16/OUT10
- net /OUT11 renamed /LEDs_1-16/OUT11
- net /OUT12 renamed /LEDs_1-16/OUT12
- net /OUT13 renamed /LEDs_1-16/OUT13
- net /OUT14 renamed /LEDs_1-16/OUT14
- net /OUT15 renamed /LEDs_1-16/OUT15
- net /OUT16 renamed /LEDs_1-16/OUT16
- net /OUT17 renamed /LEDs_17-32/OUT17
- net /OUT18 renamed /LEDs_17-32/OUT18
- net /OUT19 renamed /LEDs_17-32/OUT19
- net /OUT2 renamed /LEDs_1-16/OUT2
- net /OUT20 renamed /LEDs_17-32/OUT20
- net /OUT21 renamed /LEDs_17-32/OUT21
- net /OUT22 renamed /LEDs_17-32/OUT22
- net /OUT23 renamed /LEDs_17-32/OUT23
- net /OUT24 renamed /LEDs_17-32/OUT24
- net /OUT25 renamed /LEDs_17-32/OUT25
- net /OUT26 renamed /LEDs_17-32/OUT26
- net /OUT27 renamed /LEDs_17-32/OUT27
- net /OUT28 renamed /LEDs_17-32/OUT28
- net /OUT29 renamed /LEDs_17-32/OUT29
- net /OUT3 renamed /LEDs_1-16/OUT3
- net /OUT30 renamed /LEDs_17-32/OUT30
- net /OUT31 renamed /LEDs_17-32/OUT31
- net /OUT32 renamed /LEDs_17-32/OUT32
- net /OUT4 renamed /LEDs_1-16/OUT4
- net /OUT5 renamed /LEDs_1-16/OUT5
- net /OUT6 renamed /LEDs_1-16/OUT6
- net /OUT7 renamed /LEDs_1-16/OUT7
- net /OUT8 renamed /LEDs_1-16/OUT8
- net /OUT9 renamed /LEDs_1-16/OUT9
- net /REXT1 renamed /LEDs_1-16/REXT1
- net /REXT10 renamed /LEDs_1-16/REXT10
- net /REXT11 renamed /LEDs_1-16/REXT11
- net /REXT12 renamed /LEDs_1-16/REXT12
- net /REXT13 renamed /LEDs_1-16/REXT13
- net /REXT14 renamed /LEDs_1-16/REXT14
- net /REXT15 renamed /LEDs_1-16/REXT15
- net /REXT16 renamed /LEDs_1-16/REXT16
- net /REXT17 renamed /LEDs_17-32/REXT17
- net /REXT18 renamed /LEDs_17-32/REXT18
- net /REXT19 renamed /LEDs_17-32/REXT19
- net /REXT2 renamed /LEDs_1-16/REXT2
- net /REXT20 renamed /LEDs_17-32/REXT20
- net /REXT21 renamed /LEDs_17-32/REXT21
- net /REXT22 renamed /LEDs_17-32/REXT22
- net /REXT23 renamed /LEDs_17-32/REXT23
- net /REXT24 renamed /LEDs_17-32/REXT24
- net /REXT25 renamed /LEDs_17-32/REXT25
- net /REXT26 renamed /LEDs_17-32/REXT26
- net /REXT27 renamed /LEDs_17-32/REXT27
- net /REXT28 renamed /LEDs_17-32/REXT28
- net /REXT29 renamed /LEDs_17-32/REXT29
- net /REXT3 renamed /LEDs_1-16/REXT3
- net /REXT30 renamed /LEDs_17-32/REXT30
- net /REXT31 renamed /LEDs_17-32/REXT31
- net /REXT32 renamed /LEDs_17-32/REXT32
- net /REXT4 renamed /LEDs_1-16/REXT4
- net /REXT5 renamed /LEDs_1-16/REXT5
- net /REXT6 renamed /LEDs_1-16/REXT6
- net /REXT7 renamed /LEDs_1-16/REXT7
- net /REXT8 renamed /LEDs_1-16/REXT8
- net /REXT9 renamed /LEDs_1-16/REXT9
- net PWM1 renamed /LEDs_1-16/PWM1
- net PWM10 renamed /LEDs_1-16/PWM10
- net PWM11 renamed /LEDs_1-16/PWM11
- net PWM12 renamed /LEDs_1-16/PWM12
- net PWM13 renamed /LEDs_1-16/PWM13
- net PWM14 renamed /LEDs_1-16/PWM14
- net PWM15 renamed /LEDs_1-16/PWM15
- net PWM16 renamed /LEDs_1-16/PWM16
- net PWM17 renamed /LEDs_17-32/PWM17
- net PWM18 renamed /LEDs_17-32/PWM18
- net PWM19 renamed /LEDs_17-32/PWM19
- net PWM2 renamed /LEDs_1-16/PWM2
- net PWM20 renamed /LEDs_17-32/PWM20
- net PWM21 renamed /LEDs_17-32/PWM21
- net PWM22 renamed /LEDs_17-32/PWM22
- net PWM23 renamed /LEDs_17-32/PWM23
- net PWM24 renamed /LEDs_17-32/PWM24
- net PWM25 renamed /LEDs_17-32/PWM25
- net PWM26 renamed /LEDs_17-32/PWM26
- net PWM27 renamed /LEDs_17-32/PWM27
- net PWM28 renamed /LEDs_17-32/PWM28
- net PWM29 renamed /LEDs_17-32/PWM29
- net PWM3 renamed /LEDs_1-16/PWM3
- net PWM30 renamed /LEDs_17-32/PWM30
- net PWM31 renamed /LEDs_17-32/PWM31
- net PWM32 renamed /LEDs_17-32/PWM32
- net PWM4 renamed /LEDs_1-16/PWM4
- net PWM5 renamed /LEDs_1-16/PWM5
- net PWM6 renamed /LEDs_1-16/PWM6
- net PWM7 renamed /LEDs_1-16/PWM7
- net PWM8 renamed /LEDs_1-16/PWM8
- net PWM9 renamed /LEDs_1-16/PWM9
- net PWM_EN renamed /MCU/PWM_EN
- net SCL renamed /MCU/SCL
- net SDA renamed /MCU/SDA
- J1 pad 1: (no net) -> GND
- J1 pad 2: (no net) -> +12V
- J1 pad 3: (no net) -> unconnected-(J1-Pad3)
- U37 pad 1: (no net) -> unconnected-(U37-GPIO.1_/_RS485-Pad1)
- U37 pad 10: (no net) -> unconnected-(U37-NC-Pad10)
- U37 pad 11: (no net) -> unconnected-(U37-~{SUSPEND}-Pad11)
- U37 pad 12: (no net) -> GND
- U37 pad 13: (no net) -> unconnected-(U37-WAKEUP-Pad13)
- U37 pad 14: (no net) -> unconnected-(U37-SUSPEND-Pad14)
- U37 pad 15: (no net) -> unconnected-(U37-CTS-Pad15)
- U37 pad 16: (no net) -> unconnected-(U37-RTS-Pad16)
- U37 pad 17: (no net) -> Net-(U37-RXD)
- U37 pad 18: (no net) -> Net-(U37-TXD)
- U37 pad 19: (no net) -> Net-(U37-GPIO.3_/_RXT)
- U37 pad 2: (no net) -> unconnected-(U37-GPIO.0_/_CLK-Pad2)
- U37 pad 20: (no net) -> Net-(U37-GPIO.2_/_TXT)
- U37 pad 21: (no net) -> GND
- U37 pad 3: (no net) -> GND
- U37 pad 4: (no net) -> /Interface/D+
- U37 pad 5: (no net) -> /Interface/D-
- U37 pad 6: (no net) -> USB_VDD
- U37 pad 7: (no net) -> /Interface/<NO NET>
- U37 pad 8: (no net) -> /Interface/<NO NET>
- U37 pad 9: (no net) -> Net-(U37-~{RST})
- U38 pad 1: (no net) -> FLASH_CS
- U38 pad 2: (no net) -> MISO
- U38 pad 3: (no net) -> Net-(U38-~{WP})
- U38 pad 4: (no net) -> GND
- U38 pad 5: (no net) -> MOSI
- U38 pad 6: (no net) -> SCLK
- U38 pad 7: (no net) -> Net-(U38-~{HOLD})
- U38 pad 8: (no net) -> +3.3V
- U38 pad 9: (no net) -> GND
Routing:
- net FLASH_CS: track 0.00 -> 19.9 mm, vias 0 -> 2
- net USB_VDD: track 0.00 -> 19.9 mm, vias 0 -> 4
- net Net-(U33-LED15): track 19.0 -> 0.00 mm
- net /Interface/<NO NET>: track 0.00 -> 18.1 mm, vias 0 -> 3
- net SCLK: track 0.00 -> 17.8 mm, vias 0 -> 2
- net Net-(U33-LED1): track 17.6 -> 0.00 mm
- net Net-(U33-LED13): track 16.0 -> 0.00 mm
- net MISO: track 0.00 -> 15.9 mm, vias 0 -> 2
- net Net-(U33-LED0): track 15.9 -> 0.00 mm
- net Net-(U33-LED3): track 14.6 -> 0.00 mm
- net Net-(U33-LED14): track 14.4 -> 0.00 mm
- net Net-(U33-LED2): track 12.9 -> 0.00 mm
- net Net-(U33-LED12): track 11.3 -> 0.00 mm
- net Net-(U33-LED11): track 10.9 -> 0.00 mm
- net /Interface/D-: track 0.00 -> 10.3 mm, vias 0 -> 2
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- added copper zone on F.Cu, net (none)
Other:
- board size 115 x 142.5 mm -> 115 x 146.1 mm

Commit message: d
Parts:
- added IC**: QFN50P700X700X100-49N-D, Library:QFN50P700X700X100-49N-D, F.Cu at (139.4, 47.6)
