File: Hardware/Ring-Light v4/Ring-Light.kicad_pcb (KiCad board)
At the start: 4 copper layers, 115 x 146.1 mm, 186 parts, among them J1 694106301002, J2 1017457000B11LF, J3 U.FL-R-SMT-1_80, U1 NCR321PASX, U10 NCR321PASX, U11 NCR321PASX, U12 NCR321PASX, U13 NCR321PASX, U14 NCR321PASX, U15 NCR321PASX, U16 NCR321PASX, U17 NCR321PASX, U18 NCR321PASX, U19 NCR321PASX, U2 NCR321PASX, U20 NCR321PASX, U21 NCR321PASX, U22 NCR321PASX, U23 NCR321PASX, U24 NCR321PASX, U25 NCR321PASX, U26 NCR321PASX, U27 NCR321PASX, U28 NCR321PASX, U29 NCR321PASX, U3 NCR321PASX, U30 NCR321PASX, U31 NCR321PASX, U32 NCR321PASX, U33 PCA9685BS,118, U37 CP2102N-A02-GQFN20R, U38 W25X40CLUXIG_TR, U39 CC2640R2FRSMR, U4 NCR321PASX, U5 NCR321PASX, U6 NCR321PASX, U7 NCR321PASX, U8 NCR321PASX, U9 NCR321PASX, Y1 32.768kHz, Y2 24MHz

Commit message: m
Parts:
- removed the U39 at (102.7, 44.2)
- added C10: 100nF, Capacitor_SMD:C_0402_1005Metric, F.Cu at (95.5, 35.9)
- added C13: 100nF, Capacitor_SMD:C_0402_1005Metric, F.Cu at (104.5, 48.5)
- added C15: 100nF, Capacitor_SMD:C_0402_1005Metric, F.Cu at (105.7, 38.1)
- added R104: 100k, Resistor_SMD:R_0402_1005Metric, F.Cu at (95.4, 33.9)
- C14: renamed from REF**; value C14 -> 1.2pF
- U39: renamed from IC**; value QFN50P700X700X100-49N-D -> CC2640R2FRGZR
- moved U33 48.7 mm to (95.7, 53.2)
- moved U33 47.1 mm to (85.5, 53.1)
- moved J4 39.4 mm to (90.3, 42.8), turned to -90 degrees
- moved U39 38.6 mm to (101.2, 42.8), turned to 180 degrees
- moved R109 12.3 mm to (107.1, 56.6), turned to 90 degrees
- moved U38 12.3 mm to (104.3, 57.8)
- moved C31 12.2 mm to (103.6, 59.7)
- moved R110 10.8 mm to (108.2, 56.6), turned to 90 degrees
- moved C28 0.70 mm to (107.0, 50.2)
- moved C29 0.70 mm to (102.9, 53.4)
- moved Y2 0.70 mm to (105.5, 52.4), turned to 180 degrees
- moved Y1 0.12 mm to (109.0, 41.0)
- turned C14 to -90 degrees
- renumbered C25 to C24, C24 to C25, C29 to C28, C28 to C29, J** to J4
Connections:
- net /Interface/<NO NET> renamed /MCU/<NO NET>
- net /Interface/D+ renamed /MCU/D+
- net /Interface/D- renamed /MCU/D-
- net /Interface/LED_RX renamed /MCU/LED_RX
- net /Interface/LED_TX renamed /MCU/LED_TX
- C14 pad 1: (no net) -> GND
- C14 pad 2: (no net) -> Net-(C14-Pad2)
- J4 pad 1: (no net) -> +3.3V
- J4 pad 10: (no net) -> MCU_RESET
- J4 pad 2: (no net) -> JTAG_TMS
- J4 pad 3: (no net) -> GND
- J4 pad 4: (no net) -> JTAG_TCK
- J4 pad 5: (no net) -> GND
- J4 pad 6: (no net) -> JTAG_TDO
- J4 pad 7: (no net) -> unconnected-(J4-Pin_7-Pad7)
- J4 pad 8: (no net) -> JTAG_TDI
- J4 pad 9: (no net) -> GND
- R105 pad 2: /Interface/USB_TXD -> /MCU/RXD
- R106 pad 2: /Interface/USB_RXD -> /MCU/TXD
- U39 pad 1: (no net) -> Net-(U39-RF_P)
- U39 pad 10: (no net) -> /MCU/SDA
- U39 pad 11: (no net) -> unconnected-(U39-DIO_6-Pad11)
- U39 pad 12: (no net) -> unconnected-(U39-DIO_7-Pad12)
- U39 pad 13: (no net) -> VDDS
- U39 pad 14: (no net) -> MISO
- U39 pad 15: (no net) -> MOSI
- U39 pad 16: (no net) -> SCLK
- U39 pad 17: (no net) -> unconnected-(U39-DIO_11-Pad17)
- U39 pad 18: (no net) -> unconnected-(U39-DIO_12-Pad18)
- U39 pad 19: (no net) -> unconnected-(U39-DIO_13-Pad19)
- U39 pad 2: (no net) -> Net-(U39-RF_N)
- U39 pad 20: (no net) -> unconnected-(U39-DIO_14-Pad20)
- U39 pad 21: (no net) -> unconnected-(U39-DIO_15-Pad21)
- U39 pad 22: (no net) -> VDDS
- U39 pad 23: (no net) -> Net-(U39-DCOUPL)
- U39 pad 24: (no net) -> JTAG_TMS
- U39 pad 25: (no net) -> JTAG_TCK
- U39 pad 26: (no net) -> JTAG_TDO
- U39 pad 27: (no net) -> JTAG_TDI
- U39 pad 28: (no net) -> /MCU/RTS
- U39 pad 29: (no net) -> /MCU/CTS
- U39 pad 3: (no net) -> Net-(U39-X32K_Q1)
- U39 pad 30: (no net) -> FLASH_CS
- U39 pad 31: (no net) -> unconnected-(U39-DIO_21-Pad31)
- U39 pad 32: (no net) -> unconnected-(U39-DIO_22-Pad32)
- U39 pad 33: (no net) -> DCDC_SW
- U39 pad 34: (no net) -> VDDS
- U39 pad 35: (no net) -> MCU_RESET
- U39 pad 36: (no net) -> unconnected-(U39-DIO_23-Pad36)
- U39 pad 37: (no net) -> unconnected-(U39-DIO_24-Pad37)
- U39 pad 38: (no net) -> unconnected-(U39-DIO_25-Pad38)
- U39 pad 39: (no net) -> unconnected-(U39-DIO_26-Pad39)
- U39 pad 4: (no net) -> Net-(U39-X32K_Q2)
- U39 pad 40: (no net) -> unconnected-(U39-DIO_27-Pad40)
- U39 pad 41: (no net) -> unconnected-(U39-DIO_28-Pad41)
- U39 pad 42: (no net) -> unconnected-(U39-DIO_29-Pad42)
- U39 pad 43: (no net) -> unconnected-(U39-DIO_30-Pad43)
- U39 pad 44: (no net) -> VDDS
- U39 pad 45: (no net) -> VDDR
- U39 pad 46: (no net) -> Net-(U39-X24M_N)
- U39 pad 47: (no net) -> Net-(U39-X24M_P)
- U39 pad 48: (no net) -> VDDR
- U39 pad 49: (no net) -> GND
- U39 pad 5: (no net) -> /MCU/PWM_EN
- U39 pad 6: (no net) -> unconnected-(U39-DIO_1-Pad6)
- U39 pad 7: (no net) -> /MCU/RXD
- U39 pad 8: (no net) -> /MCU/TXD
- U39 pad 9: (no net) -> /MCU/SCL
- Y2 pad 1: Net-(U39-X24M_N) -> Net-(U39-X24M_P)
- Y2 pad 3: Net-(U39-X24M_P) -> Net-(U39-X24M_N)
Routing:
- net FLASH_CS: track 19.9 -> 35.2 mm
- net MOSI: track 10.1 -> 24.4 mm
- net SCLK: track 17.8 -> 29.0 mm
- net MISO: track 15.9 -> 23.9 mm
- net JTAG_TDI: track 0.00 -> 6.69 mm
- net JTAG_TMS: track 0.00 -> 6.51 mm
- net JTAG_TDO: track 0.00 -> 6.37 mm
- net JTAG_TCK: track 0.00 -> 6.05 mm
- net MCU_RESET: track 0.00 -> 5.56 mm
- net +3.3V: track 0.00 -> 2.23 mm
- net VDDS: track 0.00 -> 2.18 mm
- net VDDR: track 0.00 -> 1.96 mm
- net Net-(U39-X32K_Q2): track 6.06 -> 6.91 mm

Commit message: d
Parts:
- added C1: 0.1uF, Capacitor_SMD:C_0603_1608Metric, F.Cu at (177.8, 34.5)
- added C11: 10uF, Capacitor_SMD:C_0402_1005Metric, F.Cu at (187.6, 26.0)
- added C12: 100nF, Capacitor_SMD:C_0402_1005Metric, F.Cu at (141.9, 27.0)
- added C16: 100nF, Capacitor_SMD:C_0402_1005Metric, F.Cu at (99.9, 38.1)
- added C17: 100nF, Capacitor_SMD:C_0402_1005Metric, F.Cu at (144.1, 20.6)
- added C18: 10uF, Capacitor_SMD:C_0402_1005Metric, F.Cu at (95.6, 44.5)
- added C19: 100nF, Capacitor_SMD:C_0402_1005Metric, F.Cu at (144.4, 15.4)
- added C2: 0.1uF, Capacitor_SMD:C_0603_1608Metric, F.Cu at (177.8, 37.0)
- added C21: 1uF, Capacitor_SMD:C_0402_1005Metric, F.Cu at (98.0, 38.1)
- added C5: 0.1uF, Capacitor_SMD:C_0603_1608Metric, F.Cu at (166.2, 46.1)
- added C6: 22uF, Capacitor_SMD:C_0603_1608Metric, F.Cu at (166.2, 48.6)
- added FL1: BLM18HE152SN1, Inductor_SMD:L_0603_1608Metric, F.Cu at (191.0, 32.2)
- added R101: 100k, Resistor_SMD:R_0402_1005Metric, F.Cu at (190.5, 26.0)
- added R108: 10k, Resistor_SMD:R_0402_1005Metric, F.Cu at (190.5, 28.0)
- added R115: 100k, Resistor_SMD:R_0402_1005Metric, F.Cu at (190.5, 29.9)
- added R65: 10k, Resistor_SMD:R_0402_1005Metric, F.Cu at (165.6, 26.0)
- added R66: 100, Resistor_SMD:R_0402_1005Metric, F.Cu at (165.6, 28.0)
- added R67: 100, Resistor_SMD:R_0402_1005Metric, F.Cu at (165.6, 29.9)
- added R68: 100, Resistor_SMD:R_0402_1005Metric, F.Cu at (165.6, 31.9)
- added R69: 100, Resistor_SMD:R_0402_1005Metric, F.Cu at (165.6, 33.9)
- added R70: 100, Resistor_SMD:R_0402_1005Metric, F.Cu at (165.6, 35.9)
- added R71: 100, Resistor_SMD:R_0402_1005Metric, F.Cu at (165.6, 37.9)
- added R72: 100, Resistor_SMD:R_0402_1005Metric, F.Cu at (165.6, 39.9)
- added R73: 100, Resistor_SMD:R_0402_1005Metric, F.Cu at (165.6, 41.9)
- added R74: 100, Resistor_SMD:R_0402_1005Metric, F.Cu at (168.5, 26.0)
- added R75: 100, Resistor_SMD:R_0402_1005Metric, F.Cu at (168.5, 28.0)
- added R76: 100, Resistor_SMD:R_0402_1005Metric, F.Cu at (168.5, 29.9)
- added R77: 100, Resistor_SMD:R_0402_1005Metric, F.Cu at (168.5, 31.9)
- added R78: 100, Resistor_SMD:R_0402_1005Metric, F.Cu at (168.5, 33.9)
- added R79: 100, Resistor_SMD:R_0402_1005Metric, F.Cu at (168.5, 35.9)
- added R80: 100, Resistor_SMD:R_0402_1005Metric, F.Cu at (168.5, 37.9)
- added R81: 100, Resistor_SMD:R_0402_1005Metric, F.Cu at (168.5, 39.9)
- added R82: 10k, Resistor_SMD:R_0402_1005Metric, F.Cu at (168.5, 41.9)
- added R83: 100, Resistor_SMD:R_0402_1005Metric, F.Cu at (171.5, 26.0)
- added R84: 100, Resistor_SMD:R_0402_1005Metric, F.Cu at (171.5, 28.0)
- added R85: 100, Resistor_SMD:R_0402_1005Metric, F.Cu at (171.5, 29.9)
- added R86: 100, Resistor_SMD:R_0402_1005Metric, F.Cu at (171.5, 31.9)
- added R87: 100, Resistor_SMD:R_0402_1005Metric, F.Cu at (171.5, 33.9)
- added R88: 100, Resistor_SMD:R_0402_1005Metric, F.Cu at (171.5, 35.9)
- added R89: 100, Resistor_SMD:R_0402_1005Metric, F.Cu at (171.5, 37.9)
- added R90: 100, Resistor_SMD:R_0402_1005Metric, F.Cu at (171.5, 39.9)
- added R91: 100, Resistor_SMD:R_0402_1005Metric, F.Cu at (171.5, 41.9)
- added R92: 100, Resistor_SMD:R_0402_1005Metric, F.Cu at (174.4, 26.0)
- added R93: 100, Resistor_SMD:R_0402_1005Metric, F.Cu at (174.4, 28.0)
- added R94: 100, Resistor_SMD:R_0402_1005Metric, F.Cu at (174.4, 29.9)
- added R95: 100, Resistor_SMD:R_0402_1005Metric, F.Cu at (174.4, 31.9)
- added R96: 100, Resistor_SMD:R_0402_1005Metric, F.Cu at (174.4, 33.9)
- added R97: 100, Resistor_SMD:R_0402_1005Metric, F.Cu at (174.4, 35.9)
- added R98: 100, Resistor_SMD:R_0402_1005Metric, F.Cu at (174.4, 37.9)
- added R99: 100k, Resistor_SMD:R_0402_1005Metric, F.Cu at (169.6, 50.4)
- added U34: PCA9685BS,118, Library:QFN65P600X600X100-29N-D, F.Cu at (180.0, 29.1)
- added U36: TPS62177DQC, Package_SON:WSON-10-1EP_2x3mm_P0.5mm_EP0.84x2.4mm_ThermalVias, F.Cu at (170.3, 47.2)
- moved J4 69.4 mm to (25.1, 66.7)
- moved REF** 43.3 mm to (36.7, 56.3)
- moved U33 43.3 mm to (42.3, 56.3)
- moved U33 43.3 mm to (52.5, 56.4)
- moved R104 12.4 mm to (95.2, 46.2), turned to -90 degrees
- moved C10 10.4 mm to (96.2, 46.2), turned to -90 degrees
- moved J1 3.08 mm to (80.7, 34.8)
- moved C22 2.67 mm to (113.2, 45.6)
- moved C27 2.62 mm to (108.7, 46.0)
- moved C14 2.61 mm to (111.7, 45.1)
- moved L3 2.57 mm to (110.2, 45.6)
- moved L7 2.57 mm to (109.8, 44.3)
- moved Y1 0.63 mm to (108.3, 41.1)
- moved C24 0.54 mm to (109.3, 39.2)
- moved C25 0.54 mm to (107.4, 39.2)
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Connections:
- U37 pad 15: unconnected-(U37-CTS-Pad15) -> /MCU/CTS
- U37 pad 16: unconnected-(U37-RTS-Pad16) -> /MCU/RTS
Routing:
- net JTAG_TDI: track 6.69 -> 0.00 mm
- net JTAG_TMS: track 6.51 -> 0.00 mm
- net JTAG_TDO: track 6.37 -> 0.00 mm
- net JTAG_TCK: track 6.05 -> 0.00 mm
- net Net-(U39-RF_P): track 3.71 -> 7.03 mm
- net Net-(C22-Pad1): track 6.44 -> 3.78 mm
- net Net-(U39-RF_N): track 2.40 -> 5.01 mm
- net MCU_RESET: track 5.56 -> 3.26 mm
- net Net-(C14-Pad2): track 1.89 -> 0.00 mm
- net GND: track 35.2 -> 36.7 mm, vias 127 -> 129
- net Net-(U39-DCOUPL): track 0.00 -> 1.44 mm
- net VDDS: track 2.18 -> 3.50 mm
- net Net-(U39-X32K_Q1): track 9.09 -> 8.40 mm
- net Net-(U39-X32K_Q2): track 6.91 -> 6.26 mm

Commit message: m
Parts:
- added C26: 4.7uF, Capacitor_SMD:C_0805_2012Metric, F.Cu at (82.8, 24.5)
- added C9: 10uF, Capacitor_SMD:C_0805_2012Metric, F.Cu at (82.8, 21.5)
- added J5: 640445-2, Library:CONN2_640445-2_TEC, B.Cu at (82.0, 34.8)
- added REF**: DO-214AASMB_J-BEND_LTF, Library:DO-214AASMB_J-BEND_LTF, F.Cu at (87.3, 42.0)
- C3, C4: renamed from REF**; value CP_Elec_6.3x7.7 -> 100uF
- R105, R106: value 100k -> 0
- moved C17 51.5 mm to (101.2, 49.2), turned to -90 degrees
- moved C12 45.3 mm to (102.4, 49.2), turned to -90 degrees
- moved U33 40.9 mm to (83.2, 55.4)
- moved U33 39.9 mm to (92.4, 54.3)
- moved J4 37.5 mm to (46.0, 35.6)
- moved C4 9.22 mm to (66.8, 55.9)
- moved J1 7.75 mm to (72.9, 34.8)
- moved C3 7.42 mm to (66.8, 47.5)
- moved C29 3.92 mm to (105.5, 50.5), turned to 90 degrees
- moved C28 3.68 mm to (110.7, 50.5), turned to -90 degrees
- moved Y2 3.26 mm to (108.1, 50.5)
- moved C13 1.14 mm to (105.1, 47.5), turned to 0 degrees
- moved R106 0.42 mm to (110.6, 55.5)
- moved R105 0.33 mm to (109.5, 55.5)
Connections:
- C3 pad 1: (no net) -> +12V
- C3 pad 2: (no net) -> GND
- C4 pad 1: (no net) -> +12V
- C4 pad 2: (no net) -> GND
- J1 pad 2: +12V -> Net-(J5-Pin_1)
- R101 pad 2: /MCU/SDA -> Net-(U39-DIO_5)
- R105 pad 2: /MCU/RXD -> RX
- R106 pad 2: /MCU/TXD -> TX
- R115 pad 2: /MCU/SCL -> Net-(U39-DIO_4)
- U33 pad 23: /MCU/SCL -> /PWM_Drivers/SCL (x2)
- U33 pad 24: /MCU/SDA -> /PWM_Drivers/SDA (x2)
- U34 pad 23: /MCU/SCL -> /PWM_Drivers/SCL
- U34 pad 24: /MCU/SDA -> /PWM_Drivers/SDA
- U37 pad 15: /MCU/CTS -> CTS
- U37 pad 16: /MCU/RTS -> RTS
- U39 pad 10: /MCU/SDA -> Net-(U39-DIO_5)
- U39 pad 14: MISO -> unconnected-(U39-DIO_8-Pad14)
- U39 pad 15: MOSI -> unconnected-(U39-DIO_9-Pad15)
- U39 pad 16: SCLK -> unconnected-(U39-DIO_10-Pad16)
- U39 pad 28: /MCU/RTS -> unconnected-(U39-DIO_18-Pad28)
- U39 pad 29: /MCU/CTS -> unconnected-(U39-DIO_19-Pad29)
- U39 pad 30: FLASH_CS -> /MCU/PWM_EN
- U39 pad 31: unconnected-(U39-DIO_21-Pad31) -> SDA
- U39 pad 32: unconnected-(U39-DIO_22-Pad32) -> SCL
- U39 pad 36: unconnected-(U39-DIO_23-Pad36) -> RX
- U39 pad 37: unconnected-(U39-DIO_24-Pad37) -> TX
- U39 pad 38: unconnected-(U39-DIO_25-Pad38) -> RTS
- U39 pad 39: unconnected-(U39-DIO_26-Pad39) -> CTS
- U39 pad 40: unconnected-(U39-DIO_27-Pad40) -> FLASH_CS
- U39 pad 41: unconnected-(U39-DIO_28-Pad41) -> SCLK
- U39 pad 42: unconnected-(U39-DIO_29-Pad42) -> MOSI
- U39 pad 43: unconnected-(U39-DIO_30-Pad43) -> MISO
- U39 pad 5: /MCU/PWM_EN -> unconnected-(U39-DIO_0-Pad5)
- U39 pad 7: /MCU/RXD -> unconnected-(U39-DIO_2-Pad7)
- U39 pad 8: /MCU/TXD -> unconnected-(U39-DIO_3-Pad8)
- U39 pad 9: /MCU/SCL -> Net-(U39-DIO_4)
Routing:
- net RTS: track 0.00 -> 22.6 mm
- net CTS: track 0.00 -> 21.6 mm
- net TX: track 0.00 -> 19.9 mm
- net RX: track 0.00 -> 19.3 mm
- net SCLK: track 29.0 -> 13.6 mm
- net FLASH_CS: track 35.2 -> 22.2 mm
- net MOSI: track 24.4 -> 11.7 mm
- net MISO: track 23.9 -> 15.4 mm
- net VDDS: track 3.50 -> 7.06 mm, vias 0 -> 1
- net VDDR: track 1.96 -> 5.03 mm, vias 0 -> 1
- net Net-(U39-X24M_P): track 8.67 -> 9.55 mm
- net Net-(J5-Pin_1): vias 0 -> 30
- added copper zone on B.Cu, net Net-(J5-Pin_1)
- added copper zone on F.Cu, net Net-(J5-Pin_1)
- added copper zone on In1.Cu, net Net-(J5-Pin_1)
- added copper zone on In2.Cu, net Net-(J5-Pin_1)
Other:
- outline, holes or cut-outs redrawn
- board text added: "PCB Cutout Area"

Commit message: d
Parts:
- added D39: SOD3716X135N, Library:SOD3716X135N, F.Cu at (89.0, 25.4)
- added F1: FUSC6127X294N, Library:FUSC6127X294N, F.Cu at (83.7, 32.9)
- moved U33 62.5 mm to (154.8, 57.8)
- moved U33 62.5 mm to (145.6, 58.9)
- moved D38 12.5 mm to (76.2, 47.8), turned to 90 degrees
- moved J5 2.54 mm to (81.9, 37.3), turned to 180 degrees
- renumbered REF** to D38
Routing:
- net Net-(J5-Pin_1): vias 30 -> 0
- removed copper zone on B.Cu, net Net-(J5-Pin_1)
- removed copper zone on F.Cu, net Net-(J5-Pin_1)
- removed copper zone on In1.Cu, net Net-(J5-Pin_1)
- removed copper zone on In2.Cu, net Net-(J5-Pin_1)
Other:
- outline, holes or cut-outs redrawn
