File: Hardware/Ring-Light v4/Ring-Light.kicad_sch (KiCad schematic)
At the start: 17 parts, among them U1 NCR321PASX, U2 NCR321PASX, U29 PCA9685BS,118

Commit message: m
Parts:
- added C10, C11, C12, C13, C14, C15, C16, C17, C18, C19, C20, C21, C22, C23, C24, C25, C26, C27, C28, C29, C30, C31, C32, C5, C6, C7, C8, C9: 1uF, Capacitor_SMD:C_0402_1005Metric, symbol Device:C_Small
- added C34: 0.1uF, Capacitor_SMD:C_0603_1608Metric, symbol Device:C_Small
- added D10, D11, D12, D13, D14, D15, D16, D17, D18, D19, D20, D21, D22, D23, D24, D25, D26, D27, D28, D29, D30, D31, D32, D7, D8, D9: LED, Library:GWJTLRS1EMLVL5XX531, symbol Library:LED
- added R10, R12, R14, R16, R18, R20, R22, R24, R26, R28, R30, R32, R34, R36, R38, R4, R40, R42, R44, R46, R48, R50, R52, R54, R56, R58, R6, R60, R62, R64, R8: 9.09, Resistor_SMD:R_0402_1005Metric, symbol Device:R_Small
- added R11, R13, R15, R17, R19, R21, R23, R25, R27, R29, R3, R31, R33, R35, R37, R39, R41, R43, R45, R47, R49, R5, R51, R53, R55, R57, R59, R61, R63, R7, R9: 100k, Resistor_SMD:R_0402_1005Metric, symbol Device:R_Small
- added R66: 10k, Resistor_SMD:R_0402_1005Metric, symbol Device:R_Small
- added R67, R68, R69, R70, R71, R72, R73, R74, R75, R76, R77, R78, R79, R80, R81, R82, R83, R84, R85, R86, R87, R88, R89, R90, R91, R92, R93, R94, R95, R96, R97, R98: 100, Resistor_SMD:R_0402_1005Metric, symbol Device:R_Small
- added U10, U11, U12, U13, U14, U15, U16, U17, U18, U19, U20, U21, U22, U23, U24, U25, U26, U27, U28, U29, U3, U30, U31, U32, U4, U5, U6, U7, U8, U9: NCR321PASX, Library:NCR321PASX, symbol Library:NCR321PASX
- added U34: PCA9685BS,118, Library:QFN65P600X600X100-29N-D, symbol Library:PCA9685BS,118
- added U35: STM32WB50CGUx, Package_DFN_QFN:QFN-48-1EP_7x7mm_P0.5mm_EP5.6x5.6mm, symbol MCU_ST_STM32WB:STM32WB50CGUx
- C1, C3: footprint Capacitor_SMD:C_0805_2012Metric -> Capacitor_SMD:C_0402_1005Metric
- C2, C4: value 0.1uF -> 1uF; footprint Capacitor_SMD:C_0603_1608Metric -> Capacitor_SMD:C_0402_1005Metric
- R1: value 80.6 -> 100k; footprint Resistor_SMD:R_1210_3225Metric -> Resistor_SMD:R_0402_1005Metric
- R2: value 80.6 -> 9.09; footprint Resistor_SMD:R_1210_3225Metric -> Resistor_SMD:R_0402_1005Metric
- renumbered C73 to C33, R4 to R65, U29 to U33
Connections:
- net +12V: now also D1.3 (A), D1.4 (A), D2.3 (A), D2.4 (A), D5.3 (A), D5.4 (A), D6.3 (A), D6.4 (A), C10.1, C11.1, C12.1, C13.1, C14.1, C15.1, C16.1, C17.1, C18.1, C19.1, C20.1, C21.1, C22.1, C23.1, C24.1, C25.1, C26.1, C27.1, C28.1, C29.1, C30.1, C31.1, C32.1, C5.1, C6.1, C7.1, C8.1, C9.1, D10.3 (A), D10.4 (A), D11.3 (A), D11.4 (A), D12.3 (A), D12.4 (A), D13.3 (A), D13.4 (A), D14.3 (A), D14.4 (A), D15.3 (A), D15.4 (A), D16.3 (A), D16.4 (A), D17.3 (A), D17.4 (A), D18.3 (A), D18.4 (A), D19.3 (A), D19.4 (A), D20.3 (A), D20.4 (A), D21.3 (A), D21.4 (A), D22.3 (A), D22.4 (A), D23.3 (A), D23.4 (A), D24.3 (A), D24.4 (A), D25.3 (A), D25.4 (A), D26.3 (A), D26.4 (A), D27.3 (A), D27.4 (A), D28.3 (A), D28.4 (A), D29.3 (A), D29.4 (A), D30.3 (A), D30.4 (A), D31.3 (A), D31.4 (A), D32.3 (A), D32.4 (A), D7.3 (A), D7.4 (A), D8.3 (A), D8.4 (A), D9.3 (A), D9.4 (A); no longer U1.1 (VEN), U2.1 (VEN)
- net +3.3V: now also C34.1, R66.2, U34.25 (VDD)
- net GND: now also C10.2, C11.2, C12.2, C13.2, C14.2, C15.2, C16.2, C17.2, C18.2, C19.2, C20.2, C21.2, C22.2, C23.2, C24.2, C25.2, C26.2, C27.2, C28.2, C29.2, C30.2, C31.2, C32.2, C34.2, C5.2, C6.2, C7.2, C8.2, C9.2, R10.2, R11.2, R12.2, R13.2, R14.2, R15.2, R16.2, R17.2, R18.2, R19.2, R20.2, R21.2, R22.2, R23.2, R24.2, R25.2, R26.2, R27.2, R28.2, R29.2, R3.2, R30.2, R31.2, R32.2, R33.2, R34.2, R35.2, R36.2, R37.2, R38.2, R39.2, R4.2, R40.2, R41.2, R42.2, R43.2, R44.2, R45.2, R46.2, R47.2, R48.2, R49.2, R5.2, R50.2, R51.2, R52.2, R53.2, R54.2, R55.2, R56.2, R57.2, R58.2, R59.2, R6.2, R60.2, R61.2, R62.2, R63.2, R64.2, R7.2, R8.2, R9.2, U10.5 (GND), U11.5 (GND), U12.5 (GND), U13.5 (GND), U14.5 (GND), U15.5 (GND), U16.5 (GND), U17.5 (GND), U18.5 (GND), U19.5 (GND), U20.5 (GND), U21.5 (GND), U22.5 (GND), U23.5 (GND), U24.5 (GND), U25.5 (GND), U26.5 (GND), U27.5 (GND), U28.5 (GND), U29.5 (GND), U3.5 (GND), U30.5 (GND), U31.5 (GND), U32.5 (GND), U34.11 (VSS), U34.22 (EXTCLK), U34.29 (EP), U4.5 (GND), U5.5 (GND), U6.5 (GND), U7.5 (GND), U8.5 (GND), U9.5 (GND)
- net PWM1: now also R1.1, U1.1 (VEN), R67.1; no longer U33.3 (LED0)
- net PWM10: now also R19.1, R76.1, U10.1 (VEN); no longer U33.13 (LED9)
- net PWM11: now also R21.1, R77.1, U11.1 (VEN); no longer U33.14 (LED10)
- net PWM12: now also R23.1, R78.1, U12.1 (VEN); no longer U33.15 (LED11)
- net PWM13: now also R25.1, R79.1, U13.1 (VEN); no longer U33.16 (LED12)
- net PWM14: now also R27.1, R80.1, U14.1 (VEN); no longer U33.17 (LED13)
- net PWM15: now also R29.1, R81.1, U15.1 (VEN); no longer U33.18 (LED14)
- net PWM16: now also R31.1, R82.1, U16.1 (VEN); no longer U33.19 (LED15)
- net PWM2: now also U2.1 (VEN), R3.1, R68.1; no longer U33.4 (LED1)
- net PWM3: now also R5.1, R69.1, U3.1 (VEN); no longer U33.5 (LED2)
- net PWM4: now also R7.1, R70.1, U4.1 (VEN); no longer U33.6 (LED3)
- net PWM5: now also R71.1, R9.1, U5.1 (VEN); no longer U33.7 (LED4)
- net PWM6: now also R11.1, R72.1, U6.1 (VEN); no longer U33.8 (LED5)
- net PWM7: now also R13.1, R73.1, U7.1 (VEN); no longer U33.9 (LED6)
- net PWM8: now also R15.1, R74.1, U8.1 (VEN); no longer U33.10 (LED7)
- net PWM9: now also R17.1, R75.1, U9.1 (VEN); no longer U33.12 (LED8)
- net SCL: now also U34.23 (SCL)
- net SDA: now also U34.24 (SDA); no longer R65.1, U33.20 (~{OE})
- net OUT5: now reaches D5.1 (K), D5.2 (K)
- net OUT5: now also U5.6 (IOUT), U5.7 (IOUT); no longer D6.3 (A), D6.4 (A)
- net OUT4: now reaches D4.1 (K), D4.2 (K)
- net OUT4: now also U4.6 (IOUT), U4.7 (IOUT); no longer D5.3 (A), D5.4 (A)
- net REXT1: now reaches R2.1, U1.2 (REXT)
- net REXT2: now reaches U2.2 (REXT)
- net REXT2: now also R4.1; no longer R1.1
- net OUT2: now reaches U2.6 (IOUT), U2.7 (IOUT)
- net OUT2: now also D2.1 (K), D2.2 (K); no longer D6.1 (K), D6.2 (K)
- net OUT1: now reaches D1.1 (K), D1.2 (K), U1.6 (IOUT), U1.7 (IOUT)
- net OUT3: now reaches D3.1 (K), D3.2 (K)
- net OUT3: now also U3.6 (IOUT), U3.7 (IOUT); no longer D2.3 (A), D2.4 (A)
- new net: R74.2, U33.10 (LED7)
- new net: R75.2, U33.12 (LED8)
- new net: R76.2, U33.13 (LED9)
- new net: R77.2, U33.14 (LED10)
- new net: R78.2, U33.15 (LED11)
- new net: R79.2, U33.16 (LED12)
- new net: R80.2, U33.17 (LED13)
- new net: R81.2, U33.18 (LED14)
- new net: R82.2, U33.19 (LED15)
- new net: R67.2, U33.3 (LED0)
- new net: R68.2, U33.4 (LED1)
- new net: R69.2, U33.5 (LED2)
- new net: R70.2, U33.6 (LED3)
- new net: R71.2, U33.7 (LED4)
- new net: R72.2, U33.8 (LED5)
- new net: R73.2, U33.9 (LED6)
- new net: R98.2, U34.19 (LED15)
- new net: R95.2, U34.16 (LED12)
- new net: R85.2, U34.5 (LED2)
- new net: R96.2, U34.17 (LED13)
- new net: R90.2, U34.10 (LED7)
- new net: R92.2, U34.13 (LED9)
- new net: R91.2, U34.12 (LED8)
- new net: U35.32 (VSS), U35.49 (VSS)
- new net: R87.2, U34.7 (LED4)
- new net: R86.2, U34.6 (LED3)
- new net: R84.2, U34.4 (LED1)
- new net: R88.2, U34.8 (LED5)
- new net: R93.2, U34.14 (LED10)
- new net: R94.2, U34.15 (LED11)
- new net: R97.2, U34.18 (LED14)
- new net: R83.2, U34.3 (LED0)
- new net: R89.2, U34.9 (LED6)
- new net OUT10: D10.1 (K), D10.2 (K), U10.6 (IOUT), U10.7 (IOUT)
- new net OUT11: D11.1 (K), D11.2 (K), U11.6 (IOUT), U11.7 (IOUT)
- new net OUT12: D12.1 (K), D12.2 (K), U12.6 (IOUT), U12.7 (IOUT)
- new net OUT13: D13.1 (K), D13.2 (K), U13.6 (IOUT), U13.7 (IOUT)
- new net OUT14: D14.1 (K), D14.2 (K), U14.6 (IOUT), U14.7 (IOUT)
- new net OUT15: D15.1 (K), D15.2 (K), U15.6 (IOUT), U15.7 (IOUT)
- new net OUT16: D16.1 (K), D16.2 (K), U16.6 (IOUT), U16.7 (IOUT)
- new net OUT17: D17.1 (K), D17.2 (K), U17.6 (IOUT), U17.7 (IOUT)
- new net OUT18: D18.1 (K), D18.2 (K), U18.6 (IOUT), U18.7 (IOUT)
- new net OUT19: D19.1 (K), D19.2 (K), U19.6 (IOUT), U19.7 (IOUT)
- new net OUT20: D20.1 (K), D20.2 (K), U20.6 (IOUT), U20.7 (IOUT)
- new net OUT21: D21.1 (K), D21.2 (K), U21.6 (IOUT), U21.7 (IOUT)
- new net OUT22: D22.1 (K), D22.2 (K), U22.6 (IOUT), U22.7 (IOUT)
- new net OUT23: D23.1 (K), D23.2 (K), U23.6 (IOUT), U23.7 (IOUT)
- new net OUT24: D24.1 (K), D24.2 (K), U24.6 (IOUT), U24.7 (IOUT)
- new net OUT25: D25.1 (K), D25.2 (K), U25.6 (IOUT), U25.7 (IOUT)
- new net OUT26: D26.1 (K), D26.2 (K), U26.6 (IOUT), U26.7 (IOUT)
- new net OUT27: D27.1 (K), D27.2 (K), U27.6 (IOUT), U27.7 (IOUT)
- new net OUT28: D28.1 (K), D28.2 (K), U28.6 (IOUT), U28.7 (IOUT)
- new net OUT29: D29.1 (K), D29.2 (K), U29.6 (IOUT), U29.7 (IOUT)
- new net OUT30: D30.1 (K), D30.2 (K), U30.6 (IOUT), U30.7 (IOUT)
- new net OUT31: D31.1 (K), D31.2 (K), U31.6 (IOUT), U31.7 (IOUT)
- new net OUT32: D32.1 (K), D32.2 (K), U32.6 (IOUT), U32.7 (IOUT)
- new net OUT6: D6.1 (K), D6.2 (K), U6.6 (IOUT), U6.7 (IOUT)
- new net OUT7: D7.1 (K), D7.2 (K), U7.6 (IOUT), U7.7 (IOUT)
- new net OUT8: D8.1 (K), D8.2 (K), U8.6 (IOUT), U8.7 (IOUT)
- new net OUT9: D9.1 (K), D9.2 (K), U9.6 (IOUT), U9.7 (IOUT)
- new net PWM17: R33.1, R83.1, U17.1 (VEN)
- new net PWM18: R35.1, R84.1, U18.1 (VEN)
- new net PWM19: R37.1, R85.1, U19.1 (VEN)
- new net PWM20: R39.1, R86.1, U20.1 (VEN)
- new net PWM21: R41.1, R87.1, U21.1 (VEN)
- new net PWM22: R43.1, R88.1, U22.1 (VEN)
- new net PWM23: R45.1, R89.1, U23.1 (VEN)
- new net PWM24: R47.1, R90.1, U24.1 (VEN)
- new net PWM25: R49.1, R91.1, U25.1 (VEN)
- new net PWM26: R51.1, R92.1, U26.1 (VEN)
- new net PWM27: R53.1, R93.1, U27.1 (VEN)
- new net PWM28: R55.1, R94.1, U28.1 (VEN)
- new net PWM29: R57.1, R95.1, U29.1 (VEN)
- new net PWM30: R59.1, R96.1, U30.1 (VEN)
- new net PWM31: R61.1, R97.1, U31.1 (VEN)
- new net PWM32: R63.1, R98.1, U32.1 (VEN)
- new net PWM_EN: R65.1, R66.1, U33.20 (~{OE}), U34.20 (~{OE})
- new net REXT10: R20.1, U10.2 (REXT)
- new net REXT11: R22.1, U11.2 (REXT)
- new net REXT12: R24.1, U12.2 (REXT)
- new net REXT13: R26.1, U13.2 (REXT)
- new net REXT14: R28.1, U14.2 (REXT)
- new net REXT15: R30.1, U15.2 (REXT)
- new net REXT16: R32.1, U16.2 (REXT)
- new net REXT17: R34.1, U17.2 (REXT)
- new net REXT18: R36.1, U18.2 (REXT)
- new net REXT19: R38.1, U19.2 (REXT)
- new net REXT20: R40.1, U20.2 (REXT)
- new net REXT21: R42.1, U21.2 (REXT)
- new net REXT22: R44.1, U22.2 (REXT)
- new net REXT23: R46.1, U23.2 (REXT)
- new net REXT24: R48.1, U24.2 (REXT)
- new net REXT25: R50.1, U25.2 (REXT)
- new net REXT26: R52.1, U26.2 (REXT)
- new net REXT27: R54.1, U27.2 (REXT)
- new net REXT28: R56.1, U28.2 (REXT)
- new net REXT29: R58.1, U29.2 (REXT)
- new net REXT3: R6.1, U3.2 (REXT)
- new net REXT30: R60.1, U30.2 (REXT)
- new net REXT31: R62.1, U31.2 (REXT)
- new net REXT32: R64.1, U32.2 (REXT)
- new net REXT4: R8.1, U4.2 (REXT)
- new net REXT5: R10.1, U5.2 (REXT)
- new net REXT6: R12.1, U6.2 (REXT)
- new net REXT7: R14.1, U7.2 (REXT)
- new net REXT8: R16.1, U8.2 (REXT)
- new net REXT9: R18.1, U9.2 (REXT)
Other:
- moved on the sheet: C1, C33, D1, R2, R65, U1, U33

Commit message: m
Parts:
- removed C1, C2, C20, C21, C22, C23, C24, C25, C26, C27, C28, C29, C3, C30, C31, C32, C4: 1uF, Capacitor_SMD:C_0402_1005Metric, symbol Device:C_Small
- removed U35: STM32WB50CGUx, Package_DFN_QFN:QFN-48-1EP_7x7mm_P0.5mm_EP5.6x5.6mm, symbol MCU_ST_STM32WB:STM32WB50CGUx
- added C3, C4: 100uF, symbol Device:C_Polarized_Small
- added FL1: BLM18HE152SN1, Inductor_SMD:L_0603_1608Metric, symbol Device:L_Small
- added J1: 694106301002, symbol Connector:Barrel_Jack_Switch
- added L1, L2: 10uH, symbol Device:L_Small
- added R100, R101, R102, R103: 10k, Resistor_SMD:R_0402_1005Metric, symbol Device:R_Small
- added R104, R99: 100k, Resistor_SMD:R_0402_1005Metric, symbol Device:R_Small
- added SW1: ACZ11BR1E, symbol Device:RotaryEncoder_Switch
- added U35: CC2640R2FRSMR, QFN40P400X400X100-33N-D, symbol Library:CC2640R2FRSMR
- added U36: TPS62177DQC, Package_SON:WSON-10-1EP_2x3mm_P0.5mm_EP0.84x2.4mm_ThermalVias, symbol Library:TPS62177DQC
- C11: value 1uF -> 10uF
- C12, C13, C15, C16, C17, C19: value 1uF -> 100nF
- C14: value 1uF -> DNP; now not fitted
- C18: value 1uF -> 22uF
- C5: value 1uF -> 0.1uF; footprint Capacitor_SMD:C_0402_1005Metric -> Capacitor_SMD:C_0603_1608Metric
- C6: value 1uF -> 22uF; footprint Capacitor_SMD:C_0402_1005Metric -> Capacitor_SMD:C_0603_1608Metric
- C7, C8: value 1uF -> 10nF; footprint Capacitor_SMD:C_0402_1005Metric -> Capacitor_SMD:C_0603_1608Metric
- renumbered C33 to C1, C34 to C2, R67 to R66, R69 to R67, R71 to R68, R73 to R69, R75 to R70, R77 to R71, R79 to R72, R81 to R73, R68 to R74, R70 to R75, R72 to R76, R74 to R77, R76 to R78, R78 to R79, R82 to R81, R66 to R82, R85 to R84, R87 to R85, R89 to R86, R91 to R87, R93 to R88, R95 to R89, R97 to R90, R84 to R91, R86 to R92, R88 to R93, R90 to R94, R92 to R95, R94 to R96, R96 to R97
Connections:
- net +12V: now also C3.1, C4.1, J1.2, U36.2 (VIN), U36.3 (EN); no longer C10.1, C11.1, C12.1, C13.1, C14.1, C15.1, C16.1, C17.1, C18.1, C19.1, C6.1, C7.1, C8.1, C9.1
- net +3.3V: now also C6.1, FL1.1, L1.2, R102.2, R103.2, R99.1, U36.10 (VOS), U36.8 (~{SLEEP})
- net GND: now also C3.2, C4.2, J1.1, SW1.C, U35.17 (VSS_3), U35.20 (VSS_4), U35.29 (VSS_5), U35.3 (VSS_1), U35.33 (EP), U35.7 (VSS_2), U36.1 (PGND), U36.11 (PAD), U36.4 (NC), U36.5 (FB), U36.6 (AGND); no longer C14.2, C15.2, C16.2, C17.2, C18.2, C19.2
- new net: C14.1, C15.1, C16.1, C17.1, C18.1, C19.1, FL1.2
- new net: C15.2, C16.2, C19.2
- new net: L1.1, U36.9 (SW)
- new net: C10.1, R104.2, U35.21 (RESET_N)
- new net: R100.2, R103.1, SW1.B
- new net: C8.1, R101.1
- new net: R101.2, R102.1, SW1.A
- new net: C7.1, R100.1
- new net: C9.1, U35.12 (DCOUPL)
- new net DCDC_SW: L2.1, U35.18 (DCDC_SW)
- new net PG: R99.2, U36.7 (PG)
- new net VDDR: C11.1, C12.1, C13.1, L2.2, U35.28 (VDDR), U35.32 (VDDR_RF)
- new net VDDS: R104.1, U35.11 (VDDS2), U35.19 (VDDS_DCDC), U35.27 (VDDS)
- no-connect marks 0 -> 1
Other:
- moved on the sheet: C1, C2, R65, R66, R67, R68, R69, R70, R71, R72, R73, R74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

Commit message: m
Parts:
- removed C7, C8: 10nF, Capacitor_SMD:C_0603_1608Metric, symbol Device:C_Small
- removed R100, R101, R102, R103: 10k, Resistor_SMD:R_0402_1005Metric, symbol Device:R_Small
- removed SW1: ACZ11BR1E, symbol Device:RotaryEncoder_Switch
- added P1: USB_C_Plug_USB2.0, symbol Connector:USB_C_Plug_USB2.0
- added U37: CP2102N-A02-GQFN20R, Library:CP2102NA02GQFN20, symbol Library:CP2102N-A02-GQFN20R
Connections:
- new net: P1.A1 (GND), P1.A12 (GND), P1.B1 (GND), P1.B12 (GND)
- new net: P1.A4 (VBUS), P1.A9 (VBUS), P1.B4 (VBUS), P1.B9 (VBUS)

Commit message: d
Parts:
- removed P1: USB_C_Plug_USB2.0, symbol Connector:USB_C_Plug_USB2.0
- added C20: 1.0uF, Capacitor_SMD:C_0603_1608Metric, symbol Device:C_Small
- added C21: 100pF, Capacitor_SMD:C_0603_1608Metric, symbol Device:C_Small
- added C7, C8: 0.1uF, Capacitor_SMD:C_0603_1608Metric, symbol Device:C_Small
- added D33: SP0503BAHT, Package_TO_SOT_SMD:SOT-143, symbol Power_Protection:SP0503BAHT
- added D34: LTST-C170YKT, Library:GWJTLRS1EMLVL5XX531, symbol Library:LED
- added J2: USB_B_Micro, symbol Connector:USB_B_Micro
- added R100: 1k, Resistor_SMD:R_0402_1005Metric, symbol Device:R_Small
- added R101: 100k, Resistor_SMD:R_0402_1005Metric, symbol Device:R_Small
Connections:
- net GND: now also U37.12 (GND_2), U37.21 (EP_GND), U37.3 (GND_1), C20.2, C21.2, C7.2, C8.2, D33.1 (A), J2.5 (GND), R101.2
- net at U37.20 (GPIO.2_/_TXT): now also D34.1 (K), D34.2 (K)
- net at U37.4 (D+): now also D33.3 (K), J2.3 (D+)
- net at U37.5 (D-): now also D33.4 (K), J2.2 (D-)
- net at U37.6 (VDD): now also C7.1, R100.1
- net at U37.7 (VREGIN): now also U37.8 (VBUS), C20.1, C8.1, D33.2 (K), J2.1 (VBUS)
- net at U37.9 (~{RST}): now also R100.2
- new net: D34.3 (A), D34.4 (A)
- new net SH: C21.1, J2.6 (Shield), R101.1
- no-connect marks 1 -> 7
Other:
- moved on the sheet: U37

Commit message: m
Parts:
- added C24, C25: 12pF, Capacitor_SMD:C_0402_1005Metric, symbol Device:C_Small
- added C26: 15pF, Capacitor_SMD:C_0402_1005Metric, symbol Device:C_Small
- added D35: LTST-C170YKT, Diode_SMD:D_0402_1005Metric, symbol Library:LED
- added IC1: CC2640R2FRGZR, QFN50P700X700X100-49N-D, symbol Library:CC2640R2FRGZR
- added R102, R103: 1k, Resistor_SMD:R_0402_1005Metric, symbol Device:R_Small
- added R105, R106: 100k, Resistor_SMD:R_0402_1005Metric, symbol Device:R_Small
- added U38: W25X40CLUXIG_TR, Library:PSON50P300X200X60-9N, symbol Library:W25X40CLUXIG_TR
- added Y1: 32.768kHz, symbol Device:Crystal
- added Y2: 24MHz, symbol Device:Crystal_GND24
- C21: value 100pF -> 100nF
- D34: footprint Library:GWJTLRS1EMLVL5XX531 -> Diode_SMD:D_0402_1005Metric
Connections:
- net GND: now also C24.2, C25.2, Y2.2 (G), Y2.4 (G)
- net USB_VDD: now reaches C7.1, R100.1, U37.6 (VDD)
- net USB_VDD: now also R102.2, R103.2
- net at U37.17 (RXD): now also R106.1
- net at U37.18 (TXD): now also R105.1
- net at U37.19 (GPIO.3_/_RXT): now also D35.1 (K), D35.2 (K)
- net at U35.1 (RF_P): now also C26.1
- net at U35.30 (X24M_N): now also Y2.1
- net at U35.31 (X24M_P): now also Y2.3
- net at U35.5 (X32K_Q1): now also C25.1, Y1.1
- net at U35.6 (X32K_Q2): now also C24.1, Y1.2
- net at D34.3 (A), D34.4 (A): now also R102.1
- new net: D35.3 (A), D35.4 (A), R103.1
- new net UART_RX: R106.2
- new net UART_TX: R105.2
- no-connect marks 7 -> 9
Other:
- moved on the sheet: C10, C20, C21, C7, C8, C9, D33, D34, J2, R100, R101, R104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

Commit message: d
Parts:
- removed C1, C2, C7, C8: 0.1uF, Capacitor_SMD:C_0603_1608Metric, symbol Device:C_Small
- removed C10, C9: 1uF, Capacitor_SMD:C_0402_1005Metric, symbol Device:C_Small
- removed C11: 10uF, Capacitor_SMD:C_0402_1005Metric, symbol Device:C_Small
- removed C12, C13, C15, C16, C17, C19: 100nF, Capacitor_SMD:C_0402_1005Metric, symbol Device:C_Small
- removed C14: DNP, Capacitor_SMD:C_0402_1005Metric, symbol Device:C_Small
- removed C18: 22uF, Capacitor_SMD:C_0402_1005Metric, symbol Device:C_Small
- removed C20: 1.0uF, Capacitor_SMD:C_0603_1608Metric, symbol Device:C_Small
- removed C21: 100nF, Capacitor_SMD:C_0603_1608Metric, symbol Device:C_Small
- removed C24, C25: 12pF, Capacitor_SMD:C_0402_1005Metric, symbol Device:C_Small
- removed C26: 15pF, Capacitor_SMD:C_0402_1005Metric, symbol Device:C_Small
- removed D1, D10, D11, D12, D13, D14, D15, D16, D17, D18, D19, D2, D20, D21, D22, D23, D24, D25, D26, D27, D28, D29, D3, D30, D31, D32, D4, D5, D6, D7, D8, D9: LED, Library:GWJTLRS1EMLVL5XX531, symbol Library:LED
- removed D33: SP0503BAHT, Package_TO_SOT_SMD:SOT-143, symbol Power_Protection:SP0503BAHT
- removed D34, D35: LTST-C170YKT, Diode_SMD:D_0402_1005Metric, symbol Library:LED
- removed FL1: BLM18HE152SN1, Inductor_SMD:L_0603_1608Metric, symbol Device:L_Small
- removed IC1: CC2640R2FRGZR, QFN50P700X700X100-49N-D, symbol Library:CC2640R2FRGZR
- removed J2: USB_B_Micro, symbol Connector:USB_B_Micro
- removed L2: 10uH, symbol Device:L_Small
- removed R1, R101, R104, R105, R106, R11, R13, R15, R17, R19, R21, R23, R25, R27, R29, R3, R31, R33, R35, R37, R39, R41, R43, R45, R47, R49, R5, R51, R53, R55, R57, R59, R61, R63, R7, R9: 100k, Resistor_SMD:R_0402_1005Metric, symbol Device:R_Small
- removed R10, R12, R14, R16, R18, R2, R20, R22, R24, R26, R28, R30, R32, R34, R36, R38, R4, R40, R42, R44, R46, R48, R50, R52, R54, R56, R58, R6, R60, R62, R64, R8: 9.09, Resistor_SMD:R_0402_1005Metric, symbol Device:R_Small
- removed R100, R102, R103: 1k, Resistor_SMD:R_0402_1005Metric, symbol Device:R_Small
- removed R65, R82: 10k, Resistor_SMD:R_0402_1005Metric, symbol Device:R_Small
- removed R66, R67, R68, R69, R70, R71, R72, R73, R74, R75, R76, R77, R78, R79, R80, R81, R83, R84, R85, R86, R87, R88, R89, R90, R91, R92, R93, R94, R95, R96, R97, R98: 100, Resistor_SMD:R_0402_1005Metric, symbol Device:R_Small
- removed U1, U10, U11, U12, U13, U14, U15, U16, U17, U18, U19, U2, U20, U21, U22, U23, U24, U25, U26, U27, U28, U29, U3, U30, U31, U32, U4, U5, U6, U7, U8, U9: NCR321PASX, Library:NCR321PASX, symbol Library:NCR321PASX
- removed U33, U34: PCA9685BS,118, Library:QFN65P600X600X100-29N-D, symbol Library:PCA9685BS,118
- removed U35: CC2640R2FRSMR, QFN40P400X400X100-33N-D, symbol Library:CC2640R2FRSMR
- removed U37: CP2102N-A02-GQFN20R, Library:CP2102NA02GQFN20, symbol Library:CP2102N-A02-GQFN20R
- removed U38: W25X40CLUXIG_TR, Library:PSON50P300X200X60-9N, symbol Library:W25X40CLUXIG_TR
- removed Y1: 32.768kHz, symbol Device:Crystal
- removed Y2: 24MHz, symbol Device:Crystal_GND24
Connections:
- no-connect marks 9 -> 1
Other:
- added sheet Interface (Interface.kicad_sch)
- added sheet LEDs_1-16 (LEDs_1-16.kicad_sch)
- added sheet LEDs_17-32 (LEDs_17-32.kicad_sch)
- added sheet MCU (MCU.kicad_sch)
- added sheet PWM_Drivers (PWM_Drivers.kicad_sch)
- moved on the sheet: C3, C4, C5, C6, J1, L1, R99, U36

Commit message: m
Other:
- moved on the sheet: C3, C4, C5, C6, J1, L1, R99, U36

Commit message: m
Other:
- sheet MCU ports: added JTAG_TCK, JTAG_TDI, JTAG_TDO, JTAG_TMS, MCU_RESET, PWM_EN, SCL, SDA; removed none
