File: Hardware/Ring-Light v4/Ring-Light.kicad_sch (KiCad schematic)
At the start: 8 parts, among them J1 694106301002, U36 TPS62177DQC

Commit message: d
Other:
- removed sheet Interface
- sheet MCU ports: added none; removed JTAG_TCK, JTAG_TDI, JTAG_TDO, JTAG_TMS, MCU_RESET
Changed lines of the file:
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@@
-	)
-	(sheet
-		(at 43.18 69.85)
-		(size 41.91 31.75)
-		(exclude_from_sim no)
-		(in_bom yes)
-		(on_board yes)
-		(dnp no)
-		(fields_autoplaced yes)
-		(stroke
-			(width 0.1524)
-			(type solid)
-		)
-		(fill
-			(color 0 0 0 0.0000)
-		)
-		(property "Sheetname" "Interface"
-			(at 43.18 69.1384 0)
-			(effects
-				(font
-					(size 1.27 1.27)
-				)
-				(justify left bottom)
-			)
-		)
-		(property "Sheetfile" "Interface.kicad_sch"
-			(at 43.18 102.1846 0)
-			(effects
-				(font
-					(size 1.27 1.27)
-				)
-				(justify left top)
-			)
-		)
-		(instances
-			(project "Ring-Light"
-				(path "/7146df34-bb5a-4ab6-bd6d-8aad9726b4e6"
-					(page "6")
-				)
-			)
-		)
 	)
 	(sheet
@@
 			)
 		)
-		(pin "JTAG_TCK" input
-			(at 157.48 68.58 180)
-			(effects
-				(font
-					(size 1.27 1.27)
-				)
-				(justify left)
-			)
-		)
-		(pin "JTAG_TDI" input
-			(at 157.48 71.12 180)
-			(effects
-				(font
-					(size 1.27 1.27)
-				)
-				(justify left)
-			)
-		)
-		(pin "JTAG_TDO" input
-			(at 157.48 73.66 180)
-			(effects
-				(font
-					(size 1.27 1.27)
-				)
-				(justify left)
-			)
-		)
-		(pin "JTAG_TMS" input
-			(at 157.48 76.2 180)
-			(effects
-				(font
-					(size 1.27 1.27)
-				)
-				(justify left)
-			)
-		)
-		(pin "MCU_RESET" input
-			(at 157.48 78.74 180)
-			(effects
-				(font
-					(size 1.27 1.27)
-				)
-				(justify left)
-			)
-		)

Commit message: m
Parts:
- added C26: 4.7uF, Capacitor_SMD:C_0805_2012Metric, symbol Device:C_Small
- added C9: 10uF, Capacitor_SMD:C_0805_2012Metric, symbol Device:C_Small
- added D38: SMAJ15A, Diode_SMD:D_SMA, symbol Diode:SMAJ15A
- added F1: Fuse, symbol Device:Fuse
- added J5: 640445-2, symbol Connector_Generic:Conn_02x01
Connections:
- net +12V: now also C26.1, C9.1, F1.2; no longer J1.2
- net GND: now also C26.2, C9.2, D38.2 (A2)
- new net: D38.1 (A1), F1.1, J5.2 (Pin_2)
- new net: J1.2, J5.1 (Pin_1)
Other:
- moved on the sheet: C3, C4, C5, C6, J1, L1, R99, U36
