File: Hardware/Ring-Light v4/MCU.kicad_sch (KiCad schematic)
At the start: 22 parts, among them IC1 CC2640R2FRGZR, U35 CC2640R2FRSMR, U38 W25X40CLUXIG_TR, Y1 32.768kHz, Y2 24MHz

Commit message: m
Parts:
- added AE1: Inverted F, symbol Device:Antenna
- added C22: 12pF, Capacitor_SMD:C_0402_1005Metric, symbol Device:C_Small
- added C23, C27, C29: 1pF, Capacitor_SMD:C_0402_1005Metric, symbol Device:C_Small
- added C28: DNM, Capacitor_SMD:C_0402_1005Metric, symbol Device:C_Small
- added C30: 0.5pF, Capacitor_SMD:C_0402_1005Metric, symbol Device:C_Small
- added C31: 100nF, Capacitor_SMD:C_0402_1005Metric, symbol Device:C_Small
- added J3: ~, symbol Library:M8430-2610RB3
- added L3, L4: 2.4nH, symbol Device:L_Small
- added L5, L6: 2nH, symbol Device:L_Small
- added R107: 0, Resistor_SMD:R_0402_1005Metric, symbol Device:R_Small
- added R108, R109: 10k, Resistor_SMD:R_0402_1005Metric, symbol Device:R_Small
- added R110: 2.2k, Resistor_SMD:R_0402_1005Metric, symbol Device:R_Small
- C14: value DNP -> 12pF; now fitted
- renumbered IC1 to U?
Connections:
- net +3.3V: now also U38.8 (VCC), C31.2, R108.2, R109.2, R110.2
- net DCDC_SW: now also U?.33 (DCDC_SW)
- net GND: now also C15.2, C16.2, C17.2, C18.2, C19.2, U38.4 (GND), U38.9 (EXP), C27.1, C28.1, C29.1, C30.1, C31.1, J3.3, L3.1
- net VDDR: now also U?.45 (VDDR), U?.48 (VDDR_RF); no longer U35.28 (VDDR), U35.32 (VDDR_RF)
- net VDDS: now also C15.1, C16.1, C17.1, C18.1, C19.1, FL1.2, U?.13 (VDDS2), U?.22 (VDDS3), U?.34 (VDDS_DCDC), U?.44 (VDDS); no longer U35.11 (VDDS2), U35.19 (VDDS_DCDC), U35.27 (VDDS)
- net at C25.1, Y1.1: now also U?.4 (X32K_Q2); no longer U35.5 (X32K_Q1)
- net at Y2.1: now also U?.47 (X24M_P); no longer U35.30 (X24M_N)
- net at Y2.3: now also U?.46 (X24M_N); no longer U35.31 (X24M_P)
- net MCU_RESET: now reaches C10.1, R104.2
- net MCU_RESET: now also U?.35 (RESET_N); no longer U35.21 (RESET_N)
- net FLASH_CS: now reaches U38.1 (~{CS})
- net FLASH_CS: now also U?.20 (DIO_14), R110.1
- net MISO: now reaches U38.2 (DO(IO1))
- net MISO: now also U?.28 (DIO_18)
- net at U38.3 (~{WP}): now also R109.1
- net MOSI: now reaches U38.5 (DI(IO0))
- net MOSI: now also U?.29 (DIO_19)
- net SCLK: now reaches U38.6 (CLK)
- net at U38.7 (~{HOLD}): now also R108.1
- net at C24.1, Y1.2: now also U?.3 (X32K_Q1); no longer U35.6 (X32K_Q2)
- net at C14.2: now also C23.1, L3.2
- net at U?.1 (RF_P): now also C14.1
- net at U?.2 (RF_N): now also C22.1
- net MCU_TMS: now reaches U?.24 (JTAG_TMSC)
- net MCU_TCK: now reaches U?.25 (JTAG_TCKC)
- new net: C22.2, C27.2, L4.1
- new net: C23.2, C28.2, L4.2, L5.1
- new net: C29.2, L5.2, L6.1
- new net: J3.1, L6.2
- new net: AE1.1 (A), C30.2, R107.2
- new net: J3.2, R107.1
- new net: U35.11 (VDDS2), U35.19 (VDDS_DCDC), U35.27 (VDDS)
- new net: U35.28 (VDDR), U35.32 (VDDR_RF)
Other:
- note added: "Pin 13"
- note added: "Pin 22"
- note added: "Pin 34"
- note added: "Pin 44"
- note added: "Pin 45"
- note added: "Pin 48"
- moved on the sheet: C10, C11, C12, C13, C15, C16, C17, C18, C19, C24, C25, C26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

Commit message: m
Parts:
- removed C30: 0.5pF, Capacitor_SMD:C_0402_1005Metric, symbol Device:C_Small
- removed J3: ~, symbol Library:M8430-2610RB3
- removed L4: 2.4nH, symbol Device:L_Small
- removed L5, L6: 2nH, symbol Device:L_Small
- removed R107: 0, Resistor_SMD:R_0402_1005Metric, symbol Device:R_Small
- removed U?: CC2640R2FRGZR, QFN50P700X700X100-49N-D, symbol Library:CC2640R2FRGZR
- added C21: 1uF, Capacitor_SMD:C_0402_1005Metric, symbol Device:C_Small
- added J3: U.FL-R-SMT-1_80, Library:UFLRSMT180, symbol Connector:Conn_Coaxial
- added L7: 15nH, symbol Device:L_Small
- added R111: DNM, Resistor_SMD:R_0402_1005Metric, symbol Device:R_Small
- added R112, R113: 0, Resistor_SMD:R_0402_1005Metric, symbol Device:R_Small
- added U39: CC2640R2FRSMR, QFN40P400X400X100-33N-D, symbol Library:CC2640R2FRSMR
- C10: value 1uF -> 100nF
- C14: value 12pF -> 1.2pF
- C23, C29: value 1pF -> DNM; now not fitted
- C27: value 1pF -> 1.2pF
- L3: value 2.4nH -> 2nH
Connections:
- net DCDC_SW: now also U39.18 (DCDC_SW)
- net FLASH_CS: now also U39.24 (DIO_7)
- net GND: now also C14.1, C23.1, C28.2, C29.2, C21.2, J3.2 (Ext), J3.3 (Ext), U39.17 (VSS_3), U39.20 (VSS_4), U39.29 (VSS_5), U39.3 (VSS_1), U39.33 (EP), U39.7 (VSS_2); no longer C28.1, C29.1, L3.1
- net MCU_RESET: now also U39.21 (RESET_N)
- net MISO: now also U39.25 (DIO_8)
- net MOSI: now also U39.26 (DIO_9)
- net SCLK: now also U39.23 (DIO_6)
- net VDDR: now also U39.28 (VDDR), U39.32 (VDDR_RF)
- net VDDS: now also U39.11 (VDDS2), U39.19 (VDDS_DCDC), U39.27 (VDDS)
- net at C27.2: now also L3.1, L7.2, U39.1 (RF_P); no longer C22.2
- net at C14.2, L3.2: now also C22.2; no longer C23.1
- net ANT: now reaches C23.2
- net ANT: now also AE1.1 (A), R113.1; no longer C28.2
- net at C25.1, Y1.1: now also U39.5 (X32K_Q1)
- net at Y2.1: now also C28.1, U39.30 (X24M_N)
- net at Y2.3: now also C29.1, U39.31 (X24M_P)
- net at C22.1: now also R111.1, R112.2
- net at C24.1, Y1.2: now also U39.6 (X32K_Q2)
- new net: R112.1, R113.2
- new net: L7.1, U39.2 (RF_N)
- new net: C21.1, U39.12 (DCOUPL)
- new net: J3.1 (In), R111.2
- new net JTAG_TCK: U39.14 (JTAG_TCKC)
- new net JTAG_TDI: U39.16 (DIO_4)
- new net JTAG_TDO: U39.15 (DIO_3)
- new net JTAG_TMS: U39.13 (JTAG_TMSC)
- new net PWM_EN: U39.8 (DIO_0)
- new net SCL: U39.10 (DIO_2)
- new net SDA: U39.9 (DIO_1)
- no-connect marks 0 -> 1
Other:
- moved on the sheet: AE1, C10, C24, C25, C27, R104, Y1, Y2

Commit message: d
Parts:
- removed C26: 15pF, Capacitor_SMD:C_0402_1005Metric, symbol Device:C_Small
- removed C9: 1uF, Capacitor_SMD:C_0402_1005Metric, symbol Device:C_Small
- removed U35, U39: CC2640R2FRSMR, QFN40P400X400X100-33N-D, symbol Library:CC2640R2FRSMR
- added C20: 1.0uF, Capacitor_SMD:C_0402_1005Metric, symbol Device:C_Small
- added C7, C8: 0.1uF, Capacitor_SMD:C_0402_1005Metric, symbol Device:C_Small
- added D33, D34, D35: TPD1E10B06DPYR, Library:TPD1E10B06DPYR, symbol Diode:ESD5Zxx
- added D36, D37: LTST-C170YKT, Diode_SMD:D_0402_1005Metric, symbol Library:LED
- added J2: 1017457000B11LF, symbol Connector:USB_C_Receptacle
- added J4: Conn_02x05_Counter_Clockwise, symbol Connector_Generic:Conn_02x05_Counter_Clockwise
- added R100, R102, R103, R107, R114: 1k, Resistor_SMD:R_0402_1005Metric, symbol Device:R_Small
- added R105, R106: 100k, Resistor_SMD:R_0402_1005Metric, symbol Device:R_Small
- added U35: CC2640R2FRGZR, QFN50P700X700X100-49N-D, symbol Library:CC2640R2FRGZR
- added U37: CP2102N-A02-GQFN20R, Library:CP2102NA02GQFN20, symbol Library:CP2102N-A02-GQFN20R
Connections:
- net DCDC_SW: now also U35.33 (DCDC_SW)
- net GND: now also C20.2, C7.2, C8.2, D33.2 (A), D34.2 (A), D35.2 (A), J2.13 (SHIELD), J2.A1 (GND), R107.1, R114.1, U35.49 (EP), U37.12 (GND_2), U37.21 (EP_GND), U37.3 (GND_1)
- net JTAG_TCK: now also U35.25 (JTAG_TCKC)
- net JTAG_TMS: now also U35.24 (JTAG_TMSC)
- net MCU_RESET: now also U35.35 (RESET_N)
- net VDDR: now also U35.45 (VDDR), U35.48 (VDDR_RF)
- net VDDS: now also U35.13 (VDDS2), U35.22 (VDDS3), U35.34 (VDDS_DCDC), U35.44 (VDDS)
- net at C27.2, L3.1, L7.2: now also U35.2 (RF_N)
- net at C25.1, Y1.1: now also U35.4 (X32K_Q2)
- net at C28.1, Y2.1: now also U35.47 (X24M_P)
- net at C29.1, Y2.3: now also U35.46 (X24M_N)
- net at L7.1: now also U35.1 (RF_P)
- net at C21.1: now also U35.23 (DCOUPL)
- net at C24.1, Y1.2: now also U35.3 (X32K_Q1)
- new net: C20.1, C8.1, D33.1 (K), J2.A4 (VBUS), J2.B4 (VBUS), U37.7 (VREGIN), U37.8 (VBUS)
- new net: R106.1, U37.17 (RXD)
- new net: R100.2, U37.9 (~{RST})
- new net: J2.B5 (CC2), R114.2
- new net: J2.A5 (CC1), R107.2
- new net: R105.1, U37.18 (TXD)
- new net: D37.1 (K), D37.2 (K), U37.19 (GPIO.3_/_RXT)
- new net: D36.1 (K), D36.2 (K), U37.20 (GPIO.2_/_TXT)
- new net: J2.14 (SHIELD), J2.15 (SHIELD), J2.16 (SHIELD)
- new net D+: D34.1 (K), J2.A6 (D+), J2.B6 (D+), U37.4 (D+)
- new net D-: D35.1 (K), J2.A7 (D-), J2.B7 (D-), U37.5 (D-)
- new net LED_RX: D37.3 (A), D37.4 (A), R103.1
- new net LED_TX: D36.3 (A), D36.4 (A), R102.1
- new net USB_RXD: R106.2
- new net USB_TXD: R105.2
- new net USB_VDD: C7.1, R100.1, R102.2, R103.2, U37.6 (VDD)
- no-connect marks 1 -> 9
Other:
- moved on the sheet: AE1, C10, C11, C12, C13, C14, C15, C16, C17, C18, C19, C21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

Commit message: m
Parts:
- removed J4: Conn_02x05_Counter_Clockwise, symbol Connector_Generic:Conn_02x05_Counter_Clockwise
- added J4: 2002112100010C4LF, symbol Connector_Generic:Conn_02x05_Odd_Even
- added R101, R115: 100k, Resistor_SMD:R_0402_1005Metric, symbol Device:R_Small
- C18: value 22uF -> 10uF
- Y1: footprint (none) -> Library:FC135327680KAAG0
- Y2: footprint (none) -> Library:TSX-3225
- renumbered U35 to U39
Connections:
- net USB_RXD is gone; now on net TXD: R106.2
- net USB_TXD is gone; now on net RXD: R105.2
- net +3.3V: now also J4.1 (Pin_1), R101.1, R115.1
- net CTS: now also U39.29 (DIO_19)
- net FLASH_CS: now also U39.30 (DIO_20)
- net GND: now also J4.3 (Pin_3), J4.5 (Pin_5), J4.9 (Pin_9)
- net JTAG_TCK: now also J4.4 (Pin_4)
- net JTAG_TDI: now also U39.27 (DIO_17), J4.8 (Pin_8)
- net JTAG_TDO: now also U39.26 (DIO_16), J4.6 (Pin_6)
- net JTAG_TMS: now also J4.2 (Pin_2)
- net MCU_RESET: now also J4.10 (Pin_10)
- net MISO: now also U39.14 (DIO_8)
- net MOSI: now also U39.15 (DIO_9)
- net PWM_EN: now also U39.5 (DIO_0)
- net RTS: now also U39.28 (DIO_18)
- net RXD: now also U39.7 (DIO_2)
- net SCL: now also U39.9 (DIO_4), R115.2
- net SCLK: now also U39.16 (DIO_10)
- net SDA: now also U39.10 (DIO_5), R101.2
- net TXD: now also U39.8 (DIO_3)
- net at C27.2, L3.1, L7.2: now also U39.1 (RF_P); no longer U39.2 (RF_N)
- net at C25.1, U39.4 (X32K_Q2): now also Y1.2; no longer Y1.1
- net at L7.1: now also U39.2 (RF_N); no longer U39.1 (RF_P)
- net at C24.1, U39.3 (X32K_Q1): now also Y1.1; no longer Y1.2
- no-connect marks 9 -> 10
Other:
- moved on the sheet: AE1, C10, C14, C20, C21, C22, C23, C24, C25, C27, C28, C29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

Commit message: d
Connections:
- net CTS: now also U37.15 (CTS)
- net RTS: now also U37.16 (RTS)
- no-connect marks 10 -> 8
Changed lines of the file:
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@@
-	)
-	(no_connect
-		(at 163.83 173.99)
 	)
 	(no_connect
@@
 	)
 	(no_connect
-		(at 163.83 168.91)
-	)
-	(no_connect
 		(at 163.83 163.83)
 	)
@@
 	(wire
 		(pts
+			(xy 165.1 173.99) (xy 163.83 173.99)
+		)
+		(stroke
+			(width 0)
+			(type default)
+		)
+	)
+	(wire
+		(pts
 			(xy 116.84 44.45) (xy 118.11 44.45)
 		)
@@
 		(pts
 			(xy 114.3 173.99) (xy 114.3 177.8)
+		)
+		(stroke
+			(width 0)
+			(type default)
+		)
+	)
+	(wire
+		(pts
+			(xy 165.1 168.91) (xy 163.83 168.91)
 		)
 		(stroke
@@
 		)
 	)
+	(hierarchical_label "RTS"
+		(shape input)
+		(at 165.1 173.99 0)
+		(effects
+			(font
+				(size 1.27 1.27)
+			)
+			(justify left)
+		)
+	)
 	(hierarchical_label "CTS"
 		(shape input)
@@
 		)
 	)
+	(hierarchical_label "CTS"
+		(shape input)
+		(at 165.1 168.91 0)
+		(effects
+			(font
+				(size 1.27 1.27)
+			)
+			(justify left)
+		)
+	)

Commit message: m
Parts:
- R105, R106: value 100k -> 0
Connections:
- net CTS: now also U39.39 (DIO_26); no longer U39.29 (DIO_19)
- net FLASH_CS: now also U39.40 (DIO_27); no longer U39.30 (DIO_20)
- net MISO: now also U39.43 (DIO_30); no longer U39.14 (DIO_8)
- net MOSI: now also U39.42 (DIO_29); no longer U39.15 (DIO_9)
- net PWM_EN: now also U39.30 (DIO_20); no longer U39.5 (DIO_0)
- net RTS: now also U39.38 (DIO_25); no longer U39.28 (DIO_18)
- net SCL: now also U39.32 (DIO_22); no longer R115.2, U39.9 (DIO_4)
- net SCLK: now also U39.41 (DIO_28); no longer U39.16 (DIO_10)
- net SDA: now also U39.31 (DIO_21); no longer R101.2, U39.10 (DIO_5)
- net RX: now reaches U39.36 (DIO_23)
- net RX: now also R105.2
- net TX: now reaches U39.37 (DIO_24)
- net TX: now also R106.2
- net RXD: no longer names the net of U39.7 (DIO_2)
- net RXD: no longer R105.2
- net TXD: no longer names the net of U39.8 (DIO_3)
- net TXD: no longer R106.2
- new net: R115.2, U39.9 (DIO_4)
- new net: R101.2, U39.10 (DIO_5)
