File: Hardware/Ring-Light v5/Ring-Light.kicad_pcb (KiCad board)
At the start: 4 copper layers, 115 x 146.1 mm, 251 parts, among them J1 694106301002, J2 1017457000B11LF, J3 U.FL-R-SMT-1_80, J4 2002112100010C4LF, J5 640445-2, Q1 PMOS, U1 NCR321PASX, U10 NCR321PASX, U11 NCR321PASX, U12 NCR321PASX, U13 NCR321PASX, U14 NCR321PASX, U15 NCR321PASX, U16 NCR321PASX, U17 NCR321PASX, U18 NCR321PASX, U19 NCR321PASX, U2 NCR321PASX, U20 NCR321PASX, U21 NCR321PASX, U22 NCR321PASX, U23 NCR321PASX, U24 NCR321PASX, U25 NCR321PASX, U26 NCR321PASX, U27 NCR321PASX, U28 NCR321PASX, U29 NCR321PASX, U3 NCR321PASX, U30 NCR321PASX, U31 NCR321PASX, U32 NCR321PASX, U33 PCA9685BS,118, U34 PCA9685BS,118, U36 TPS62177DQC, U37 CP2102N-A02-GQFN20R, U38 W25X40CLUXIG_TR, U39 CC2640R2FRGZR, U4 NCR321PASX, U5 NCR321PASX, U6 NCR321PASX, U7 NCR321PASX, U8 NCR321PASX, U9 NCR321PASX, Y1 32.768kHz, Y2 24MHz

Commit message: m
Parts:
- added C28: 12pF, Capacitor_SMD:C_0402_1005Metric, F.Cu at (106.1, 49.5)
- added C29: 12pF, Capacitor_SMD:C_0402_1005Metric, F.Cu at (109.2, 52.9)
- added R101: 10k, Resistor_SMD:R_0402_1005Metric, F.Cu at (95.0, 48.5)
- L2: footprint Inductor_SMD:L_0402_1005Metric -> Inductor_SMD:L_0805_2012Metric
- moved R65 35.8 mm to (90.8, 50.1)
- moved J4 24.1 mm to (80.0, 21.3)
- moved FL1 18.0 mm to (78.7, 54.4), turned to 90 degrees
- moved C10 12.1 mm to (96.1, 47.5), turned to 180 degrees
- moved R104 11.1 mm to (96.0, 46.4), turned to 0 degrees
- moved C19 4.34 mm to (94.1, 46.4)
- moved C18 2.45 mm to (94.1, 45.3)
- moved C11 2.28 mm to (92.1, 45.3), turned to 0 degrees
- moved L2 2.25 mm to (93.2, 43.8)
- moved C1 1.38 mm to (85.5, 48.6), turned to 180 degrees
- moved C2 0.99 mm to (97.2, 48.5)
- moved R119 0.95 mm to (90.8, 48.0)
- moved R74 0.83 mm to (81.8, 60.5)
- moved R75 0.83 mm to (83.2, 60.5)
- moved R76 0.83 mm to (84.5, 60.5)
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Connections:
- U33 pad 1: unconnected-(U33-A3-Pad1) -> GND
- U33 pad 2: unconnected-(U33-A4-Pad2) -> GND
- U33 pad 21: unconnected-(U33-A5-Pad21) -> GND
- U33 pad 26: unconnected-(U33-A0-Pad26) -> GND
- U33 pad 27: unconnected-(U33-A1-Pad27) -> GND
- U33 pad 28: unconnected-(U33-A2-Pad28) -> GND
- U34 pad 1: unconnected-(U34-A3-Pad1) -> GND
- U34 pad 2: unconnected-(U34-A4-Pad2) -> GND
- U34 pad 21: unconnected-(U34-A5-Pad21) -> GND
- U34 pad 26: unconnected-(U34-A0-Pad26) -> Net-(U34-A0)
- U34 pad 27: unconnected-(U34-A1-Pad27) -> GND
- U34 pad 28: unconnected-(U34-A2-Pad28) -> GND
- U39 pad 31: /MCU/SCL -> /MCU/SDA
- U39 pad 32: /MCU/SDA -> /MCU/SCL
- U39 pad 36: MISO -> CTS
- U39 pad 37: MOSI -> RTS
- U39 pad 38: SCLK -> TX
- U39 pad 40: RX -> MOSI
- U39 pad 41: TX -> SCLK
- U39 pad 42: RTS -> MISO
- U39 pad 43: CTS -> RX
Routing:
- net +3.3V: track 28.2 -> 82.9 mm, vias 2 -> 11
- net /MCU/SDA: track 0.00 -> 34.0 mm, vias 0 -> 3
- net /MCU/SCL: track 0.00 -> 32.0 mm, vias 0 -> 3
- net /MCU/PWM_EN: track 6.93 -> 37.9 mm, vias 2 -> 4
- net RTS: track 1.38 -> 24.2 mm, vias 0 -> 2
- net CTS: track 2.38 -> 24.1 mm, vias 0 -> 2
- net TX: track 0.79 -> 21.8 mm, vias 0 -> 2
- net SCLK: track 0.87 -> 21.8 mm, vias 0 -> 2
- net MOSI: track 1.01 -> 21.0 mm, vias 0 -> 2
- net RX: track 0.84 -> 17.5 mm, vias 0 -> 2
- net VDDR: track 25.2 -> 41.5 mm, vias 1 -> 2
- net MISO: track 3.18 -> 18.9 mm, vias 1 -> 2
- net FLASH_CS: track 5.83 -> 19.4 mm, vias 0 -> 2
- net /LEDs_1-16/PWM1: track 15.1 -> 5.29 mm
- net /LEDs_1-16/PWM8: track 10.4 -> 2.30 mm
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
Commit message: m
Parts:
- removed the REF** at (135.3, 34.7)
- added D1: LED, Library:GWJTLRS1EMLVL5XX531, F.Cu at (94.1, 76.7)
- added D10, D48: LED, Library:GWJTLRS1EMLVL5XX531, F.Cu at (52.9, 126.9)
- added D11, D49: LED, Library:GWJTLRS1EMLVL5XX531, F.Cu at (55.3, 134.8)
- added D12, D50: LED, Library:GWJTLRS1EMLVL5XX531, F.Cu at (59.2, 142.0)
- added D13, D51: LED, Library:GWJTLRS1EMLVL5XX531, F.Cu at (64.4, 148.4)
- added D14, D52: LED, Library:GWJTLRS1EMLVL5XX531, F.Cu at (70.8, 153.6)
- added D15, D53: LED, Library:GWJTLRS1EMLVL5XX531, F.Cu at (78.1, 157.5)
- added D16, D54: LED, Library:GWJTLRS1EMLVL5XX531, F.Cu at (85.9, 159.9)
- added D17, D55: LED, Library:GWJTLRS1EMLVL5XX531, F.Cu at (94.1, 160.7)
- added D18, D56: LED, Library:GWJTLRS1EMLVL5XX531, F.Cu at (102.3, 159.9)
- added D19, D57: LED, Library:GWJTLRS1EMLVL5XX531, F.Cu at (110.2, 157.5)
- added D2 (x2): LED, Library:GWJTLRS1EMLVL5XX531, F.Cu at (85.9, 77.5)
- added D20, D58: LED, Library:GWJTLRS1EMLVL5XX531, F.Cu at (117.5, 153.6)
- added D21, D59: LED, Library:GWJTLRS1EMLVL5XX531, F.Cu at (123.8, 148.4)
- added D22, D60: LED, Library:GWJTLRS1EMLVL5XX531, F.Cu at (129.0, 142.0)
- added D23, D61: LED, Library:GWJTLRS1EMLVL5XX531, F.Cu at (132.9, 134.7)
- added D24, D62: LED, Library:GWJTLRS1EMLVL5XX531, F.Cu at (135.3, 126.9)
- added D25, D63: LED, Library:GWJTLRS1EMLVL5XX531, F.Cu at (136.1, 118.7)
- added D26, D64: LED, Library:GWJTLRS1EMLVL5XX531, F.Cu at (135.3, 110.5)
- added D27, D65: LED, Library:GWJTLRS1EMLVL5XX531, F.Cu at (132.9, 102.6)
- added D28, D66: LED, Library:GWJTLRS1EMLVL5XX531, F.Cu at (129.0, 95.3)
- added D29, D67: LED, Library:GWJTLRS1EMLVL5XX531, F.Cu at (123.8, 89.0)
- added D3, D41: LED, Library:GWJTLRS1EMLVL5XX531, F.Cu at (78.0, 79.9)
- added D30, D68: LED, Library:GWJTLRS1EMLVL5XX531, F.Cu at (117.4, 83.7)
- added D31, D69: LED, Library:GWJTLRS1EMLVL5XX531, F.Cu at (110.2, 79.9)
- added D32: LED, Library:GWJTLRS1EMLVL5XX531, F.Cu at (102.3, 77.5)
- added D4, D42: LED, Library:GWJTLRS1EMLVL5XX531, F.Cu at (70.8, 83.8)
- added D43, D5: LED, Library:GWJTLRS1EMLVL5XX531, F.Cu at (64.4, 89.0)
- added D44, D6: LED, Library:GWJTLRS1EMLVL5XX531, F.Cu at (59.2, 95.3)
- added D45, D7: LED, Library:GWJTLRS1EMLVL5XX531, F.Cu at (55.3, 102.6)
- added D46, D8: LED, Library:GWJTLRS1EMLVL5XX531, F.Cu at (52.9, 110.5)
- added D47, D9: LED, Library:GWJTLRS1EMLVL5XX531, F.Cu at (52.1, 118.7)
- added J6: Conn_01x01, , F.Cu at (64.2, 54.8)
- added J7: Conn_01x01, , F.Cu at (61.0, 54.8)
- added J8: Conn_01x01, , F.Cu at (83.3, 82.8)
- added J9: Conn_01x01, , F.Cu at (70.3, 89.7)
- D33, D34, D35: footprint Library:TPD1E10B06DPYR -> Diode_SMD:D_SOD-523
- D36, D37: value LTST-C170YKT -> VLMY1500-GS08; footprint Diode_SMD:D_0402_1005Metric -> LED_SMD:LED_0402_1005Metric
- MH1: renamed from REF**12; footprint MountingHole:MountingHole_2.2mm_M2 -> Library:MountingHole_2.2mm_M2
- MH2: renamed from REF**8; footprint MountingHole:MountingHole_2.2mm_M2 -> Library:MountingHole_2.2mm_M2
- MH3: renamed from REF**4; footprint MountingHole:MountingHole_2.2mm_M2 -> Library:MountingHole_2.2mm_M2
- MH4: renamed from REF**; footprint MountingHole:MountingHole_2.2mm_M2 -> Library:MountingHole_2.2mm_M2
- MH5: renamed from REF**28; footprint MountingHole:MountingHole_2.2mm_M2 -> Library:MountingHole_2.2mm_M2
- MH5: renamed from REF**24; footprint MountingHole:MountingHole_2.2mm_M2 -> Library:MountingHole_2.2mm_M2
- MH6: renamed from REF**20; footprint MountingHole:MountingHole_2.2mm_M2 -> Library:MountingHole_2.2mm_M2
- MH7: renamed from REF**16; footprint MountingHole:MountingHole_2.2mm_M2 -> Library:MountingHole_2.2mm_M2
- Q1: value PMOS -> SQJ415EP-T1_GE3
- moved J4 24.0 mm to (91.5, 42.5), turned to -90 degrees
- moved D70 8.23 mm to (102.3, 77.5), turned to -101.25 degrees
- moved C3 2.49 mm to (64.8, 46.7), turned to 180 degrees
- moved D37 1.23 mm to (114.5, 59.3), turned to -90 degrees
- moved D36 1.11 mm to (113.3, 59.3), turned to -90 degrees
- moved D34 0.19 mm to (118.5, 56.3)
- moved D35 0.14 mm to (118.5, 53.6)
- moved R103 0.13 mm to (112.2, 59.3), turned to -90 degrees
- moved R107 0.11 mm to (117.3, 59.2)
- turned R102 to -90 degrees
- turned Y1 to 0 degrees
- renumbered D1 to D70
Connections:
- D36 pad 1: Net-(U37-GPIO.2_/_TXT) -> Net-(D36-K)
- D36 pad 2: Net-(U37-GPIO.2_/_TXT) -> Net-(D36-A)
- D37 pad 1: Net-(U37-GPIO.3_/_RXT) -> Net-(D37-K)
- D37 pad 2: Net-(U37-GPIO.3_/_RXT) -> Net-(D37-A)
- J1 pad 1: GND -> Net-(F1-Pad1)
- J1 pad 2: Net-(F1-Pad1) -> GND
- R102 pad 1: /MCU/LED_TX -> USB_VDD
- R102 pad 2: USB_VDD -> Net-(D37-A)
- R103 pad 1: /MCU/LED_RX -> USB_VDD
- R103 pad 2: USB_VDD -> Net-(D36-A)
- R66 pad 1: /LEDs_1-16/PWM1 -> /LEDs_1-16/PWM8
- R67 pad 1: /LEDs_1-16/PWM3 -> /LEDs_1-16/PWM6
- R68 pad 1: /LEDs_1-16/PWM5 -> /LEDs_1-16/PWM4
- R69 pad 1: /LEDs_1-16/PWM7 -> /LEDs_1-16/PWM2
- R70 pad 1: /LEDs_1-16/PWM9 -> /LEDs_1-16/PWM16
- R71 pad 1: /LEDs_1-16/PWM11 -> /LEDs_1-16/PWM14
- R72 pad 1: /LEDs_1-16/PWM13 -> /LEDs_1-16/PWM12
- R73 pad 1: /LEDs_1-16/PWM15 -> /LEDs_1-16/PWM10
- R74 pad 1: /LEDs_1-16/PWM2 -> /LEDs_1-16/PWM7
- R75 pad 1: /LEDs_1-16/PWM4 -> /LEDs_1-16/PWM5
- R76 pad 1: /LEDs_1-16/PWM6 -> /LEDs_1-16/PWM3
- R77 pad 1: /LEDs_1-16/PWM8 -> /LEDs_1-16/PWM1
- R78 pad 1: /LEDs_1-16/PWM10 -> /LEDs_1-16/PWM15
- R79 pad 1: /LEDs_1-16/PWM12 -> /LEDs_1-16/PWM13
- R80 pad 1: /LEDs_1-16/PWM14 -> /LEDs_1-16/PWM11
- R81 pad 1: /LEDs_1-16/PWM16 -> /LEDs_1-16/PWM9
- R83 pad 1: /LEDs_17-32/PWM17 -> /LEDs_17-32/PWM24
- R84 pad 1: /LEDs_17-32/PWM19 -> /LEDs_17-32/PWM22
- R85 pad 1: /LEDs_17-32/PWM21 -> /LEDs_17-32/PWM20
- R86 pad 1: /LEDs_17-32/PWM23 -> /LEDs_17-32/PWM18
- R87 pad 1: /LEDs_17-32/PWM25 -> /LEDs_17-32/PWM32
- R88 pad 1: /LEDs_17-32/PWM27 -> /LEDs_17-32/PWM30
- R89 pad 1: /LEDs_17-32/PWM29 -> /LEDs_17-32/PWM28
- R90 pad 1: /LEDs_17-32/PWM31 -> /LEDs_17-32/PWM26
- R91 pad 1: /LEDs_17-32/PWM18 -> /LEDs_17-32/PWM23
- R92 pad 1: /LEDs_17-32/PWM20 -> /LEDs_17-32/PWM21
- R93 pad 1: /LEDs_17-32/PWM22 -> /LEDs_17-32/PWM19
- R94 pad 1: /LEDs_17-32/PWM24 -> /LEDs_17-32/PWM17
- R95 pad 1: /LEDs_17-32/PWM26 -> /LEDs_17-32/PWM31
- R96 pad 1: /LEDs_17-32/PWM28 -> /LEDs_17-32/PWM29
- R97 pad 1: /LEDs_17-32/PWM30 -> /LEDs_17-32/PWM27
- R98 pad 1: /LEDs_17-32/PWM32 -> /LEDs_17-32/PWM25
- U37 pad 19: Net-(U37-GPIO.3_/_RXT) -> Net-(D36-K)
- U37 pad 20: Net-(U37-GPIO.2_/_TXT) -> Net-(D37-K)
- Y1 pad 1: Net-(U39-X32K_Q1) -> Net-(U39-X32K_Q2)
- Y1 pad 2: Net-(U39-X32K_Q2) -> Net-(U39-X32K_Q1)
Routing:
- net +3.3V: track 82.9 -> 102.4 mm, vias 11 -> 13
- net VDDS: track 42.9 -> 54.5 mm, vias 4 -> 12
- net +12V: track 0.00 -> 11.3 mm, vias 160 -> 178
- net /LEDs_1-16/PWM1: track 5.29 -> 16.5 mm, vias 0 -> 2
- net Net-(D39-K): track 0.00 -> 10.9 mm, vias 0 -> 10
- net JTAG_TMS: track 0.00 -> 10.0 mm, vias 0 -> 1
- net JTAG_TDI: track 0.00 -> 9.96 mm, vias 0 -> 1
- net JTAG_TDO: track 0.00 -> 9.24 mm, vias 0 -> 1
- net JTAG_TCK: track 0.00 -> 8.72 mm, vias 0 -> 1
- net /LEDs_1-16/PWM2: track 2.33 -> 10.9 mm
- net MCU_RESET: track 3.35 -> 11.6 mm, vias 0 -> 2
- net /LEDs_17-32/PWM32: track 2.60 -> 10.4 mm
- net Net-(U34-LED0): track 0.70 -> 8.06 mm
- net Net-(U33-LED0): track 0.70 -> 8.00 mm
- net Net-(U34-LED15): track 2.76 -> 9.82 mm, vias 1 -> 2
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- added copper zone on In1.Cu, net +3.3V
- added copper zone on B.Cu, net Net-(D38-A1)
- added copper zone on In1.Cu, net Net-(D38-A1)
- added copper zone on In2.Cu, net Net-(D38-A1)
- added copper zone on B.Cu, net Net-(D39-K)
- added copper zone on In1.Cu, net Net-(D39-K)
- added copper zone on In2.Cu, net Net-(D39-K)
- added copper zone on In1.Cu, net Net-(F1-Pad1)
- added copper zone on F.Cu, net VDDS
- added copper zone on In1.Cu, net VDDS

Commit message: m
Other:
- board text added: "12V"
- board text added: "2621"
- board text added: "RINGLIGHT 1.0.0"
