File: Hardware/Ring-Light v5/LEDs_1-16.kicad_sch (KiCad schematic)
At the start: 64 parts, among them U1 NCR321PASX, U10 NCR321PASX, U11 NCR321PASX, U12 NCR321PASX, U13 NCR321PASX, U14 NCR321PASX, U15 NCR321PASX, U16 NCR321PASX, U2 NCR321PASX, U3 NCR321PASX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

Commit message: m
Other:
- note added: "LEDS 1-16"
Changed lines of the file:
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@@
 	(generator_version "9.0")
 	(paper "USLegal")
+	(text "LEDS 1-16\n"
+		(exclude_from_sim no)
+		(at 109.728 186.69 0)
+		(effects
+			(font
+				(size 2.54 2.54)
+			)
+		)
+	)
 	(junction
 		(at 210.82 57.15)
@@
 	)
 	(junction
+		(at 26.67 54.61)
+		(diameter 0)
+		(color 0 0 0 0)
+	)
+	(junction
 		(at 259.08 57.15)
 		(diameter 0)
@@
 	(wire
 		(pts
+			(xy 26.67 54.61) (xy 26.67 55.88)
+		)
+		(stroke
+			(width 0)
+			(type default)
+		)
+	)
+	(wire
+		(pts
 			(xy 124.46 48.26) (xy 124.46 55.88)
 		)
@@
 	(wire
 		(pts
+			(xy 19.05 54.61) (xy 26.67 54.61)
+		)
+		(stroke
+			(width 0)
+			(type default)
+		)
+	)
+	(wire
+		(pts
 			(xy 195.58 27.94) (xy 195.58 34.29)
 		)
@@
 	(wire
 		(pts
-			(xy 26.67 48.26) (xy 26.67 55.88)
+			(xy 26.67 48.26) (xy 26.67 54.61)
 		)
 		(stroke
@@
 	)
 	(symbol
-		(lib_name "NCR321PASX_1")
 		(lib_id "Library:NCR321PASX")
 		(at 142.24 100.33 0)
@@
 	)
 	(symbol
-		(lib_name "NCR321PASX_1")
 		(lib_id "Library:NCR321PASX")
 		(at 190.5 100.33 0)
@@
 	)
 	(symbol
-		(lib_name "NCR321PASX_1")
 		(lib_id "Library:NCR321PASX")
 		(at 190.5 49.53 0)
@@
 	)
 	(symbol
-		(lib_name "NCR321PASX_1")
 		(lib_id "Library:NCR321PASX")
 		(at 287.02 49.53 0)
@@
 	)
 	(symbol
-		(lib_name "NCR321PASX_1")
 		(lib_id "Library:NCR321PASX")
 		(at 140.97 49.53 0)
@@
 	)
 	(symbol
-		(lib_name "NCR321PASX_1")
 		(lib_id "Library:NCR321PASX")
 		(at 92.71 151.13 0)
@@
 	)
 	(symbol
-		(lib_name "NCR321PASX_1")
 		(lib_id "Library:NCR321PASX")
 		(at 190.5 151.13 0)
@@
 	)
 	(symbol
-		(lib_name "NCR321PASX_1")
 		(lib_id "Library:NCR321PASX")
 		(at 238.76 100.33 0)
@@
 	)
 	(symbol
-		(lib_name "NCR321PASX_1")
 		(lib_id "Library:NCR321PASX")
 		(at 288.29 100.33 0)
@@
 	)
 	(symbol
-		(lib_name "NCR321PASX_1")
 		(lib_id "Library:NCR321PASX")
 		(at 140.97 151.13 0)
@@
 	)
 	(symbol
-		(lib_name "NCR321PASX_1")
 		(lib_id "Library:NCR321PASX")
 		(at 238.76 49.53 0)
@@
 	)
 	(symbol
-		(lib_name "NCR321PASX_1")
 		(lib_id "Library:NCR321PASX")
 		(at 92.71 100.33 0)
@@
 	)
 	(symbol
-		(lib_name "NCR321PASX_1")
 		(lib_id "Library:NCR321PASX")
 		(at 43.18 151.13 0)
@@
 	)
 	(symbol
-		(lib_name "NCR321PASX_1")
 		(lib_id "Library:NCR321PASX")
 		(at 43.18 100.33 0)
@@
 	)
 	(symbol
-		(lib_name "NCR321PASX_1")
+		(lib_id "power:PWR_FLAG")
+		(at 19.05 54.61 0)
+		(unit 1)
+		(exclude_from_sim no)
+		(in_bom yes)
+		(on_board yes)
+		(dnp no)
+		(fields_autoplaced yes)
+		(property "Reference" "#FLG06"
+			(at 19.05 52.705 0)
+			(effects
+				(font
+					(size 1.27 1.27)
+				)
+				(hide yes)
+			)
+		)
+		(property "Value" "PWR_FLAG"
+			(at 19.05 49.53 0)
+			(effects
+				(font
+					(size 1.27 1.27)
+				)
+			)
+		)
+		(property "Footprint" ""
+			(at 19.05 54.61 0)
+			(effects
+				(font
+					(size 1.27 1.27)
+				)
+				(hide yes)
+			)
+		)
+		(property "Datasheet" "~"
+			(at 19.05 54.61 0)
+			(effects
+				(font
+					(size 1.27 1.27)
+				)
+				(hide yes)
+			)
+		)
+		(property "Description" "Special symbol for telling ERC where power comes from"
+			(at 19.05 54.61 0)
+			(effects
+				(font
+					(size 1.27 1.27)
+				)
+				(hide yes)
+			)
+		)
+		(pin "1"
+		)
+		(instances
+			(project "Ring-Light"
+				(path "/7146df34-bb5a-4ab6-bd6d-8aad9726b4e6/cbf711bc-3cf1-4aff-a749-f3b8b0d61f93"
+					(reference "#FLG06")
+					(unit 1)
+				)
+			)
+		)
+	)
+	(symbol
 		(lib_id "Library:NCR321PASX")
 		(at 43.18 49.53 0)
@@
 	)
 	(symbol
-		(lib_name "NCR321PASX_1")
 		(lib_id "Library:NCR321PASX")
 		(at 92.71 49.53 0)
