File: Hardware/Ring-Light v5/LEDs_17-32.kicad_sch (KiCad schematic)
At the start: 64 parts, among them U17 NCR321PASX, U18 NCR321PASX, U19 NCR321PASX, U20 NCR321PASX, U21 NCR321PASX, U22 NCR321PASX, U23 NCR321PASX, U24 NCR321PASX, U25 NCR321PASX, U26 NCR321PASX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

Commit message: m
Other:
- note added: "LEDS 17-32"
Changed lines of the file:
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@@
 	(generator_version "9.0")
 	(paper "USLegal")
+	(text "LEDS 17-32\n"
+		(exclude_from_sim no)
+		(at 119.126 188.722 0)
+		(effects
+			(font
+				(size 2.54 2.54)
+			)
+		)
+	)
 	(junction
 		(at 298.45 34.29)
@@
 	)
 	(symbol
-		(lib_name "NCR321PASX_1")
 		(lib_id "Library:NCR321PASX")
 		(at 293.37 49.53 0)
@@
 	)
 	(symbol
-		(lib_name "NCR321PASX_1")
 		(lib_id "Library:NCR321PASX")
 		(at 97.79 100.33 0)
@@
 	)
 	(symbol
-		(lib_name "NCR321PASX_1")
 		(lib_id "Library:NCR321PASX")
 		(at 148.59 100.33 0)
@@
 	)
 	(symbol
-		(lib_name "NCR321PASX_1")
 		(lib_id "Library:NCR321PASX")
 		(at 48.26 100.33 0)
@@
 	)
 	(symbol
-		(lib_name "NCR321PASX_1")
 		(lib_id "Library:NCR321PASX")
 		(at 294.64 100.33 0)
@@
 	)
 	(symbol
-		(lib_name "NCR321PASX_1")
 		(lib_id "Library:NCR321PASX")
 		(at 146.05 49.53 0)
@@
 	)
 	(symbol
-		(lib_name "NCR321PASX_1")
 		(lib_id "Library:NCR321PASX")
 		(at 243.84 49.53 0)
@@
 	)
 	(symbol
-		(lib_name "NCR321PASX_1")
 		(lib_id "Library:NCR321PASX")
 		(at 48.26 49.53 0)
@@
 	)
 	(symbol
-		(lib_name "NCR321PASX_1")
 		(lib_id "Library:NCR321PASX")
 		(at 97.79 151.13 0)
@@
 	)
 	(symbol
-		(lib_name "NCR321PASX_1")
 		(lib_id "Library:NCR321PASX")
 		(at 48.26 151.13 0)
@@
 	)
 	(symbol
-		(lib_name "NCR321PASX_1")
 		(lib_id "Library:NCR321PASX")
 		(at 198.12 152.4 0)
@@
 	)
 	(symbol
-		(lib_name "NCR321PASX_1")
 		(lib_id "Library:NCR321PASX")
 		(at 196.85 100.33 0)
@@
 	)
 	(symbol
-		(lib_name "NCR321PASX_1")
 		(lib_id "Library:NCR321PASX")
 		(at 148.59 152.4 0)
@@
 	)
 	(symbol
-		(lib_name "NCR321PASX_1")
 		(lib_id "Library:NCR321PASX")
 		(at 97.79 49.53 0)
@@
 	)
 	(symbol
-		(lib_name "NCR321PASX_1")
 		(lib_id "Library:NCR321PASX")
 		(at 195.58 49.53 0)
@@
 	)
 	(symbol
-		(lib_name "NCR321PASX_1")
 		(lib_id "Library:NCR321PASX")
 		(at 245.11 100.33 0)
