File: Hardware/Ring-Light v5/Ring-Light.kicad_sch (KiCad schematic)
At the start: 21 parts, among them J1 694106301002, J5 640445-2, Q1 PMOS, U36 TPS62177DQC

Commit message: m
Other:
- moved on the sheet: C26, C3, C30, C4, C9
Changed lines of the file:
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@@
 	(wire
 		(pts
-			(xy 104.14 35.56) (xy 104.14 49.53)
+			(xy 104.14 40.64) (xy 104.14 49.53)
 		)
 		(stroke
@@
 	(wire
 		(pts
-			(xy 104.14 29.21) (xy 104.14 30.48)
+			(xy 104.14 29.21) (xy 104.14 35.56)
 		)
 		(stroke
@@
 	(wire
 		(pts
-			(xy 95.25 35.56) (xy 95.25 49.53)
+			(xy 95.25 40.64) (xy 95.25 49.53)
 		)
 		(stroke
@@
 	(wire
 		(pts
-			(xy 138.43 29.21) (xy 138.43 30.48)
+			(xy 138.43 29.21) (xy 138.43 35.56)
 		)
 		(stroke
@@
 	(wire
 		(pts
-			(xy 138.43 49.53) (xy 138.43 35.56)
+			(xy 138.43 49.53) (xy 138.43 40.64)
 		)
 		(stroke
@@
 	(wire
 		(pts
-			(xy 127 30.48) (xy 127 29.21)
+			(xy 127 35.56) (xy 127 29.21)
 		)
 		(stroke
@@
 	(wire
 		(pts
-			(xy 115.57 29.21) (xy 115.57 30.48)
+			(xy 115.57 29.21) (xy 115.57 35.56)
 		)
 		(stroke
@@
 	(wire
 		(pts
-			(xy 95.25 29.21) (xy 95.25 30.48)
+			(xy 95.25 29.21) (xy 95.25 35.56)
 		)
 		(stroke
@@
 	(wire
 		(pts
-			(xy 127 35.56) (xy 127 49.53)
+			(xy 127 40.64) (xy 127 49.53)
 		)
 		(stroke
@@
 	(wire
 		(pts
-			(xy 115.57 35.56) (xy 115.57 49.53)
+			(xy 115.57 40.64) (xy 115.57 49.53)
 		)
 		(stroke
@@
 	(symbol
 		(lib_id "Device:C_Small")
-		(at 104.14 33.02 0)
+		(at 104.14 38.1 0)
 		(unit 1)
 		(exclude_from_sim no)
@@
 		(dnp no)
 		(property "Reference" "C26"
-			(at 106.68 32.258 0)
+			(at 106.68 37.338 0)
 			(effects
 				(font
@@
 		)
 		(property "Value" "4.7uF"
-			(at 106.68 34.036 0)
+			(at 106.68 39.116 0)
 			(effects
 				(font
@@
 		)
 		(property "Footprint" "Capacitor_SMD:C_0805_2012Metric"
-			(at 104.14 33.02 0)
+			(at 104.14 38.1 0)
 			(effects
 				(font
@@
 		)
 		(property "Datasheet" "~"
-			(at 104.14 33.02 0)
+			(at 104.14 38.1 0)
 			(effects
 				(font
@@
 		)
 		(property "Description" "Unpolarized capacitor, small symbol"
-			(at 104.14 33.02 0)
+			(at 104.14 38.1 0)
 			(effects
 				(font
@@
 					(unit 1)
 				)
-				(path "/7146df34-bb5a-4ab6-bd6d-8aad9726b4e6/fdaac70b-54b8-4a78-a210-de38a02463ef"
-					(reference "R118")
-					(unit 1)
-				)
 			)
 		)
@@
 	(symbol
 		(lib_id "Device:C_Polarized_Small")
-		(at 127 33.02 0)
+		(at 127 38.1 0)
 		(unit 1)
 		(exclude_from_sim no)
@@
 		(fields_autoplaced yes)
 		(property "Reference" "C4"
-			(at 129.54 31.2038 0)
+			(at 129.54 36.2838 0)
 			(effects
 				(font
@@
 		)
 		(property "Value" "100uF"
-			(at 129.54 33.7438 0)
+			(at 129.54 38.8238 0)
 			(effects
 				(font
@@
 		)
 		(property "Footprint" ""
-			(at 127 33.02 0)
+			(at 127 38.1 0)
 			(effects
 				(font
@@
 		)
 		(property "Datasheet" "~"
-			(at 127 33.02 0)
+			(at 127 38.1 0)
 			(effects
 				(font
@@
 		)
 		(property "Description" "Polarized capacitor, small symbol"
-			(at 127 33.02 0)
+			(at 127 38.1 0)
 			(effects
 				(font
@@
 	(symbol
 		(lib_id "Device:C_Small")
-		(at 115.57 33.02 0)
+		(at 115.57 38.1 0)
 		(unit 1)
 		(exclude_from_sim no)
@@
 		(dnp no)
 		(property "Reference" "C9"
-			(at 118.11 32.258 0)
+			(at 118.11 37.338 0)
 			(effects
 				(font
@@
 		)
 		(property "Value" "10uF"
-			(at 118.11 34.036 0)
+			(at 118.11 39.116 0)
 			(effects
 				(font
@@
 		)
 		(property "Footprint" "Capacitor_SMD:C_0805_2012Metric"
-			(at 115.57 33.02 0)
+			(at 115.57 38.1 0)
 			(effects
 				(font
@@
 		)
 		(property "Datasheet" "~"
-			(at 115.57 33.02 0)
+			(at 115.57 38.1 0)
 			(effects
 				(font
@@
 		)
 		(property "Description" "Unpolarized capacitor, small symbol"
-			(at 115.57 33.02 0)
+			(at 115.57 38.1 0)
 			(effects
 				(font
@@
 	(symbol
 		(lib_id "Device:C_Small")
-		(at 95.25 33.02 0)
+		(at 95.25 38.1 0)
 		(unit 1)
 		(exclude_from_sim no)
@@
 		(dnp no)
 		(property "Reference" "C30"
-			(at 97.79 32.258 0)
+			(at 97.79 37.338 0)
 			(effects
 				(font
@@
 		)
 		(property "Value" "1uF"
-			(at 97.79 34.036 0)
+			(at 97.79 39.116 0)
 			(effects
 				(font
@@
 		)
 		(property "Footprint" "Capacitor_SMD:C_0805_2012Metric"
-			(at 95.25 33.02 0)
+			(at 95.25 38.1 0)
 			(effects
 				(font
@@
 		)
 		(property "Datasheet" "~"
-			(at 95.25 33.02 0)
+			(at 95.25 38.1 0)
 			(effects
 				(font
@@
 		)
 		(property "Description" "Unpolarized capacitor, small symbol"
-			(at 95.25 33.02 0)
+			(at 95.25 38.1 0)
 			(effects
 				(font
@@
 	(symbol
 		(lib_id "Device:C_Polarized_Small")
-		(at 138.43 33.02 0)
+		(at 138.43 38.1 0)
 		(unit 1)
 		(exclude_from_sim no)
@@
 		(fields_autoplaced yes)
 		(property "Reference" "C3"
-			(at 140.97 31.2038 0)
+			(at 140.97 36.2838 0)
 			(effects
 				(font
@@
 		)
 		(property "Value" "100uF"
-			(at 140.97 33.7438 0)
+			(at 140.97 38.8238 0)
 			(effects
 				(font
@@
 		)
 		(property "Footprint" ""
-			(at 138.43 33.02 0)
+			(at 138.43 38.1 0)
 			(effects
 				(font
@@
 		)
 		(property "Datasheet" "~"
-			(at 138.43 33.02 0)
+			(at 138.43 38.1 0)
 			(effects
 				(font
@@
 		)
 		(property "Description" "Polarized capacitor, small symbol"
-			(at 138.43 33.02 0)
-			(effects
-				(font
+			(at 138.43 38.1 0)
+			(effects
+				(font

Commit message: m
Parts:
- removed Q1: PMOS, symbol Simulation_SPICE:PMOS
- added J6, J7, J8, J9: Conn_01x01, symbol Connector_Generic:Conn_01x01
- added Q1: SQJ415EP-T1_GE3, Library:SOT_SQJ415EP_VIS, symbol Library:PMOS
Connections:
- net +12V: now also J6.1 (Pin_1), J7.1 (Pin_1), J8.1 (Pin_1), J9.1 (Pin_1)
- net GND: now also J1.2; no longer J1.1
- net at D38.1 (A1), F1.2: now also Q1.5 (D)
- net at F1.1: now also J1.1; no longer J1.2
- net at D39.1 (K), J5.1 (Pin_1), R117.1: now also Q1.1 (S), Q1.2 (S), Q1.3 (S)
- net at D39.2 (A), R116.1, R117.2: now also Q1.4 (G)
Other:
- note added: "12V WIRE JUMPER PADS"
- note added: "PWR REG"
- moved on the sheet: C26, C3, C30, C32, C4, C5, C6, C9, D38, D39, F1, J1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

Commit message: m
Parts:
- C32, C6: footprint Capacitor_SMD:C_0603_1608Metric -> Capacitor_SMD:C_0805_2012Metric
- C5: value 0.1uF -> 2.2uF; footprint Capacitor_SMD:C_0603_1608Metric -> Capacitor_SMD:C_0805_2012Metric
Other:
- moved on the sheet: C5
